File: kicad/design_emb.sch (KiCad schematic (older format))
At the start: 0 parts

Commit message: creacion bus y libreria
Changed lines of the file:
@@
 LIBS:stm32
 LIBS:Lattice
+LIBS:stm32f446zetx
 LIBS:design_emb-cache
 EELAYER 25 0
@@
 F0 "Sheet1" 60
 F1 "hoja1.sch" 60
+F2 "FMC[15:0]" I R 14350 1800 60
 $EndSheet
 $EndSCHEMATC
