File: kicad/design_emb.sch (KiCad schematic (older format))
At the start: 0 parts

Commit message: reguladores y conexión a stm32
Changed lines of the file:
@@
 F0 "Sheet1" 60
 F1 "STM32F446ZETx.sch" 60
-F2 "FMC[15:0]" I R 21950 5800 60
+F2 "FMC[15:0]" I R 21950 7850 118
+F3 "FMC_AD[15:0]" I R 21950 8300 118
+F4 "FMC_CLK" I R 21950 8700 118
+F5 "FMC_NOE" I R 21950 9200 118
+F6 "FMC_NWE" I R 21950 9700 118
+F7 "FMC_WAIT" I R 21950 10250 118
+F8 "FMC_NE1" I R 21950 10750 118
+F9 "FMC_A[24:16]" I R 21950 11200 118
+F10 "FMC_NBL[1:0]" I R 21950 11650 118
+F11 "FMC_NL" I R 21950 12050 118
+F12 "FMC_NE2" I R 21950 12500 118
+F13 "VDD_3V3" I R 21950 14800 118
 $EndSheet
 $Sheet
@@
 $EndSheet
 $Sheet
-S 13050 19300 5950 4300
+S 16250 19300 5950 4300
 U 5B986AB9
 F0 "Sheet4" 60
 F1 "power.sch" 60
+F2 "+3V3" O R 22200 20600 118
+F3 "+3V3_FPGA" O R 22200 21050 118
+F4 "+1V2_FPGA" O R 22200 21400 118
 $EndSheet
+Wire Wire Line
+	22200 20600 23850 20600
+Wire Wire Line
+	23850 20600 23850 14800
+Wire Wire Line
+	23850 14800 21950 14800
 $EndSCHEMATC

Commit message: comunicación omega2 y stm32
Parts:
- added J?: Conn_01x03, symbol conn:Conn_01x03
- added U? (x2): SRX.X.TCT, TO_SOT_Packages_SMD:SOT-143, symbol ESD_Protection:SRX.X.TCT
Connections:
- net labels added: GND, RX_OUT, SERIAL_RX, SERIAL_TX, TX_IN
- wire segments 3 -> 24
- no-connect marks 0 -> 2
Other:
- note added: "SR3.3.TCT / SR2.8.TCT"
- note added: "User serial communication\n\n"
Changed lines of the file:
@@
 F12 "FMC_NE2" I R 21950 12500 118
 F13 "VDD_3V3" I R 21950 14800 118
-$EndSheet
-$Sheet
-S 28900 4950 5200 7550
-U 5B86E517
-F0 "Sheet2" 60
-F1 "OMEGA2sch.sch" 60
+F14 "UART5_TX" O R 21950 6250 118
+F15 "UART5_RX" I R 21950 6450 118
 $EndSheet
 $Sheet
@@
 Wire Wire Line
 	23850 14800 21950 14800
+$Comp
+L ESD_Protection:SRX.X.TCT U?
+U 1 1 5B9A3C31
+P 41100 3350
+AR Path="/5B7D9546/5B9A3C31" Ref="U?"  Part="1"
+AR Path="/5B9A3C31" Ref="U?"  Part="1"
+F 0 "U?" H 41000 3150 60  0000 C CNN
+F 1 "SRX.X.TCT" H 41100 3591 60  0000 C CNN
+F 2 "TO_SOT_Packages_SMD:SOT-143" H 41100 3350 60  0001 C CNN
+F 3 "https://co.mouser.com/datasheet/2/761/sr2_8-1277654.pdf" H 41100 3350 60  0001 C CNN
+	1    41100 3350
+	1    0    0    -1
+$EndComp
+Wire Wire Line
+	40800 3250 40700 3250
+$Comp
+L power:GND #PWR?
+U 1 1 5B9A3C39
+P 40700 3250
+AR Path="/5B7D9546/5B9A3C39" Ref="#PWR?"  Part="1"
+AR Path="/5B9A3C39" Ref="#PWR?"  Part="1"
+F 0 "#PWR?" H 40700 3000 50  0001 C CNN
+F 1 "GND" V 40705 3122 50  0000 R CNN
+F 2 "" H 40700 3250 50  0001 C CNN
+F 3 "" H 40700 3250 50  0001 C CNN
+	1    40700 3250
+	0    1    1    0
+$EndComp
+Wire Wire Line
+	40800 3450 40250 3450
+$Comp
+L ESD_Protection:SRX.X.TCT U?
+U 1 1 5B9A3C41
+P 41100 3900
+AR Path="/5B7D9546/5B9A3C41" Ref="U?"  Part="1"
+AR Path="/5B9A3C41" Ref="U?"  Part="1"
+F 0 "U?" H 41000 3700 60  0000 C CNN
+F 1 "SRX.X.TCT" H 41100 4141 60  0000 C CNN
+F 2 "TO_SOT_Packages_SMD:SOT-143" H 41100 3900 60  0001 C CNN
+F 3 "https://co.mouser.com/datasheet/2/761/sr2_8-1277654.pdf" H 41100 3900 60  0001 C CNN
+	1    41100 3900
+	1    0    0    -1
+$EndComp
+Wire Wire Line
+	40800 3800 40700 3800
+$Comp
+L power:GND #PWR?
+U 1 1 5B9A3C49
+P 40700 3800
+AR Path="/5B7D9546/5B9A3C49" Ref="#PWR?"  Part="1"
+AR Path="/5B9A3C49" Ref="#PWR?"  Part="1"
+F 0 "#PWR?" H 40700 3550 50  0001 C CNN
+F 1 "GND" V 40705 3672 50  0000 R CNN
+F 2 "" H 40700 3800 50  0001 C CNN
+F 3 "" H 40700 3800 50  0001 C CNN
+	1    40700 3800
+	0    1    1    0
+$EndComp
+Wire Wire Line
+	40800 4000 40250 4000
+NoConn ~ 41400 3250
+NoConn ~ 41400 3800
+Wire Wire Line
+	42200 3450 41400 3450
+Wire Wire Line
+	42200 3550 41500 3550
+Wire Wire Line
+	41500 3550 41500 4000
+Wire Wire Line
+	41500 4000 41400 4000
+Text Label 42050 3450 2    60   ~ 0
+RX_OUT
+Text Label 42000 3550 2    60   ~ 0
+TX_IN
+Wire Wire Line
+	42200 3650 42100 3650
+Wire Wire Line
+	42100 3650 42100 3850
+$Comp
+L power:GND #PWR?
+U 1 1 5B9A3C62
+P 42100 3850
+AR Path="/5B7D9546/5B9A3C62" Ref="#PWR?"  Part="1"
+AR Path="/5B9A3C62" Ref="#PWR?"  Part="1"
+F 0 "#PWR?" H 42100 3600 50  0001 C CNN
+F 1 "GND" H 42105 3677 50  0000 C CNN
+F 2 "" H 42100 3850 50  0001 C CNN
+F 3 "" H 42100 3850 50  0001 C CNN
+	1    42100 3850
+	1    0    0    -1
+$EndComp
+Text Notes 43350 2850 2    197  Italic 0
+User serial communication\n\n
+Text Notes 41950 4400 2    98   ~ 0
+SR3.3.TCT / SR2.8.TCT
+$Sheet
+S 28900 4950 5200 7550
+U 5B86E517
+F0 "Sheet2" 60
+F1 "OMEGA2sch.sch" 60
+F2 "VDD" I L 28900 11450 118
+F3 "V3.3OUT" I L 28900 11650 118
+F4 "SPI_MISO" B L 28900 7200 118
+F5 "SPI_MOSI" B L 28900 7450 118
+F6 "SPI_CS" B L 28900 7750 118
+F7 "SPI_CLK" B L 28900 8000 118
+F8 "SERIAL_TX" O R 34100 5600 118
+F9 "SERIAL_RX" I R 34100 5850 118
+F10 "UART_RX" I L 28900 5600 118
+F11 "UART_TX" O L 28900 5850 118
+$EndSheet
+Wire Wire Line
+	21950 6250 25400 6250
+Wire Wire Line
+	25400 6250 25400 5600
+Wire Wire Line
+	25400 5600 28900 5600
+Wire Wire Line
+	21950 6450 25600 6450
+Wire Wire Line
+	25600 5850 28900 5850
+Wire Wire Line
+	25600 5850 25600 6450
+Text Label 40300 3450 0    60   ~ 0
+SERIAL_RX
+Text Label 40300 4000 0    60   ~ 0
+SERIAL_TX
+Wire Wire Line
+	34650 5600 34100 5600
+Text Label 34150 5600 0    60   ~ 0
+SERIAL_RX
+Wire Wire Line
+	34650 5850 34100 5850
+Text Label 34150 5850 0    60   ~ 0
+SERIAL_TX
+$Comp
+L conn:Conn_01x03 J?
+U 1 1 5B9A3C53
+P 42400 3550
+AR Path="/5B7D9546/5B9A3C53" Ref="J?"  Part="1"
+AR Path="/5B9A3C53" Ref="J?"  Part="1"
+F 0 "J?" H 42480 3592 50  0000 L CNN
+F 1 "Conn_01x03" H 42480 3501 50  0000 L CNN
+F 2 "" H 42400 3550 50  0001 C CNN
+F 3 "~" H 42400 3550 50  0001 C CNN
+	1    42400 3550
+	1    0    0    -1
+$EndComp
+Wire Wire Line
+	28900 11450 28100 11450
+Wire Wire Line
+	28100 11450 28100 14800
+Wire Wire Line
+	28100 14800 23850 14800
+Connection ~ 23850 14800
 $EndSCHEMATC

Commit message: design_emb.sch
Connections:
- net labels added: CONTROL, ENABLE, FMC_A, FMC_AD
- wire segments 24 -> 27
Changed lines of the file:
@@
 EESchema Schematic File Version 4
-LIBS:power
-LIBS:74xx
 LIBS:stm32f446zetx
 LIBS:design_emb-cache
@@
 F0 "Sheet1" 60
 F1 "STM32F446ZETx.sch" 60
-F2 "FMC[15:0]" I R 21950 7850 118
-F3 "FMC_AD[15:0]" I R 21950 8300 118
-F4 "FMC_CLK" I R 21950 8700 118
-F5 "FMC_NOE" I R 21950 9200 118
-F6 "FMC_NWE" I R 21950 9700 118
-F7 "FMC_WAIT" I R 21950 10250 118
-F8 "FMC_NE1" I R 21950 10750 118
-F9 "FMC_A[24:16]" I R 21950 11200 118
-F10 "FMC_NBL[1:0]" I R 21950 11650 118
-F11 "FMC_NL" I R 21950 12050 118
-F12 "FMC_NE2" I R 21950 12500 118
-F13 "VDD_3V3" I R 21950 14800 118
-F14 "UART5_TX" O R 21950 6250 118
-F15 "UART5_RX" I R 21950 6450 118
+F2 "FMC_AD[15:0]" I R 21950 8300 118
+F3 "FMC_A[24:16]" I R 21950 11200 118
+F4 "FMC_NBL[1:0]" I R 21950 11650 118
+F5 "VDD_3V3" I R 21950 14800 118
+F6 "UART5_TX" O R 21950 6250 118
+F7 "UART5_RX" I R 21950 6450 118
+F8 "Cont[5...0]" O R 21950 13000 118
 $EndSheet
 $Sheet
@@
 F0 "sheet3" 60
 F1 "fpga.sch" 60
-$EndSheet
-$Sheet
-S 16250 19300 5950 4300
+F2 "FMC_AD[15...0]" B L 29050 16450 118
+F3 "FMC_A[16...24]" B L 29050 16750 118
+F4 "ICE40_ENABLE[1...0]" B L 29050 16150 118
+F5 "RESET_B" B L 29050 15800 118
+F6 "ICE40_SPI[3...0]" B L 29050 15650 118
+F7 "Cont[5...0]" B L 29050 17000 118
+$EndSheet
+$Sheet
+S 16250 19250 5950 4300
 U 5B986AB9
 F0 "Sheet4" 60
 F1 "power.sch" 60
-F2 "+3V3" O R 22200 20600 118
-F3 "+3V3_FPGA" O R 22200 21050 118
-F4 "+1V2_FPGA" O R 22200 21400 118
-$EndSheet
-Wire Wire Line
-	22200 20600 23850 20600
-Wire Wire Line
-	23850 20600 23850 14800
+F2 "+3V3" O R 22200 20550 118
+F3 "+3V3_FPGA" O R 22200 21000 118
+F4 "+1V2_FPGA" O R 22200 21350 118
+$EndSheet
+Wire Wire Line
+	22200 20550 23850 20550
+Wire Wire Line
+	23850 20550 23850 14800
 Wire Wire Line
 	23850 14800 21950 14800
@@
 F2 "VDD" I L 28900 11450 118
 F3 "V3.3OUT" I L 28900 11650 118
-F4 "SPI_MISO" B L 28900 7200 118
-F5 "SPI_MOSI" B L 28900 7450 118
-F6 "SPI_CS" B L 28900 7750 118
-F7 "SPI_CLK" B L 28900 8000 118
-F8 "SERIAL_TX" O R 34100 5600 118
-F9 "SERIAL_RX" I R 34100 5850 118
-F10 "UART_RX" I L 28900 5600 118
-F11 "UART_TX" O L 28900 5850 118
+F4 "SERIAL_TX" O R 34100 5600 118
+F5 "SERIAL_RX" I R 34100 5850 118
+F6 "UART_RX" I L 28900 5600 118
+F7 "UART_TX" O L 28900 5850 118
+F8 "RST" B L 28900 11900 118
+F9 "OMEGA_SPI[3...0]" B L 28900 12400 118
 $EndSheet
 Wire Wire Line
@@
 	28100 14800 23850 14800
 Connection ~ 23850 14800
+Text Label 28300 16450 0    118  ~ 0
+FMC_AD
+Text Label 28300 16750 0    118  ~ 0
+FMC_A
+Wire Bus Line
+	21950 8300 23000 8300
+Text Label 22150 8300 0    118  ~ 0
+FMC_AD
+Wire Bus Line
+	21950 11200 22800 11200
+Text Label 22100 11200 0    118  ~ 0
+FMC_A
+Wire Bus Line
+	21950 13000 22500 13000
+Text Label 22050 13000 0    118  ~ 0
+CONTROL
+Text Label 29000 17000 2    118  ~ 0
+CONTROL
+Text Label 28300 16150 0    118  ~ 0
+ENABLE
+Wire Bus Line
+	21950 11650 22800 11650
+Text Label 22100 11650 0    118  ~ 0
+ENABLE
+Wire Wire Line
+	29050 15800 28450 15800
+Wire Wire Line
+	28450 15800 28450 11900
+Wire Wire Line
+	28450 11900 28900 11900
+Wire Bus Line
+	29050 15650 28700 15650
+Wire Bus Line
+	28700 15650 28700 12400
+Wire Bus Line
+	28700 12400 28900 12400
+Wire Bus Line
+	28300 16450 29050 16450
+Wire Bus Line
+	28300 16150 29050 16150
+Wire Bus Line
+	28300 16750 29050 16750
+Wire Bus Line
+	28250 17000 29050 17000
 $EndSCHEMATC

Commit message: footprints y JTAG
Parts:
- J1: renamed from J?; footprint (none) -> Connectors_Terminal_Blocks:TerminalBlock_Altech_AK300-3_P5.00mm
- gave numbers to parts that had none: 2
Connections:
- wire segments 27 -> 25
Changed lines of the file:
@@
 $EndDescr
 $Sheet
-S 10100 5400 11850 10200
+S 9900 7150 11850 10200
 U 5B7D9546
 F0 "Sheet1" 60
 F1 "STM32F446ZETx.sch" 60
-F2 "FMC_AD[15:0]" I R 21950 8300 118
-F3 "FMC_A[24:16]" I R 21950 11200 118
-F4 "FMC_NBL[1:0]" I R 21950 11650 118
-F5 "VDD_3V3" I R 21950 14800 118
-F6 "UART5_TX" O R 21950 6250 118
-F7 "UART5_RX" I R 21950 6450 118
-F8 "Cont[5...0]" O R 21950 13000 118
-$EndSheet
-$Sheet
-S 29050 15350 6000 8800
+F2 "FMC_AD[15:0]" I R 21750 14150 118
+F3 "FMC_A[24:16]" I R 21750 14450 118
+F4 "FMC_NBL[1:0]" I R 21750 13850 118
+F5 "VDD_3V3" I R 21750 16550 118
+F6 "UART5_TX" O R 21750 8000 118
+F7 "UART5_RX" I R 21750 8200 118
+F8 "Cont[5...0]" O R 21750 14750 118
+F9 "BOOT0" I R 21750 9000 118
+F10 "JTAG[5...0]" B R 21750 8750 118
+$EndSheet
+$Sheet
+S 28850 17100 6000 8800
 U 5B8BCB6B
 F0 "sheet3" 60
 F1 "fpga.sch" 60
-F2 "FMC_AD[15...0]" B L 29050 16450 118
-F3 "FMC_A[16...24]" B L 29050 16750 118
-F4 "ICE40_ENABLE[1...0]" B L 29050 16150 118
-F5 "RESET_B" B L 29050 15800 118
-F6 "ICE40_SPI[3...0]" B L 29050 15650 118
-F7 "Cont[5...0]" B L 29050 17000 118
-$EndSheet
-$Sheet
-S 16250 19250 5950 4300
+F2 "FMC_AD[15...0]" B L 28850 18200 118
+F3 "FMC_A[16...24]" B L 28850 18500 118
+F4 "ICE40_ENABLE[1...0]" B L 28850 17900 118
+F5 "ICE40_SPI[3...0]" B L 28850 17400 118
+F6 "Cont[5...0]" B L 28850 18750 118
+$EndSheet
+$Sheet
+S 16050 21000 5950 4300
 U 5B986AB9
 F0 "Sheet4" 60
 F1 "power.sch" 60
-F2 "+3V3" O R 22200 20550 118
-F3 "+3V3_FPGA" O R 22200 21000 118
-F4 "+1V2_FPGA" O R 22200 21350 118
-$EndSheet
-Wire Wire Line
-	22200 20550 23850 20550
-Wire Wire Line
-	23850 20550 23850 14800
-Wire Wire Line
-	23850 14800 21950 14800
+F2 "+3V3" O R 22000 22300 118
+F3 "+3V3_FPGA" O R 22000 22750 118
+F4 "+1V2_FPGA" O R 22000 23100 118
+$EndSheet
+Wire Wire Line
+	22000 22300 23650 22300
+Wire Wire Line
+	23650 22300 23650 16550
+Wire Wire Line
+	23650 16550 21750 16550
 $Comp
 L ESD_Protection:SRX.X.TCT U?
@@
 P 41100 3350
 AR Path="/5B7D9546/5B9A3C31" Ref="U?"  Part="1"
-AR Path="/5B9A3C31" Ref="U?"  Part="1"
-F 0 "U?" H 41000 3150 60  0000 C CNN
+AR Path="/5B9A3C31" Ref="U1"  Part="1"
+F 0 "U1" H 41000 3150 60  0000 C CNN
 F 1 "SRX.X.TCT" H 41100 3591 60  0000 C CNN
 F 2 "TO_SOT_Packages_SMD:SOT-143" H 41100 3350 60  0001 C CNN
@@
 P 40700 3250
 AR Path="/5B7D9546/5B9A3C39" Ref="#PWR?"  Part="1"
-AR Path="/5B9A3C39" Ref="#PWR?"  Part="1"
-F 0 "#PWR?" H 40700 3000 50  0001 C CNN
+AR Path="/5B9A3C39" Ref="#PWR01"  Part="1"
+F 0 "#PWR01" H 40700 3000 50  0001 C CNN
 F 1 "GND" V 40705 3122 50  0000 R CNN
 F 2 "" H 40700 3250 50  0001 C CNN
@@
 P 41100 3900
 AR Path="/5B7D9546/5B9A3C41" Ref="U?"  Part="1"
-AR Path="/5B9A3C41" Ref="U?"  Part="1"
-F 0 "U?" H 41000 3700 60  0000 C CNN
+AR Path="/5B9A3C41" Ref="U2"  Part="1"
+F 0 "U2" H 41000 3700 60  0000 C CNN
 F 1 "SRX.X.TCT" H 41100 4141 60  0000 C CNN
 F 2 "TO_SOT_Packages_SMD:SOT-143" H 41100 3900 60  0001 C CNN
@@
 P 40700 3800
 AR Path="/5B7D9546/5B9A3C49" Ref="#PWR?"  Part="1"
-AR Path="/5B9A3C49" Ref="#PWR?"  Part="1"
-F 0 "#PWR?" H 40700 3550 50  0001 C CNN
+AR Path="/5B9A3C49" Ref="#PWR02"  Part="1"
+F 0 "#PWR02" H 40700 3550 50  0001 C CNN
 F 1 "GND" V 40705 3672 50  0000 R CNN
 F 2 "" H 40700 3800 50  0001 C CNN
@@
 P 42100 3850
 AR Path="/5B7D9546/5B9A3C62" Ref="#PWR?"  Part="1"
-AR Path="/5B9A3C62" Ref="#PWR?"  Part="1"
-F 0 "#PWR?" H 42100 3600 50  0001 C CNN
+AR Path="/5B9A3C62" Ref="#PWR03"  Part="1"
+F 0 "#PWR03" H 42100 3600 50  0001 C CNN
 F 1 "GND" H 42105 3677 50  0000 C CNN
 F 2 "" H 42100 3850 50  0001 C CNN
@@
 SR3.3.TCT / SR2.8.TCT
 $Sheet
-S 28900 4950 5200 7550
+S 28700 6700 5200 7550
 U 5B86E517
 F0 "Sheet2" 60
 F1 "OMEGA2sch.sch" 60
-F2 "VDD" I L 28900 11450 118
-F3 "V3.3OUT" I L 28900 11650 118
-F4 "SERIAL_TX" O R 34100 5600 118
-F5 "SERIAL_RX" I R 34100 5850 118
-F6 "UART_RX" I L 28900 5600 118
-F7 "UART_TX" O L 28900 5850 118
-F8 "RST" B L 28900 11900 118
-F9 "OMEGA_SPI[3...0]" B L 28900 12400 118
-$EndSheet
-Wire Wire Line
-	21950 6250 25400 6250
-Wire Wire Line
-	25400 6250 25400 5600
-Wire Wire Line
-	25400 5600 28900 5600
-Wire Wire Line
-	21950 6450 25600 6450
-Wire Wire Line
-	25600 5850 28900 5850
-Wire Wire Line
-	25600 5850 25600 6450
+F2 "3V3_VDD" I L 28700 13200 118
+F3 "SERIAL_TX" O R 33900 7350 118
+F4 "SERIAL_RX" I R 33900 7600 118
+F5 "UART_RX" I L 28700 7350 118
+F6 "UART_TX" O L 28700 7600 118
+F7 "OMEGA_SPI[3...0]" B L 28700 14150 118
+F8 "JTAG[5...0]" B L 28700 8750 118
+F9 "BOOT0" O L 28700 9000 118
+$EndSheet
+Wire Wire Line
+	21750 8000 25200 8000
+Wire Wire Line
+	25200 8000 25200 7350
+Wire Wire Line
+	25200 7350 28700 7350
+Wire Wire Line
+	21750 8200 25400 8200
+Wire Wire Line
+	25400 7600 28700 7600
+Wire Wire Line
+	25400 7600 25400 8200
 Text Label 40300 3450 0    60   ~ 0
 SERIAL_RX
@@
 SERIAL_TX
 Wire Wire Line
-	34650 5600 34100 5600
-Text Label 34150 5600 0    60   ~ 0
+	34450 7350 33900 7350
+Text Label 33950 7350 0    60   ~ 0
 SERIAL_RX
 Wire Wire Line
-	34650 5850 34100 5850
-Text Label 34150 5850 0    60   ~ 0
+	34450 7600 33900 7600
+Text Label 33950 7600 0    60   ~ 0
 SERIAL_TX
 $Comp
@@
 P 42400 3550
 AR Path="/5B7D9546/5B9A3C53" Ref="J?"  Part="1"
-AR Path="/5B9A3C53" Ref="J?"  Part="1"
-F 0 "J?" H 42480 3592 50  0000 L CNN
+AR Path="/5B9A3C53" Ref="J1"  Part="1"
+F 0 "J1" H 42480 3592 50  0000 L CNN
 F 1 "Conn_01x03" H 42480 3501 50  0000 L CNN
-F 2 "" H 42400 3550 50  0001 C CNN
+F 2 "Connectors_Terminal_Blocks:TerminalBlock_Altech_AK300-3_P5.00mm" H 42400 3550 50  0001 C CNN
 F 3 "~" H 42400 3550 50  0001 C CNN
 	1    42400 3550
@@
 $EndComp
 Wire Wire Line
-	28900 11450 28100 11450
-Wire Wire Line
-	28100 11450 28100 14800
-Wire Wire Line
-	28100 14800 23850 14800
-Connection ~ 23850 14800
-Text Label 28300 16450 0    118  ~ 0
+	28700 13200 27900 13200
+Wire Wire Line
+	27900 13200 27900 16550
+Wire Wire Line
+	27900 16550 23650 16550
+Connection ~ 23650 16550
+Text Label 28100 18200 0    118  ~ 0
 FMC_AD
-Text Label 28300 16750 0    118  ~ 0
+Text Label 28100 18500 0    118  ~ 0
 FMC_A
 Wire Bus Line
-	21950 8300 23000 8300
-Text Label 22150 8300 0    118  ~ 0
+	21750 14150 22800 14150
+Text Label 21950 14150 0    118  ~ 0
 FMC_AD
-Wire Bus Line
-	21950 11200 22800 11200
-Text Label 22100 11200 0    118  ~ 0
+Text Label 21900 14450 0    118  ~ 0
 FMC_A
 Wire Bus Line
-	21950 13000 22500 13000
-Text Label 22050 13000 0    118  ~ 0
+	21750 14750 22800 14750
+Text Label 21850 14750 0    118  ~ 0
 CONTROL
-Text Label 29000 17000 2    118  ~ 0
+Text Label 28800 18750 2    118  ~ 0
 CONTROL
-Text Label 28300 16150 0    118  ~ 0
+Text Label 28100 17900 0    118  ~ 0
 ENABLE
 Wire Bus Line
-	21950 11650 22800 11650
-Text Label 22100 11650 0    118  ~ 0
+	21750 13850 22800 13850
+Text Label 21900 13850 0    118  ~ 0
 ENABLE
-Wire Wire Line
-	29050 15800 28450 15800
-Wire Wire Line
-	28450 15800 28450 11900
-Wire Wire Line
-	28450 11900 28900 11900
-Wire Bus Line
-	29050 15650 28700 15650
-Wire Bus Line
-	28700 15650 28700 12400
-Wire Bus Line
-	28700 12400 28900 12400
-Wire Bus Line
-	28300 16450 29050 16450
-Wire Bus Line
-	28300 16150 29050 16150
-Wire Bus Line
-	28300 16750 29050 16750
-Wire Bus Line
-	28250 17000 29050 17000
+Wire Bus Line
+	28850 17400 28500 17400
+Wire Bus Line
+	28500 17400 28500 14150
+Wire Bus Line
+	28500 14150 28700 14150
+Wire Bus Line
+	27950 18200 28850 18200
+Wire Bus Line
+	27950 17900 28850 17900
+Wire Bus Line
+	27950 18500 28850 18500
+Wire Bus Line
+	27950 18750 28850 18750
+Wire Bus Line
+	21750 14450 22800 14450
+Wire Bus Line
+	21750 8750 28700 8750
+Wire Wire Line
+	28700 9000 21750 9000
 $EndSCHEMATC

Commit message: perifericos stm32
Connections:
- wire segments 25 -> 28
Changed lines of the file:
@@
 $Descr A0 46811 33110
 encoding utf-8
-Sheet 1 5
+Sheet 1 6
 Title ""
 Date ""
@@
 $EndDescr
 $Sheet
-S 9900 7150 11850 10200
+S 11100 7100 11850 10200
 U 5B7D9546
 F0 "Sheet1" 60
 F1 "STM32F446ZETx.sch" 60
-F2 "FMC_AD[15:0]" I R 21750 14150 118
-F3 "FMC_A[24:16]" I R 21750 14450 118
-F4 "FMC_NBL[1:0]" I R 21750 13850 118
-F5 "VDD_3V3" I R 21750 16550 118
-F6 "UART5_TX" O R 21750 8000 118
-F7 "UART5_RX" I R 21750 8200 118
-F8 "Cont[5...0]" O R 21750 14750 118
-F9 "BOOT0" I R 21750 9000 118
-F10 "JTAG[5...0]" B R 21750 8750 118
-$EndSheet
-$Sheet
-S 28850 17100 6000 8800
+F2 "FMC_AD[15:0]" I R 22950 14100 118
+F3 "FMC_A[24:16]" I R 22950 14400 118
+F4 "FMC_NBL[1:0]" I R 22950 13800 118
+F5 "VDD_3V3" I R 22950 16500 118
+F6 "UART5_TX" O R 22950 7950 118
+F7 "UART5_RX" I R 22950 8150 118
+F8 "Cont[5...0]" O R 22950 14700 118
+F9 "BOOT0" I R 22950 8950 118
+F10 "JTAG[5...0]" B R 22950 8700 118
+F11 "OUT_REL1" O L 11100 13000 118
+F12 "OUT_REL2" O L 11100 13500 118
+$EndSheet
+$Sheet
+S 30050 17050 6000 8800
 U 5B8BCB6B
 F0 "sheet3" 60
 F1 "fpga.sch" 60
-F2 "FMC_AD[15...0]" B L 28850 18200 118
-F3 "FMC_A[16...24]" B L 28850 18500 118
-F4 "ICE40_ENABLE[1...0]" B L 28850 17900 118
-F5 "ICE40_SPI[3...0]" B L 28850 17400 118
-F6 "Cont[5...0]" B L 28850 18750 118
-$EndSheet
-$Sheet
-S 16050 21000 5950 4300
+F2 "FMC_AD[15...0]" B L 30050 18150 118
+F3 "FMC_A[16...24]" B L 30050 18450 118
+F4 "ICE40_ENABLE[1...0]" B L 30050 17850 118
+F5 "ICE40_SPI[3...0]" B L 30050 17350 118
+F6 "Cont[5...0]" B L 30050 18700 118
+$EndSheet
+$Sheet
+S 17250 20950 5950 4300
 U 5B986AB9
 F0 "Sheet4" 60
 F1 "power.sch" 60
-F2 "+3V3" O R 22000 22300 118
-F3 "+3V3_FPGA" O R 22000 22750 118
-F4 "+1V2_FPGA" O R 22000 23100 118
-$EndSheet
-Wire Wire Line
-	22000 22300 23650 22300
-Wire Wire Line
-	23650 22300 23650 16550
-Wire Wire Line
-	23650 16550 21750 16550
+F2 "+3V3" O R 23200 22250 118
+F3 "+3V3_FPGA" O R 23200 22700 118
+F4 "+1V2_FPGA" O R 23200 23050 118
+$EndSheet
+Wire Wire Line
+	23200 22250 24850 22250
+Wire Wire Line
+	24850 22250 24850 16500
+Wire Wire Line
+	24850 16500 22950 16500
 $Comp
 L ESD_Protection:SRX.X.TCT U?
@@
 SR3.3.TCT / SR2.8.TCT
 $Sheet
-S 28700 6700 5200 7550
+S 29900 6650 5200 7550
 U 5B86E517
 F0 "Sheet2" 60
 F1 "OMEGA2sch.sch" 60
-F2 "3V3_VDD" I L 28700 13200 118
-F3 "SERIAL_TX" O R 33900 7350 118
-F4 "SERIAL_RX" I R 33900 7600 118
-F5 "UART_RX" I L 28700 7350 118
-F6 "UART_TX" O L 28700 7600 118
-F7 "OMEGA_SPI[3...0]" B L 28700 14150 118
-F8 "JTAG[5...0]" B L 28700 8750 118
-F9 "BOOT0" O L 28700 9000 118
-$EndSheet
-Wire Wire Line
-	21750 8000 25200 8000
-Wire Wire Line
-	25200 8000 25200 7350
-Wire Wire Line
-	25200 7350 28700 7350
-Wire Wire Line
-	21750 8200 25400 8200
-Wire Wire Line
-	25400 7600 28700 7600
-Wire Wire Line
-	25400 7600 25400 8200
+F2 "3V3_VDD" I L 29900 13150 118
+F3 "SERIAL_TX" O R 35100 7300 118
+F4 "SERIAL_RX" I R 35100 7550 118
+F5 "UART_RX" I L 29900 7300 118
+F6 "UART_TX" O L 29900 7550 118
+F7 "OMEGA_SPI[3...0]" B L 29900 14100 118
+F8 "JTAG[5...0]" B L 29900 8700 118
+F9 "BOOT0" O L 29900 8950 118
+$EndSheet
+Wire Wire Line
+	22950 7950 26400 7950
+Wire Wire Line
+	26400 7950 26400 7300
+Wire Wire Line
+	26400 7300 29900 7300
+Wire Wire Line
+	22950 8150 26600 8150
+Wire Wire Line
+	26600 7550 29900 7550
+Wire Wire Line
+	26600 7550 26600 8150
 Text Label 40300 3450 0    60   ~ 0
 SERIAL_RX
@@
 SERIAL_TX
 Wire Wire Line
-	34450 7350 33900 7350
-Text Label 33950 7350 0    60   ~ 0
+	35650 7300 35100 7300
+Text Label 35150 7300 0    60   ~ 0
 SERIAL_RX
 Wire Wire Line
-	34450 7600 33900 7600
-Text Label 33950 7600 0    60   ~ 0
+	35650 7550 35100 7550
+Text Label 35150 7550 0    60   ~ 0
 SERIAL_TX
 $Comp
@@
 $EndComp
 Wire Wire Line
-	28700 13200 27900 13200
-Wire Wire Line
-	27900 13200 27900 16550
-Wire Wire Line
-	27900 16550 23650 16550
-Connection ~ 23650 16550
-Text Label 28100 18200 0    118  ~ 0
+	29900 13150 29100 13150
+Wire Wire Line
+	29100 13150 29100 16500
+Wire Wire Line
+	29100 16500 24850 16500
+Connection ~ 24850 16500
+Text Label 29300 18150 0    118  ~ 0
 FMC_AD
-Text Label 28100 18500 0    118  ~ 0
+Text Label 29300 18450 0    118  ~ 0
 FMC_A
 Wire Bus Line
-	21750 14150 22800 14150
-Text Label 21950 14150 0    118  ~ 0
+	22950 14100 24000 14100
+Text Label 23150 14100 0    118  ~ 0
 FMC_AD
-Text Label 21900 14450 0    118  ~ 0
+Text Label 23100 14400 0    118  ~ 0
 FMC_A
 Wire Bus Line
-	21750 14750 22800 14750
-Text Label 21850 14750 0    118  ~ 0
+	22950 14700 24000 14700
+Text Label 23050 14700 0    118  ~ 0
 CONTROL
-Text Label 28800 18750 2    118  ~ 0
+Text Label 30000 18700 2    118  ~ 0
 CONTROL
-Text Label 28100 17900 0    118  ~ 0
+Text Label 29300 17850 0    118  ~ 0
 ENABLE
 Wire Bus Line
-	21750 13850 22800 13850
-Text Label 21900 13850 0    118  ~ 0
+	22950 13800 24000 13800
+Text Label 23100 13800 0    118  ~ 0
 ENABLE
 Wire Bus Line
-	28850 17400 28500 17400
-Wire Bus Line
-	28500 17400 28500 14150
-Wire Bus Line
-	28500 14150 28700 14150
-Wire Bus Line
-	27950 18200 28850 18200
-Wire Bus Line
-	27950 17900 28850 17900
-Wire Bus Line
-	27950 18500 28850 18500
-Wire Bus Line
-	27950 18750 28850 18750
-Wire Bus Line
-	21750 14450 22800 14450
-Wire Bus Line
-	21750 8750 28700 8750
-Wire Wire Line
-	28700 9000 21750 9000
+	30050 17350 29700 17350
+Wire Bus Line
+	29700 17350 29700 14100
+Wire Bus Line
+	29700 14100 29900 14100
+Wire Bus Line
+	29150 18150 30050 18150
+Wire Bus Line
+	29150 17850 30050 17850
+Wire Bus Line
+	29150 18450 30050 18450
+Wire Bus Line
+	29150 18700 30050 18700
+Wire Bus Line
+	22950 14400 24000 14400
+Wire Bus Line
+	22950 8700 29900 8700
+Wire Wire Line
+	29900 8950 22950 8950
+$Sheet
+S 4750 12000 2950 2950
+U 5BACBF11
+F0 "Sheet5" 60
+F1 "perf_stm.sch" 60
+F2 "IN_REL1" I R 7700 13000 118
+F3 "IN_REL2" I R 7700 13500 118
+$EndSheet
+Wire Wire Line
+	19600 23200 19600 23250
+Wire Wire Line
+	11100 13000 7700 13000
+Wire Wire Line
+	11100 13500 7700 13500
 $EndSCHEMATC
