File: kicad/OMEGA2sch.sch (KiCad schematic (older format))
At the start: 1 part

Commit message: comunicación omega2 y stm32
Parts:
- added C?: 100nF, symbol device:CP1
Connections:
- net labels added: SERIAL_RX, SERIAL_TX, UART_RX, UART_TX
- wire segments 6 -> 9
Changed lines of the file:
@@
 $Descr A4 11693 8268
 encoding utf-8
-Sheet 3 5
+Sheet 5 5
 Title ""
 Date ""
@@
 	1    0    0    -1
 $EndComp
-Text HLabel 7050 2500 2    60   Input ~ 0
+Text HLabel 8250 2500 2    60   Input ~ 0
 VDD
 Text HLabel 7050 2600 2    60   Input ~ 0
@@
 Wire Wire Line
 	4550 3500 4650 3500
+Text HLabel 7050 3100 2    60   Output ~ 0
+SERIAL_TX
+Text HLabel 7050 3200 2    60   Input ~ 0
+SERIAL_RX
+Text HLabel 7050 3400 2    60   Input ~ 0
+UART_RX
+Text HLabel 7050 3300 2    60   Output ~ 0
+UART_TX
+Wire Wire Line
+	7050 2500 7950 2500
+$Comp
+L device:CP1 C?
+U 1 1 5B9A6A14
+P 7950 2750
+F 0 "C?" H 8065 2796 50  0000 L CNN
+F 1 "100nF" H 8065 2705 50  0000 L CNN
+F 2 "" H 7950 2750 50  0001 C CNN
+F 3 "" H 7950 2750 50  0001 C CNN
+	1    7950 2750
+	1    0    0    -1
+$EndComp
+Wire Wire Line
+	7950 2600 7950 2500
+Connection ~ 7950 2500
+Wire Wire Line
+	7950 2500 8250 2500
+$Comp
+L power:GND #PWR?
+U 1 1 5B9A6AE7
+P 7950 2900
+F 0 "#PWR?" H 7950 2650 50  0001 C CNN
+F 1 "GND" H 7955 2727 50  0000 C CNN
+F 2 "" H 7950 2900 50  0001 C CNN
+F 3 "" H 7950 2900 50  0001 C CNN
+	1    7950 2900
+	1    0    0    -1
+$EndComp
 $EndSCHEMATC

Commit message: usb omega2
Parts:
- added C?: 0.1uF, symbol device:CP1
- added C?: 33uF, symbol device:CP1
- added D?: D_Scho, symbol device:D_Schottky
- added J?: USB_A, symbol conn:USB_A
- added L?: L, symbol device:L
- added LSRF?: SRF2012-900YA, IND_BOURNS_SRF2012A, symbol SFR2012:SRF2012-900YA
- added U?: RCLAMP0502B, symbol rclamp0502b:RCLAMP0502B
Connections:
- net labels added: USB+, USB-
- wire segments 9 -> 32
Other:
- note added: "+5VDC\n"

Commit message: leds de prueba
Parts:
- added C? (x3): 100nF, symbol device:CP1
- added D?: LED_PROBE, symbol device:LED
- added R?: 10K, symbol device:R
- added R?: 1K, symbol device:R
- added SW?: SW_Push, symbol Switch:SW_Push
Connections:
- net labels added: 3V3_VDD, PROBE, RESET
- wire segments 32 -> 51
Changed lines of the file:
@@
 $EndComp
 Text HLabel 5850 2550 2    60   Input ~ 0
-VDD
+3V3_VDD
 Text HLabel 4650 2650 2    60   Input ~ 0
 V3.3OUT
@@
 L power:GND #PWR?
 U 1 1 5B916F98
-P 5200 4450
-F 0 "#PWR?" H 5200 4200 50  0001 C CNN
-F 1 "GND" V 5205 4322 50  0000 R CNN
-F 2 "" H 5200 4450 50  0001 C CNN
-F 3 "" H 5200 4450 50  0001 C CNN
-	1    5200 4450
-	0    -1   -1   0
+P 5100 5100
+F 0 "#PWR?" H 5100 4850 50  0001 C CNN
+F 1 "GND" V 5105 4972 50  0000 R CNN
+F 2 "" H 5100 5100 50  0001 C CNN
+F 3 "" H 5100 5100 50  0001 C CNN
+	1    5100 5100
+	1    0    0    -1
 $EndComp
 $Comp
 L power:GND #PWR?
 U 1 1 5B916FF6
-P 5200 4550
-F 0 "#PWR?" H 5200 4300 50  0001 C CNN
-F 1 "GND" V 5205 4422 50  0000 R CNN
-F 2 "" H 5200 4550 50  0001 C CNN
-F 3 "" H 5200 4550 50  0001 C CNN
-	1    5200 4550
-	0    -1   -1   0
-$EndComp
-Wire Wire Line
-	4650 4450 5200 4450
-Wire Wire Line
-	4650 4550 5200 4550
+P 4700 5100
+F 0 "#PWR?" H 4700 4850 50  0001 C CNN
+F 1 "GND" V 4705 4972 50  0000 R CNN
+F 2 "" H 4700 5100 50  0001 C CNN
+F 3 "" H 4700 5100 50  0001 C CNN
+	1    4700 5100
+	1    0    0    -1
+$EndComp
+Wire Wire Line
+	4650 4550 4700 4550
 Text HLabel 2150 3450 0    60   BiDi ~ 0
 SPI_CS
@@
 Wire Wire Line
 	7600 4350 7700 4350
+Wire Wire Line
+	2250 2550 1850 2550
+Text Label 1950 2550 0    60   ~ 0
+RESET
+$Comp
+L Switch:SW_Push SW?
+U 1 1 5B9A9974
+P 10000 2900
+F 0 "SW?" V 9954 3048 50  0000 L CNN
+F 1 "SW_Push" V 10045 3048 50  0000 L CNN
+F 2 "" H 10000 3100 50  0001 C CNN
+F 3 "" H 10000 3100 50  0001 C CNN
+	1    10000 2900
+	0    1    1    0
+$EndComp
+$Comp
+L device:CP1 C?
+U 1 1 5B9A9A3A
+P 9550 2700
+F 0 "C?" H 9665 2746 50  0000 L CNN
+F 1 "100nF" H 9665 2655 50  0000 L CNN
+F 2 "" H 9550 2700 50  0001 C CNN
+F 3 "" H 9550 2700 50  0001 C CNN
+	1    9550 2700
+	1    0    0    -1
+$EndComp
+Wire Wire Line
+	9550 2850 9550 3150
+Wire Wire Line
+	9550 3150 9800 3150
+Wire Wire Line
+	10000 3150 10000 3100
+$Comp
+L power:GND #PWR?
+U 1 1 5B9A9FD7
+P 9800 3150
+F 0 "#PWR?" H 9800 2900 50  0001 C CNN
+F 1 "GND" H 9805 2977 50  0000 C CNN
+F 2 "" H 9800 3150 50  0001 C CNN
+F 3 "" H 9800 3150 50  0001 C CNN
+	1    9800 3150
+	1    0    0    -1
+$EndComp
+Connection ~ 9800 3150
+Wire Wire Line
+	9800 3150 10000 3150
+Wire Wire Line
+	9550 2350 9550 2550
+$Comp
+L device:R R?
+U 1 1 5B9AB3E4
+P 9650 1800
+F 0 "R?" H 9720 1846 50  0000 L CNN
+F 1 "10K" H 9720 1755 50  0000 L CNN
+F 2 "" V 9580 1800 50  0001 C CNN
+F 3 "" H 9650 1800 50  0001 C CNN
+	1    9650 1800
+	1    0    0    -1
+$EndComp
+Wire Wire Line
+	9650 1950 9650 2350
+Text HLabel 9650 1400 1    60   Input ~ 0
+3V3_VDD
+Connection ~ 9650 2350
+Wire Wire Line
+	9650 2350 9550 2350
+Wire Wire Line
+	9650 2350 10000 2350
+Wire Wire Line
+	9550 2350 9150 2350
+Connection ~ 9550 2350
+Text Label 9200 2350 0    60   ~ 0
+RESET
+Wire Wire Line
+	10000 2350 10000 2700
+Wire Wire Line
+	9650 1400 9650 1650
+$Comp
+L device:CP1 C?
+U 1 1 5B9B405E
+P 4700 4950
+F 0 "C?" H 4815 4996 50  0000 L CNN
+F 1 "100nF" H 4815 4905 50  0000 L CNN
+F 2 "" H 4700 4950 50  0001 C CNN
+F 3 "" H 4700 4950 50  0001 C CNN
+	1    4700 4950
+	1    0    0    -1
+$EndComp
+$Comp
+L device:CP1 C?
+U 1 1 5B9B414A
+P 5100 4950
+F 0 "C?" H 5215 4996 50  0000 L CNN
+F 1 "100nF" H 5215 4905 50  0000 L CNN
+F 2 "" H 5100 4950 50  0001 C CNN
+F 3 "" H 5100 4950 50  0001 C CNN
+	1    5100 4950
+	1    0    0    -1
+$EndComp
+Wire Wire Line
+	4700 4800 4700 4550
+Wire Wire Line
+	5100 4800 5100 4450
+Wire Wire Line
+	4650 4450 5100 4450
+$Comp
+L device:LED D?
+U 1 1 5B9BB014
+P 9800 4300
+F 0 "D?" V 9838 4182 50  0000 R CNN
+F 1 "LED_PROBE" V 9747 4182 50  0000 R CNN
+F 2 "" H 9800 4300 50  0001 C CNN
+F 3 "" H 9800 4300 50  0001 C CNN
+	1    9800 4300
+	0    -1   -1   0
+$EndComp
+$Comp
+L device:R R?
+U 1 1 5B9BB11B
+P 9800 3900
+F 0 "R?" H 9870 3946 50  0000 L CNN
+F 1 "1K" H 9870 3855 50  0000 L CNN
+F 2 "" V 9730 3900 50  0001 C CNN
+F 3 "" H 9800 3900 50  0001 C CNN
+	1    9800 3900
+	1    0    0    -1
+$EndComp
+Wire Wire Line
+	9800 4150 9800 4050
+Wire Wire Line
+	9800 4450 9800 4600
+$Comp
+L power:GND #PWR?
+U 1 1 5B9BC1D8
+P 9800 4600
+F 0 "#PWR?" H 9800 4350 50  0001 C CNN
+F 1 "GND" H 9805 4427 50  0000 C CNN
+F 2 "" H 9800 4600 50  0001 C CNN
+F 3 "" H 9800 4600 50  0001 C CNN
+	1    9800 4600
+	1    0    0    -1
+$EndComp
+Wire Wire Line
+	9800 3750 9800 3650
+Wire Wire Line
+	9800 3650 9500 3650
+Text Label 9550 3650 0    60   ~ 0
+PROBE
+Wire Wire Line
+	1850 2750 2250 2750
+Text Label 1950 2750 0    60   ~ 0
+PROBE
 $EndSCHEMATC

Commit message: anotaciones
Other:
- note added: "ONION OMEGA-2"
- note added: "PROBE LED"
- note added: "RESET BUTTON"
Changed lines of the file:
@@
 EESchema Schematic File Version 4
+LIBS:power
+LIBS:74xx
 LIBS:stm32f446zetx
+LIBS:design_emb-cache
 EELAYER 26 0
 EELAYER END
@@
 Text Label 1950 2750 0    60   ~ 0
 PROBE
+Text Notes 9550 4550 1    79   ~ 0
+PROBE LED
+Text Notes 9300 2100 1    79   ~ 0
+RESET BUTTON
+Text Notes 600  850  0    197  ~ 39
+ONION OMEGA-2
 $EndSCHEMATC

Commit message: design_emb.sch
Connections:
- net labels added: OMEGA_SPI[3...0], RST, SPI_SCLK, SPI_SS
- net labels removed: SPI_CLK, SPI_CS
- wire segments 51 -> 52
Changed lines of the file:
@@
 EESchema Schematic File Version 4
-LIBS:power
-LIBS:74xx
 LIBS:stm32f446zetx
 LIBS:design_emb-cache
@@
 Text HLabel 4650 2650 2    60   Input ~ 0
 V3.3OUT
-Text HLabel 2150 3750 0    60   BiDi ~ 0
-SPI_MISO
-Text HLabel 2150 3650 0    60   BiDi ~ 0
-SPI_MOSI
-Wire Wire Line
-	2150 3750 2250 3750
-Wire Wire Line
-	2150 3650 2250 3650
 $Comp
 L power:GND #PWR?
@@
 Wire Wire Line
 	4650 4550 4700 4550
-Text HLabel 2150 3450 0    60   BiDi ~ 0
-SPI_CS
-Wire Wire Line
-	2150 3450 2250 3450
-Text HLabel 2150 3550 0    60   BiDi ~ 0
-SPI_CLK
-Wire Wire Line
-	2150 3550 2250 3550
 Text HLabel 4650 3150 2    60   Output ~ 0
 SERIAL_TX
@@
 Text Notes 600  850  0    197  ~ 39
 ONION OMEGA-2
+Wire Wire Line
+	2250 3050 1700 3050
+Text Label 1800 3050 0    60   ~ 0
+RST
+Wire Wire Line
+	1750 3450 2250 3450
+Wire Wire Line
+	1750 3550 2250 3550
+Wire Wire Line
+	1750 3650 2250 3650
+Wire Wire Line
+	1750 3750 2250 3750
+Text Label 1800 3450 0    60   ~ 0
+SPI_SS
+Text Label 1800 3550 0    60   ~ 0
+SPI_SCLK
+Text Label 1800 3650 0    60   ~ 0
+SPI_MOSI
+Text Label 1800 3750 0    60   ~ 0
+SPI_MISO
+Entry Wire Line
+	1650 3350 1750 3450
+Entry Wire Line
+	1650 3450 1750 3550
+Entry Wire Line
+	1650 3550 1750 3650
+Entry Wire Line
+	1650 3650 1750 3750
+Wire Bus Line
+	1650 3250 1500 3250
+Wire Bus Line
+	1650 3250 1650 3750
+Text HLabel 1500 3250 0    60   BiDi ~ 0
+OMEGA_SPI[3...0]
 $EndSCHEMATC

Commit message: footprints resistencias y condensadores
Parts:
- C? (x6): footprint (none) -> Capacitors_Tantalum_SMD:CP_Tantalum_Case-A_EIA-3216-18_Hand
- D?: footprint (none) -> LEDs:LED_0603_HandSoldering
- L?: footprint (none) -> Inductors_SMD:L_0805_HandSoldering
- R?: value 10K -> 10k; footprint (none) -> Resistors_SMD:R_0603_HandSoldering
- R?: value 1K -> 1k; footprint (none) -> Resistors_SMD:R_0603_HandSoldering
Changed lines of the file:
@@
 EESchema Schematic File Version 4
+LIBS:power
+LIBS:74xx
 LIBS:stm32f446zetx
 LIBS:design_emb-cache
@@
 F 0 "C?" H 5665 2846 50  0000 L CNN
 F 1 "100nF" H 5665 2755 50  0000 L CNN
-F 2 "" H 5550 2800 50  0001 C CNN
+F 2 "Capacitors_Tantalum_SMD:CP_Tantalum_Case-A_EIA-3216-18_Hand" H 5550 2800 50  0001 C CNN
 F 3 "" H 5550 2800 50  0001 C CNN
 	1    5550 2800
@@
 F 0 "L?" H 7753 4246 50  0000 L CNN
 F 1 "L" H 7753 4155 50  0000 L CNN
-F 2 "" H 7700 4200 50  0001 C CNN
+F 2 "Inductors_SMD:L_0805_HandSoldering" H 7700 4200 50  0001 C CNN
 F 3 "" H 7700 4200 50  0001 C CNN
 	1    7700 4200
@@
 F 0 "C?" H 7115 4846 50  0000 L CNN
 F 1 "0.1uF" H 7115 4755 50  0000 L CNN
-F 2 "" H 7000 4800 50  0001 C CNN
+F 2 "Capacitors_Tantalum_SMD:CP_Tantalum_Case-A_EIA-3216-18_Hand" H 7000 4800 50  0001 C CNN
 F 3 "" H 7000 4800 50  0001 C CNN
 	1    7000 4800
@@
 F 0 "C?" H 6715 4846 50  0000 L CNN
 F 1 "33uF" H 6715 4755 50  0000 L CNN
-F 2 "" H 6600 4800 50  0001 C CNN
+F 2 "Capacitors_Tantalum_SMD:CP_Tantalum_Case-A_EIA-3216-18_Hand" H 6600 4800 50  0001 C CNN
 F 3 "" H 6600 4800 50  0001 C CNN
 	1    6600 4800
@@
 F 0 "C?" H 9665 2746 50  0000 L CNN
 F 1 "100nF" H 9665 2655 50  0000 L CNN
-F 2 "" H 9550 2700 50  0001 C CNN
+F 2 "Capacitors_Tantalum_SMD:CP_Tantalum_Case-A_EIA-3216-18_Hand" H 9550 2700 50  0001 C CNN
 F 3 "" H 9550 2700 50  0001 C CNN
 	1    9550 2700
@@
 P 9650 1800
 F 0 "R?" H 9720 1846 50  0000 L CNN
-F 1 "10K" H 9720 1755 50  0000 L CNN
-F 2 "" V 9580 1800 50  0001 C CNN
+F 1 "10k" H 9720 1755 50  0000 L CNN
+F 2 "Resistors_SMD:R_0603_HandSoldering" V 9580 1800 50  0001 C CNN
 F 3 "" H 9650 1800 50  0001 C CNN
 	1    9650 1800
@@
 F 0 "C?" H 4815 4996 50  0000 L CNN
 F 1 "100nF" H 4815 4905 50  0000 L CNN
-F 2 "" H 4700 4950 50  0001 C CNN
+F 2 "Capacitors_Tantalum_SMD:CP_Tantalum_Case-A_EIA-3216-18_Hand" H 4700 4950 50  0001 C CNN
 F 3 "" H 4700 4950 50  0001 C CNN
 	1    4700 4950
@@
 F 0 "C?" H 5215 4996 50  0000 L CNN
 F 1 "100nF" H 5215 4905 50  0000 L CNN
-F 2 "" H 5100 4950 50  0001 C CNN
+F 2 "Capacitors_Tantalum_SMD:CP_Tantalum_Case-A_EIA-3216-18_Hand" H 5100 4950 50  0001 C CNN
 F 3 "" H 5100 4950 50  0001 C CNN
 	1    5100 4950
@@
 F 0 "D?" V 9838 4182 50  0000 R CNN
 F 1 "LED_PROBE" V 9747 4182 50  0000 R CNN
-F 2 "" H 9800 4300 50  0001 C CNN
+F 2 "LEDs:LED_0603_HandSoldering" H 9800 4300 50  0001 C CNN
 F 3 "" H 9800 4300 50  0001 C CNN
 	1    9800 4300
@@
 P 9800 3900
 F 0 "R?" H 9870 3946 50  0000 L CNN
-F 1 "1K" H 9870 3855 50  0000 L CNN
-F 2 "" V 9730 3900 50  0001 C CNN
+F 1 "1k" H 9870 3855 50  0000 L CNN
+F 2 "Resistors_SMD:R_0603_HandSoldering" V 9730 3900 50  0001 C CNN
 F 3 "" H 9800 3900 50  0001 C CNN
 	1    9800 3900
@@
 Wire Bus Line
 	1650 3250 1500 3250
+Text HLabel 1500 3250 0    60   BiDi ~ 0
+OMEGA_SPI[3...0]
 Wire Bus Line
 	1650 3250 1650 3750
-Text HLabel 1500 3250 0    60   BiDi ~ 0
-OMEGA_SPI[3...0]
 $EndSCHEMATC
