File: kicad/OMEGA2sch.sch (KiCad schematic (older format))
At the start: 16 parts

Commit message: footprints y JTAG
Parts:
- D5: renamed from D?; footprint (none) -> Diodes_SMD:D_SOD-123
- U9: renamed from U?; footprint (none) -> dgk_footprints:SOT-523
- gave numbers to parts that had none: 14
Connections:
- net labels added: BOOT0, JNRST, JTAG[5...0], JTCK, JTDI, JTDO, JTMS, JTRST
- wire segments 52 -> 58
Changed lines of the file:
@@
 EESchema Schematic File Version 4
+LIBS:power
+LIBS:74xx
 LIBS:stm32f446zetx
 LIBS:design_emb-cache
@@
 $EndDescr
 $Comp
-L OMEGA2:OMEGA2 U?
+L OMEGA2:OMEGA2 U8
 U 1 1 5B86E552
 P 3450 3550
-F 0 "U?" H 3450 4817 50  0000 C CNN
+F 0 "U8" H 3450 4817 50  0000 C CNN
 F 1 "OMEGA2" H 3450 4726 50  0000 C CNN
 F 2 "XCVR_OMEGA2" H 3450 3550 50  0001 L BNN
@@
 V3.3OUT
 $Comp
-L power:GND #PWR?
+L power:GND #PWR032
 U 1 1 5B916F98
 P 5100 5100
-F 0 "#PWR?" H 5100 4850 50  0001 C CNN
+F 0 "#PWR032" H 5100 4850 50  0001 C CNN
 F 1 "GND" V 5105 4972 50  0000 R CNN
 F 2 "" H 5100 5100 50  0001 C CNN
@@
 $EndComp
 $Comp
-L power:GND #PWR?
+L power:GND #PWR031
 U 1 1 5B916FF6
 P 4700 5100
-F 0 "#PWR?" H 4700 4850 50  0001 C CNN
+F 0 "#PWR031" H 4700 4850 50  0001 C CNN
 F 1 "GND" V 4705 4972 50  0000 R CNN
 F 2 "" H 4700 5100 50  0001 C CNN
@@
 	4650 2550 5550 2550
 $Comp
-L device:CP1 C?
+L device:CP1 C48
 U 1 1 5B9A6A14
 P 5550 2800
-F 0 "C?" H 5665 2846 50  0000 L CNN
+F 0 "C48" H 5665 2846 50  0000 L CNN
 F 1 "100nF" H 5665 2755 50  0000 L CNN
 F 2 "Capacitors_Tantalum_SMD:CP_Tantalum_Case-A_EIA-3216-18_Hand" H 5550 2800 50  0001 C CNN
@@
 	5550 2550 5850 2550
 $Comp
-L power:GND #PWR?
+L power:GND #PWR033
 U 1 1 5B9A6AE7
 P 5550 2950
-F 0 "#PWR?" H 5550 2700 50  0001 C CNN
+F 0 "#PWR033" H 5550 2700 50  0001 C CNN
 F 1 "GND" H 5555 2777 50  0000 C CNN
 F 2 "" H 5550 2950 50  0001 C CNN
@@
 USB-
 $Comp
-L conn:USB_A J?
+L conn:USB_A J3
 U 1 1 5B997DEA
 P 7600 3650
-F 0 "J?" H 7370 3641 50  0000 R CNN
+F 0 "J3" H 7370 3641 50  0000 R CNN
 F 1 "USB_A" H 7370 3550 50  0000 R CNN
 F 2 "" H 7750 3600 50  0001 C CNN
@@
 $EndComp
 $Comp
-L SFR2012:SRF2012-900YA LSRF?
+L SFR2012:SRF2012-900YA LSRF1
 U 1 1 5B998611
 P 6300 3700
-F 0 "LSRF?" H 6300 4039 60  0000 C CNN
+F 0 "LSRF1" H 6300 4039 60  0000 C CNN
 F 1 "SRF2012-900YA" H 6300 3933 60  0000 C CNN
 F 2 "IND_BOURNS_SRF2012A" H 6275 3465 60  0001 C CNN
@@
 	4650 3750 6000 3750
 $Comp
-L rclamp0502b:RCLAMP0502B U?
+L rclamp0502b:RCLAMP0502B U9
 U 1 1 5B998CC3
 P 7100 2500
-F 0 "U?" H 6573 2872 60  0000 R CNN
+F 0 "U9" H 6573 2872 60  0000 R CNN
 F 1 "RCLAMP0502B" H 6573 2978 60  0000 R CNN
-F 2 "" H 7100 2500 60  0001 C CNN
+F 2 "dgk_footprints:SOT-523" H 7100 2500 60  0001 C CNN
 F 3 "" H 7100 2500 60  0001 C CNN
 	1    7100 2500
@@
 $EndComp
 $Comp
-L power:GND #PWR?
+L power:GND #PWR035
 U 1 1 5B9992E0
 P 6600 5000
-F 0 "#PWR?" H 6600 4750 50  0001 C CNN
+F 0 "#PWR035" H 6600 4750 50  0001 C CNN
 F 1 "GND" H 6605 4827 50  0000 C CNN
 F 2 "" H 6600 5000 50  0001 C CNN
@@
 $EndComp
 $Comp
-L device:L L?
+L device:L L3
 U 1 1 5B999333
 P 7700 4200
-F 0 "L?" H 7753 4246 50  0000 L CNN
+F 0 "L3" H 7753 4246 50  0000 L CNN
 F 1 "L" H 7753 4155 50  0000 L CNN
 F 2 "Inductors_SMD:L_0805_HandSoldering" H 7700 4200 50  0001 C CNN
@@
 	7600 4050 7600 4350
 $Comp
-L power:GND #PWR?
+L power:GND #PWR037
 U 1 1 5B999501
 P 7600 4450
-F 0 "#PWR?" H 7600 4200 50  0001 C CNN
+F 0 "#PWR037" H 7600 4200 50  0001 C CNN
 F 1 "GND" H 7605 4277 50  0000 C CNN
 F 2 "" H 7600 4450 50  0001 C CNN
@@
 	6900 3750 7300 3750
 $Comp
-L power:GND #PWR?
+L power:GND #PWR036
 U 1 1 5B99A0B4
 P 6800 2350
-F 0 "#PWR?" H 6800 2100 50  0001 C CNN
+F 0 "#PWR036" H 6800 2100 50  0001 C CNN
 F 1 "GND" H 6805 2177 50  0000 C CNN
 F 2 "" H 6800 2350 50  0001 C CNN
@@
 $EndComp
 $Comp
-L device:CP1 C?
+L device:CP1 C50
 U 1 1 5B99A930
 P 7000 4800
-F 0 "C?" H 7115 4846 50  0000 L CNN
+F 0 "C50" H 7115 4846 50  0000 L CNN
 F 1 "0.1uF" H 7115 4755 50  0000 L CNN
 F 2 "Capacitors_Tantalum_SMD:CP_Tantalum_Case-A_EIA-3216-18_Hand" H 7000 4800 50  0001 C CNN
@@
 $EndComp
 $Comp
-L device:CP1 C?
+L device:CP1 C49
 U 1 1 5B99A976
 P 6600 4800
-F 0 "C?" H 6715 4846 50  0000 L CNN
+F 0 "C49" H 6715 4846 50  0000 L CNN
 F 1 "33uF" H 6715 4755 50  0000 L CNN
 F 2 "Capacitors_Tantalum_SMD:CP_Tantalum_Case-A_EIA-3216-18_Hand" H 6600 4800 50  0001 C CNN
@@
 	6600 4500 7000 4500
 $Comp
-L device:D_Schottky D?
+L device:D_Schottky D5
 U 1 1 5B99B7D5
 P 6150 4800
-F 0 "D?" V 6104 4721 50  0000 R CNN
+F 0 "D5" V 6104 4721 50  0000 R CNN
 F 1 "D_Scho" V 6195 4721 50  0000 R CNN
-F 2 "" H 6150 4800 50  0001 C CNN
+F 2 "Diodes_SMD:D_SOD-123" H 6150 4800 50  0001 C CNN
 F 3 "" H 6150 4800 50  0001 C CNN
 	1    6150 4800
@@
 	7000 3450 7300 3450
 $Comp
-L power:VDD #PWR?
+L power:VDD #PWR034
 U 1 1 5B99E334
 P 6150 4250
-F 0 "#PWR?" H 6150 4100 50  0001 C CNN
+F 0 "#PWR034" H 6150 4100 50  0001 C CNN
 F 1 "VDD" V 6168 4377 50  0000 L CNN
 F 2 "" H 6150 4250 50  0001 C CNN
@@
 RESET
 $Comp
-L Switch:SW_Push SW?
+L Switch:SW_Push SW3
 U 1 1 5B9A9974
 P 10000 2900
-F 0 "SW?" V 9954 3048 50  0000 L CNN
+F 0 "SW3" V 9954 3048 50  0000 L CNN
 F 1 "SW_Push" V 10045 3048 50  0000 L CNN
 F 2 "" H 10000 3100 50  0001 C CNN
@@
 $EndComp
 $Comp
-L device:CP1 C?
+L device:CP1 C51
 U 1 1 5B9A9A3A
 P 9550 2700
-F 0 "C?" H 9665 2746 50  0000 L CNN
+F 0 "C51" H 9665 2746 50  0000 L CNN
 F 1 "100nF" H 9665 2655 50  0000 L CNN
 F 2 "Capacitors_Tantalum_SMD:CP_Tantalum_Case-A_EIA-3216-18_Hand" H 9550 2700 50  0001 C CNN
@@
 	10000 3150 10000 3100
 $Comp
-L power:GND #PWR?
+L power:GND #PWR038
 U 1 1 5B9A9FD7
 P 9800 3150
-F 0 "#PWR?" H 9800 2900 50  0001 C CNN
+F 0 "#PWR038" H 9800 2900 50  0001 C CNN
 F 1 "GND" H 9805 2977 50  0000 C CNN
 F 2 "" H 9800 3150 50  0001 C CNN
@@
 	9550 2350 9550 2550
 $Comp
-L device:R R?
+L device:R R7
 U 1 1 5B9AB3E4
 P 9650 1800
-F 0 "R?" H 9720 1846 50  0000 L CNN
+F 0 "R7" H 9720 1846 50  0000 L CNN
 F 1 "10k" H 9720 1755 50  0000 L CNN
 F 2 "Resistors_SMD:R_0603_HandSoldering" V 9580 1800 50  0001 C CNN
@@
 	9650 1400 9650 1650
 $Comp
-L device:CP1 C?
+L device:CP1 C46
 U 1 1 5B9B405E
 P 4700 4950
-F 0 "C?" H 4815 4996 50  0000 L CNN
+F 0 "C46" H 4815 4996 50  0000 L CNN
 F 1 "100nF" H 4815 4905 50  0000 L CNN
 F 2 "Capacitors_Tantalum_SMD:CP_Tantalum_Case-A_EIA-3216-18_Hand" H 4700 4950 50  0001 C CNN
@@
 $EndComp
 $Comp
-L device:CP1 C?
+L device:CP1 C47
 U 1 1 5B9B414A
 P 5100 4950
-F 0 "C?" H 5215 4996 50  0000 L CNN
+F 0 "C47" H 5215 4996 50  0000 L CNN
 F 1 "100nF" H 5215 4905 50  0000 L CNN
 F 2 "Capacitors_Tantalum_SMD:CP_Tantalum_Case-A_EIA-3216-18_Hand" H 5100 4950 50  0001 C CNN
@@
 	4650 4450 5100 4450
 $Comp
-L device:LED D?
+L device:LED D6
 U 1 1 5B9BB014
 P 9800 4300
-F 0 "D?" V 9838 4182 50  0000 R CNN
+F 0 "D6" V 9838 4182 50  0000 R CNN
 F 1 "LED_PROBE" V 9747 4182 50  0000 R CNN
 F 2 "LEDs:LED_0603_HandSoldering" H 9800 4300 50  0001 C CNN
@@
 $EndComp
 $Comp
-L device:R R?
+L device:R R8
 U 1 1 5B9BB11B
 P 9800 3900
-F 0 "R?" H 9870 3946 50  0000 L CNN
+F 0 "R8" H 9870 3946 50  0000 L CNN
 F 1 "1k" H 9870 3855 50  0000 L CNN
 F 2 "Resistors_SMD:R_0603_HandSoldering" V 9730 3900 50  0001 C CNN
@@
 	9800 4450 9800 4600
 $Comp
-L power:GND #PWR?
+L power:GND #PWR039
 U 1 1 5B9BC1D8
 P 9800 4600
-F 0 "#PWR?" H 9800 4350 50  0001 C CNN
+F 0 "#PWR039" H 9800 4350 50  0001 C CNN
 F 1 "GND" H 9805 4427 50  0000 C CNN
 F 2 "" H 9800 4600 50  0001 C CNN
@@
 ONION OMEGA-2
 Wire Wire Line
-	2250 3050 1700 3050
-Text Label 1800 3050 0    60   ~ 0
+	2250 3050 1850 3050
+Text Label 2000 3050 0    60   ~ 0
 RST
 Wire Wire Line
@@
 Text HLabel 1500 3250 0    60   BiDi ~ 0
 OMEGA_SPI[3...0]
+Wire Wire Line
+	2250 3950 1850 3950
+Wire Wire Line
+	2250 3250 1850 3250
+Wire Wire Line
+	2250 3150 1850 3150
+Wire Wire Line
+	2250 4250 1850 4250
+Wire Wire Line
+	2250 4050 1850 4050
+Wire Wire Line
+	2250 4150 1850 4150
+Entry Wire Line
+	1750 3050 1850 3150
+Entry Wire Line
+	1750 3150 1850 3250
+Entry Wire Line
+	1750 3850 1850 3950
+Entry Wire Line
+	1750 3950 1850 4050
+Entry Wire Line
+	1750 4050 1850 4150
+Entry Wire Line
+	1750 4150 1850 4250
+Wire Bus Line
+	1750 2900 1450 2900
 Wire Bus Line
 	1650 3250 1650 3750
+Wire Bus Line
+	1750 2900 1750 4150
+Text HLabel 1450 2900 0    60   BiDi ~ 0
+JTAG[5...0]
+Text Label 2000 3150 0    60   ~ 0
+JTCK
+Text Label 2000 3250 0    60   ~ 0
+JTMS
+Text Label 2000 3950 0    60   ~ 0
+JTDI
+Text Label 2000 4050 0    60   ~ 0
+JTDO
+Text Label 2000 4150 0    60   ~ 0
+JTRST
+Text Label 2000 4250 0    60   ~ 0
+JNRST
+Text HLabel 2250 2950 0    60   Output ~ 0
+BOOT0
 $EndSCHEMATC

Commit message: OMEGA2sch.sch
Parts:
- added J?: Conn_01x03, symbol conn:Conn_01x03
Connections:
- net labels removed: SERIAL_RX, SERIAL_TX
- wire segments 58 -> 61
Changed lines of the file:
@@
 EESchema Schematic File Version 4
-LIBS:power
-LIBS:74xx
 LIBS:stm32f446zetx
 LIBS:design_emb-cache
@@
 Wire Wire Line
 	4650 4550 4700 4550
-Text HLabel 4650 3150 2    60   Output ~ 0
-SERIAL_TX
-Text HLabel 4650 3250 2    60   Input ~ 0
-SERIAL_RX
 Text HLabel 4650 3450 2    60   Input ~ 0
 UART_RX
@@
 Wire Bus Line
 	1750 2900 1450 2900
-Wire Bus Line
-	1650 3250 1650 3750
-Wire Bus Line
-	1750 2900 1750 4150
 Text HLabel 1450 2900 0    60   BiDi ~ 0
 JTAG[5...0]
@@
 Text HLabel 2250 2950 0    60   Output ~ 0
 BOOT0
+$Comp
+L conn:Conn_01x03 J?
+U 1 1 5BAE7762
+P 5400 3250
+F 0 "J?" H 5480 3292 50  0000 L CNN
+F 1 "Conn_01x03" H 5480 3201 50  0000 L CNN
+F 2 "" H 5400 3250 50  0001 C CNN
+F 3 "~" H 5400 3250 50  0001 C CNN
+	1    5400 3250
+	1    0    0    -1
+$EndComp
+Wire Wire Line
+	4650 3150 5200 3150
+Wire Wire Line
+	4650 3250 5200 3250
+$Comp
+L power:GND #PWR?
+U 1 1 5BAEBC38
+P 5200 3450
+F 0 "#PWR?" H 5200 3200 50  0001 C CNN
+F 1 "GND" H 5450 3400 50  0000 R CNN
+F 2 "" H 5200 3450 50  0001 C CNN
+F 3 "" H 5200 3450 50  0001 C CNN
+	1    5200 3450
+	1    0    0    -1
+$EndComp
+Wire Wire Line
+	5200 3350 5200 3450
+Wire Bus Line
+	1650 3250 1650 3750
+Wire Bus Line
+	1750 2900 1750 4150
 $EndSCHEMATC

Commit message: OMEGA2sch.sch
Parts:
- removed J?: Conn_01x03, symbol conn:Conn_01x03
Connections:
- net labels added: SERIAL_RX, SERIAL_TX
- wire segments 61 -> 58
Changed lines of the file:
@@
 Text HLabel 2250 2950 0    60   Output ~ 0
 BOOT0
-$Comp
-L conn:Conn_01x03 J?
-U 1 1 5BAE7762
-P 5400 3250
-F 0 "J?" H 5480 3292 50  0000 L CNN
-F 1 "Conn_01x03" H 5480 3201 50  0000 L CNN
-F 2 "" H 5400 3250 50  0001 C CNN
-F 3 "~" H 5400 3250 50  0001 C CNN
-	1    5400 3250
-	1    0    0    -1
-$EndComp
-Wire Wire Line
-	4650 3150 5200 3150
-Wire Wire Line
-	4650 3250 5200 3250
-$Comp
-L power:GND #PWR?
-U 1 1 5BAEBC38
-P 5200 3450
-F 0 "#PWR?" H 5200 3200 50  0001 C CNN
-F 1 "GND" H 5450 3400 50  0000 R CNN
-F 2 "" H 5200 3450 50  0001 C CNN
-F 3 "" H 5200 3450 50  0001 C CNN
-	1    5200 3450
-	1    0    0    -1
-$EndComp
-Wire Wire Line
-	5200 3350 5200 3450
+Text HLabel 4650 3250 2    60   Input ~ 0
+SERIAL_RX
+Wire Bus Line
+	1750 2900 1750 4150
 Wire Bus Line
 	1650 3250 1650 3750
-Wire Bus Line
-	1750 2900 1750 4150
+Text HLabel 4650 3150 2    60   Output ~ 0
+SERIAL_TX
 $EndSCHEMATC

Commit message: corrección footprints
Parts:
- J3: footprint (none) -> Connectors:USB_A
- LSRF1: footprint IND_BOURNS_SRF2012A -> SFR2012:SRF2012-900YA
- U8: footprint XCVR_OMEGA2 -> omega2:ONION2
Changed lines of the file:
@@
 F 0 "U8" H 3450 4817 50  0000 C CNN
 F 1 "OMEGA2" H 3450 4726 50  0000 C CNN
-F 2 "XCVR_OMEGA2" H 3450 3550 50  0001 L BNN
+F 2 "omega2:ONION2" H 3450 3550 50  0001 L BNN
 F 3 "" H 3450 3550 50  0001 L BNN
 F 4 "Onion" H 3450 3550 50  0001 L BNN "Campo4"
@@
 F 0 "J3" H 7370 3641 50  0000 R CNN
 F 1 "USB_A" H 7370 3550 50  0000 R CNN
-F 2 "" H 7750 3600 50  0001 C CNN
-F 3 "" H 7750 3600 50  0001 C CNN
+F 2 "Connectors:USB_A" H 7750 3600 50  0001 C CNN
+F 3 "https://www.digikey.com/product-detail/en/on-shore-technology-inc/USB-A1HSW6/ED2989-ND/2677750" H 7750 3600 50  0001 C CNN
 	1    7600 3650
 	-1   0    0    -1
@@
 F 0 "LSRF1" H 6300 4039 60  0000 C CNN
 F 1 "SRF2012-900YA" H 6300 3933 60  0000 C CNN
-F 2 "IND_BOURNS_SRF2012A" H 6275 3465 60  0001 C CNN
+F 2 "SFR2012:SRF2012-900YA" H 6275 3465 60  0001 C CNN
 F 3 "" H 6000 3750 60  0000 C CNN
 	1    6300 3700
@@
 Text HLabel 4650 3250 2    60   Input ~ 0
 SERIAL_RX
+Text HLabel 4650 3150 2    60   Output ~ 0
+SERIAL_TX
+Wire Bus Line
+	1650 3250 1650 3750
 Wire Bus Line
 	1750 2900 1750 4150
-Wire Bus Line
-	1650 3250 1650 3750
-Text HLabel 4650 3150 2    60   Output ~ 0
-SERIAL_TX
 $EndSCHEMATC

Commit message: fp-lib-table
Parts:
- C46, C47, C48, C49, C50, C51: footprint Capacitors_Tantalum_SMD:CP_Tantalum_Case-A_EIA-3216-18_Hand -> Capacitors_SMD:C_0603_HandSoldering
Changed lines of the file:
@@
 F 0 "C48" H 5665 2846 50  0000 L CNN
 F 1 "100nF" H 5665 2755 50  0000 L CNN
-F 2 "Capacitors_Tantalum_SMD:CP_Tantalum_Case-A_EIA-3216-18_Hand" H 5550 2800 50  0001 C CNN
+F 2 "Capacitors_SMD:C_0603_HandSoldering" H 5550 2800 50  0001 C CNN
 F 3 "" H 5550 2800 50  0001 C CNN
 	1    5550 2800
@@
 F 0 "C50" H 7115 4846 50  0000 L CNN
 F 1 "0.1uF" H 7115 4755 50  0000 L CNN
-F 2 "Capacitors_Tantalum_SMD:CP_Tantalum_Case-A_EIA-3216-18_Hand" H 7000 4800 50  0001 C CNN
+F 2 "Capacitors_SMD:C_0603_HandSoldering" H 7000 4800 50  0001 C CNN
 F 3 "" H 7000 4800 50  0001 C CNN
 	1    7000 4800
@@
 F 0 "C49" H 6715 4846 50  0000 L CNN
 F 1 "33uF" H 6715 4755 50  0000 L CNN
-F 2 "Capacitors_Tantalum_SMD:CP_Tantalum_Case-A_EIA-3216-18_Hand" H 6600 4800 50  0001 C CNN
+F 2 "Capacitors_SMD:C_0603_HandSoldering" H 6600 4800 50  0001 C CNN
 F 3 "" H 6600 4800 50  0001 C CNN
 	1    6600 4800
@@
 F 0 "C51" H 9665 2746 50  0000 L CNN
 F 1 "100nF" H 9665 2655 50  0000 L CNN
-F 2 "Capacitors_Tantalum_SMD:CP_Tantalum_Case-A_EIA-3216-18_Hand" H 9550 2700 50  0001 C CNN
+F 2 "Capacitors_SMD:C_0603_HandSoldering" H 9550 2700 50  0001 C CNN
 F 3 "" H 9550 2700 50  0001 C CNN
 	1    9550 2700
@@
 F 0 "C46" H 4815 4996 50  0000 L CNN
 F 1 "100nF" H 4815 4905 50  0000 L CNN
-F 2 "Capacitors_Tantalum_SMD:CP_Tantalum_Case-A_EIA-3216-18_Hand" H 4700 4950 50  0001 C CNN
+F 2 "Capacitors_SMD:C_0603_HandSoldering" H 4700 4950 50  0001 C CNN
 F 3 "" H 4700 4950 50  0001 C CNN
 	1    4700 4950
@@
 F 0 "C47" H 5215 4996 50  0000 L CNN
 F 1 "100nF" H 5215 4905 50  0000 L CNN
-F 2 "Capacitors_Tantalum_SMD:CP_Tantalum_Case-A_EIA-3216-18_Hand" H 5100 4950 50  0001 C CNN
+F 2 "Capacitors_SMD:C_0603_HandSoldering" H 5100 4950 50  0001 C CNN
 F 3 "" H 5100 4950 50  0001 C CNN
 	1    5100 4950

Commit message: buses JTAG, FMC_AD y CTRL
Connections:
- net labels added: JTAG0, JTAG1, JTAG2, JTAG3, JTAG4, JTAG5
- wire segments 58 -> 64
Changed lines of the file:
@@
 Wire Wire Line
 	2250 4150 1850 4150
-Entry Wire Line
-	1750 3050 1850 3150
-Entry Wire Line
-	1750 3150 1850 3250
-Entry Wire Line
-	1750 3850 1850 3950
-Entry Wire Line
-	1750 3950 1850 4050
-Entry Wire Line
-	1750 4050 1850 4150
-Entry Wire Line
-	1750 4150 1850 4250
-Wire Bus Line
-	1750 2900 1450 2900
-Text HLabel 1450 2900 0    60   BiDi ~ 0
+Text HLabel 1850 5450 0    60   BiDi ~ 0
 JTAG[5...0]
 Text Label 2000 3150 0    60   ~ 0
@@
 Text HLabel 4650 3150 2    60   Output ~ 0
 SERIAL_TX
+Text Label 2800 5550 0    60   ~ 0
+JTCK
+Text Label 2800 5650 0    60   ~ 0
+JTMS
+Text Label 2800 5750 0    60   ~ 0
+JTDI
+Text Label 2800 5850 0    60   ~ 0
+JTDO
+Text Label 2800 5950 0    60   ~ 0
+JTRST
+Text Label 2800 6050 0    60   ~ 0
+JNRST
+Wire Wire Line
+	2250 5650 3050 5650
+Wire Wire Line
+	2250 5750 3050 5750
+Wire Wire Line
+	2250 6050 3050 6050
+Wire Wire Line
+	2250 5850 3050 5850
+Wire Wire Line
+	2250 5950 3050 5950
+Wire Wire Line
+	2250 5550 3050 5550
+Text Label 2350 5550 0    60   ~ 0
+JTAG0
+Text Label 2350 5650 0    60   ~ 0
+JTAG1
+Text Label 2350 5750 0    60   ~ 0
+JTAG2
+Text Label 2350 5850 0    60   ~ 0
+JTAG3
+Text Label 2350 5950 0    60   ~ 0
+JTAG4
+Text Label 2350 6050 0    60   ~ 0
+JTAG5
+Entry Wire Line
+	2150 5450 2250 5550
+Entry Wire Line
+	2150 5550 2250 5650
+Entry Wire Line
+	2150 5650 2250 5750
+Entry Wire Line
+	2150 5750 2250 5850
+Entry Wire Line
+	2150 5850 2250 5950
+Entry Wire Line
+	2150 5950 2250 6050
 Wire Bus Line
-	1650 3250 1650 3750
+	2150 5450 1850 5450
 Wire Bus Line
-	1750 2900 1750 4150
+	1650 3250 1650 3650
+Wire Bus Line
+	2150 5450 2150 5950
 $EndSCHEMATC
