File: kicad/STM32F446ZETx.sch (KiCad schematic (older format))
At the start: 29 parts

Commit message: comunicación omega2 y stm32
Parts:
- removed J?: Conn_01x03, symbol conn:Conn_01x03
- removed U? (x2): SRX.X.TCT, TO_SOT_Packages_SMD:SOT-143, symbol ESD_Protection:SRX.X.TCT
Connections:
- net labels removed: RX_OUT, TX_IN
- wire segments 154 -> 144
- no-connect marks 2 -> 0
Other:
- note removed: "SR3.3.TCT / SR2.8.TCT"
- note removed: "User serial communication\n\n"
Changed lines of the file:
@@
 EELAYER 26 0
 EELAYER END
-$Descr A0 46811 33110
+$Descr A1 33110 23386
 encoding utf-8
 Sheet 2 5
@@
 Text HLabel 16150 11450 2    60   Input ~ 0
 UART5_RX
-$Comp
-L ESD_Protection:SRX.X.TCT U?
-U 1 1 5B8D2986
-P 17300 1600
-F 0 "U?" H 17200 1400 60  0000 C CNN
-F 1 "SRX.X.TCT" H 17300 1841 60  0000 C CNN
-F 2 "TO_SOT_Packages_SMD:SOT-143" H 17300 1600 60  0001 C CNN
-F 3 "https://co.mouser.com/datasheet/2/761/sr2_8-1277654.pdf" H 17300 1600 60  0001 C CNN
-	1    17300 1600
-	1    0    0    -1
-$EndComp
-Wire Wire Line
-	17000 1500 16900 1500
-$Comp
-L power:GND #PWR0115
-U 1 1 5B8DE647
-P 16900 1500
-F 0 "#PWR0115" H 16900 1250 50  0001 C CNN
-F 1 "GND" V 16905 1372 50  0000 R CNN
-F 2 "" H 16900 1500 50  0001 C CNN
-F 3 "" H 16900 1500 50  0001 C CNN
-	1    16900 1500
-	0    1    1    0
-$EndComp
-Wire Wire Line
-	17000 1700 16850 1700
-Text HLabel 16850 1700 0    60   Input ~ 0
-UART5_TX
-$Comp
-L ESD_Protection:SRX.X.TCT U?
-U 1 1 5B8E61E7
-P 17300 2150
-F 0 "U?" H 17200 1950 60  0000 C CNN
-F 1 "SRX.X.TCT" H 17300 2391 60  0000 C CNN
-F 2 "TO_SOT_Packages_SMD:SOT-143" H 17300 2150 60  0001 C CNN
-F 3 "https://co.mouser.com/datasheet/2/761/sr2_8-1277654.pdf" H 17300 2150 60  0001 C CNN
-	1    17300 2150
-	1    0    0    -1
-$EndComp
-Wire Wire Line
-	17000 2050 16900 2050
-$Comp
-L power:GND #PWR0116
-U 1 1 5B8E61EF
-P 16900 2050
-F 0 "#PWR0116" H 16900 1800 50  0001 C CNN
-F 1 "GND" V 16905 1922 50  0000 R CNN
-F 2 "" H 16900 2050 50  0001 C CNN
-F 3 "" H 16900 2050 50  0001 C CNN
-	1    16900 2050
-	0    1    1    0
-$EndComp
-Wire Wire Line
-	17000 2250 16850 2250
-Text HLabel 16850 2250 0    60   Input ~ 0
-UART5_RX
-NoConn ~ 17600 1500
-NoConn ~ 17600 2050
-$Comp
-L conn:Conn_01x03 J?
-U 1 1 5B8F6811
-P 18600 1800
-F 0 "J?" H 18680 1842 50  0000 L CNN
-F 1 "Conn_01x03" H 18680 1751 50  0000 L CNN
-F 2 "" H 18600 1800 50  0001 C CNN
-F 3 "~" H 18600 1800 50  0001 C CNN
-	1    18600 1800
-	1    0    0    -1
-$EndComp
-Wire Wire Line
-	18400 1700 17600 1700
-Wire Wire Line
-	18400 1800 17700 1800
-Wire Wire Line
-	17700 1800 17700 2250
-Wire Wire Line
-	17700 2250 17600 2250
-Text Label 18250 1700 2    60   ~ 0
-RX_OUT
-Text Label 18200 1800 2    60   ~ 0
-TX_IN
-Wire Wire Line
-	18400 1900 18300 1900
-Wire Wire Line
-	18300 1900 18300 2100
-$Comp
-L power:GND #PWR0117
-U 1 1 5B9073E7
-P 18300 2100
-F 0 "#PWR0117" H 18300 1850 50  0001 C CNN
-F 1 "GND" H 18305 1927 50  0000 C CNN
-F 2 "" H 18300 2100 50  0001 C CNN
-F 3 "" H 18300 2100 50  0001 C CNN
-	1    18300 2100
-	1    0    0    -1
-$EndComp
-Text Notes 19550 1100 2    197  Italic 0
-User serial communication\n\n
-Text Notes 18150 2650 2    98   ~ 0
-SR3.3.TCT / SR2.8.TCT
 Wire Wire Line
 	15650 10950 16150 10950

Commit message: leds de prueba
Parts:
- added D?: LED_PRB, symbol device:LED
- added R? (x2): 10K, symbol device:R
- added R?: 1K, symbol device:R
Connections:
- net labels added: NRST, PROBE
- wire segments 144 -> 154
Changed lines of the file:
@@
 EELAYER 26 0
 EELAYER END
-$Descr A1 33110 23386
+$Descr A2 23386 16535
 encoding utf-8
 Sheet 2 5
@@
 Text HLabel 5900 6450 0    60   Input ~ 0
 BOOT0
-Wire Notes Line style dash_dot
-	600  16850 19850 16850
 Wire Wire Line
 	15650 8050 16400 8050
-Text HLabel 16400 8050 2    60   Input ~ 0
-BOOT1
 Wire Wire Line
 	15650 10750 16150 10750
@@
 Text Notes 5900 14650 3    60   ~ 0
 OSC= 12MHz
-Wire Notes Line style dash_dot
-	19850 16850 19850 450
 Text HLabel 6000 6850 0    60   Output ~ 0
 Vcap1
@@
 Wire Wire Line
 	10100 1600 10200 1600
+$Comp
+L device:R R?
+U 1 1 5B9CAABB
+P 19950 7750
+F 0 "R?" H 20020 7796 50  0000 L CNN
+F 1 "10K" H 20020 7705 50  0000 L CNN
+F 2 "" V 19880 7750 50  0001 C CNN
+F 3 "" H 19950 7750 50  0001 C CNN
+	1    19950 7750
+	1    0    0    -1
+$EndComp
+$Comp
+L device:R R?
+U 1 1 5B9CABDE
+P 19950 8400
+F 0 "R?" H 20020 8446 50  0000 L CNN
+F 1 "10K" H 20020 8355 50  0000 L CNN
+F 2 "" V 19880 8400 50  0001 C CNN
+F 3 "" H 19950 8400 50  0001 C CNN
+	1    19950 8400
+	1    0    0    -1
+$EndComp
+Wire Wire Line
+	19950 7900 19950 8050
+Wire Wire Line
+	19950 8050 19500 8050
+Connection ~ 19950 8050
+Wire Wire Line
+	19950 8050 19950 8250
+Text Label 15850 8050 0    60   ~ 0
+BOOT1
+Text Label 19550 8050 0    60   ~ 0
+BOOT1
+Wire Wire Line
+	19950 7600 19950 7450
+Wire Wire Line
+	19950 8550 19950 8700
+Text HLabel 19950 7450 1    60   Input ~ 0
+VDD_3V3
+$Comp
+L power:GND #PWR?
+U 1 1 5B9EC896
+P 19950 8700
+F 0 "#PWR?" H 19950 8450 50  0001 C CNN
+F 1 "GND" H 19955 8527 50  0000 C CNN
+F 2 "" H 19950 8700 50  0001 C CNN
+F 3 "" H 19950 8700 50  0001 C CNN
+	1    19950 8700
+	1    0    0    -1
+$EndComp
+Text HLabel 6250 6150 0    60   Input ~ 0
+NRST
+$Comp
+L device:R R?
+U 1 1 5B9FB69B
+P 18900 8300
+F 0 "R?" H 18830 8254 50  0000 R CNN
+F 1 "1K" H 18830 8345 50  0000 R CNN
+F 2 "" V 18830 8300 50  0001 C CNN
+F 3 "" H 18900 8300 50  0001 C CNN
+	1    18900 8300
+	-1   0    0    1
+$EndComp
+$Comp
+L device:LED D?
+U 1 1 5B9FB7FB
+P 18900 8800
+F 0 "D?" V 18938 8683 50  0000 R CNN
+F 1 "LED_PRB" V 18847 8683 50  0000 R CNN
+F 2 "" H 18900 8800 50  0001 C CNN
+F 3 "" H 18900 8800 50  0001 C CNN
+	1    18900 8800
+	0    -1   -1   0
+$EndComp
+Wire Wire Line
+	18900 8450 18900 8650
+Wire Wire Line
+	18900 8150 18900 8000
+Wire Wire Line
+	18900 8950 18900 9100
+Wire Wire Line
+	18900 8000 18500 8000
+Text Label 18550 8000 0    60   ~ 0
+PROBE
+$Comp
+L power:GND #PWR?
+U 1 1 5BA23E12
+P 18900 9100
+F 0 "#PWR?" H 18900 8850 50  0001 C CNN
+F 1 "GND" H 18905 8927 50  0000 C CNN
+F 2 "" H 18900 9100 50  0001 C CNN
+F 3 "" H 18900 9100 50  0001 C CNN
+	1    18900 9100
+	1    0    0    -1
+$EndComp
+Wire Wire Line
+	15650 7950 16400 7950
 Wire Wire Line
 	15650 12350 16500 12350
@@
 Wire Bus Line
 	5550 11850 5550 12650
+Text Label 15850 7950 0    60   ~ 0
+PROBE
 $EndSCHEMATC

Commit message: anotaciones
Other:
- note added: "BOOT SELECT"
- note added: "PROBE LED"
- note added: "STM32F446ZETx"

Commit message: design_emb.sch
Connections:
- net labels added: Cont[5...0]
- net labels removed: FMC_WAIT
Changed lines of the file:
@@
 EESchema Schematic File Version 4
-LIBS:power
-LIBS:74xx
 LIBS:stm32f446zetx
 LIBS:design_emb-cache
@@
 Text Label 15700 12250 0    60   ~ 0
 FMC_DA15
-Wire Wire Line
-	15650 11550 16150 11550
-Text HLabel 16150 11550 2    60   Input ~ 0
-FMC_CLK
 Text Label 15700 11550 0    60   ~ 0
 FMC_CLK
-Wire Wire Line
-	15650 11650 16150 11650
-Text HLabel 16150 11650 2    60   Input ~ 0
-FMC_NOE
 Text Label 15700 11650 0    60   ~ 0
 FMC_NOE
-Wire Wire Line
-	15650 11750 16150 11750
-Text HLabel 16150 11750 2    60   Input ~ 0
-FMC_NWE
 Text Label 15700 11750 0    60   ~ 0
 FMC_NWE
-Wire Wire Line
-	15650 11850 16150 11850
-Text HLabel 16150 11850 2    60   Input ~ 0
-FMC_WAIT
 Text Label 15700 11850 0    60   ~ 0
 FMC_NWAIT
-Wire Wire Line
-	15650 11950 16150 11950
 Text Label 15700 11950 0    60   ~ 0
-FMC_NE1
-Text HLabel 16150 11950 2    60   Input ~ 0
 FMC_NE1
 Wire Wire Line
@@
 Text Notes 700  1050 0    197  ~ 39
 STM32F446ZETx
+Text Notes 20850 7750 3    79   ~ 0
+BOOT SELECT
+Text Notes 18650 8900 1    79   ~ 0
+PROBE LED
+Wire Wire Line
+	15650 11550 17250 11550
+Wire Wire Line
+	15650 11650 17250 11650
+Wire Wire Line
+	15650 11750 17250 11750
+Wire Wire Line
+	15650 11850 17250 11850
+Wire Wire Line
+	15650 11950 17250 11950
+Entry Wire Line
+	17250 11550 17350 11650
+Entry Wire Line
+	17250 11650 17350 11750
+Entry Wire Line
+	17250 11750 17350 11850
+Entry Wire Line
+	17250 11850 17350 11950
+Entry Wire Line
+	17250 11950 17350 12050
+Wire Bus Line
+	17350 11450 17550 11450
+Text HLabel 17550 11450 2    60   Input ~ 0
+Cont[5...0]
+Wire Bus Line
+	16600 12450 16600 12650
 Wire Wire Line
 	15650 12350 16500 12350
 Wire Bus Line
-	16600 12450 16600 12650
+	17350 11450 17350 12050
 Wire Bus Line
 	16400 11350 16400 12850
@@
 Wire Bus Line
 	5550 11850 5550 12650
-Text Notes 20850 7750 3    79   ~ 0
-BOOT SELECT
-Text Notes 18650 8900 1    79   ~ 0
-PROBE LED
 $EndSCHEMATC

Commit message: footprints resistencias y condensadores
Parts:
- C? (x15): footprint (none) -> Capacitors_Tantalum_SMD:CP_Tantalum_Case-A_EIA-3216-18_Hand
- C? (x2): renamed from 2.2uF; value CP1 -> 2.2uF; footprint (none) -> Capacitors_Tantalum_SMD:CP_Tantalum_Case-A_EIA-3216-18_Hand
- C? (x4): renamed from 22pF; value CP1 -> 22pF; footprint (none) -> Capacitors_Tantalum_SMD:CP_Tantalum_Case-A_EIA-3216-18_Hand
- D?: footprint (none) -> LEDs:LED_0603_HandSoldering
- L?: footprint (none) -> Inductors_SMD:L_0805_HandSoldering
- OSC?: renamed from 32.768kHz; value Crystal -> 32.768kHz
- OSC?: renamed from 16MHz; value Crystal -> 16MHz
- R? (x2): value 10K -> 10k; footprint (none) -> Resistors_SMD:R_0603_HandSoldering
- R?: value 1K -> 1k; footprint (none) -> Resistors_SMD:R_0603_HandSoldering
Changed lines of the file:
@@
 EESchema Schematic File Version 4
+LIBS:power
+LIBS:74xx
 LIBS:stm32f446zetx
 LIBS:design_emb-cache
@@
 F 0 "C?" H 9815 2946 50  0000 L CNN
 F 1 "1uF" H 9815 2855 50  0000 L CNN
-F 2 "" H 9700 2900 50  0001 C CNN
+F 2 "Capacitors_Tantalum_SMD:CP_Tantalum_Case-A_EIA-3216-18_Hand" H 9700 2900 50  0001 C CNN
 F 3 "~" H 9700 2900 50  0001 C CNN
 	1    9700 2900
@@
 OSC32_OUT
 $Comp
-L Device:Crystal 32.768kHz
+L Device:Crystal OSC?
 U 1 1 5B91A6BE
 P 4850 14650
-F 0 "32.768kHz" H 4850 14918 50  0000 C CNN
-F 1 "Crystal" H 4850 14827 50  0000 C CNN
+F 0 "OSC?" H 4850 14918 50  0000 C CNN
+F 1 "32.768kHz" H 4850 14827 50  0000 C CNN
 F 2 "" H 4850 14650 50  0001 C CNN
 F 3 "~" H 4850 14650 50  0001 C CNN
@@
 	5150 14650 5150 14300
 $Comp
-L Device:CP1 22pF
+L Device:CP1 C?
 U 1 1 5B923F54
 P 4550 14950
-F 0 "22pF" H 4665 14996 50  0000 L CNN
-F 1 "CP1" H 4665 14905 50  0000 L CNN
-F 2 "" H 4550 14950 50  0001 C CNN
+F 0 "C?" H 4665 14996 50  0000 L CNN
+F 1 "22pF" H 4665 14905 50  0000 L CNN
+F 2 "Capacitors_Tantalum_SMD:CP_Tantalum_Case-A_EIA-3216-18_Hand" H 4550 14950 50  0001 C CNN
 F 3 "~" H 4550 14950 50  0001 C CNN
 	1    4550 14950
@@
 $EndComp
 $Comp
-L Device:CP1 22pF
+L Device:CP1 C?
 U 1 1 5B923FA0
 P 5150 14950
-F 0 "22pF" H 5265 14996 50  0000 L CNN
-F 1 "CP1" H 5265 14905 50  0000 L CNN
-F 2 "" H 5150 14950 50  0001 C CNN
+F 0 "C?" H 5265 14996 50  0000 L CNN
+F 1 "22pF" H 5265 14905 50  0000 L CNN
+F 2 "Capacitors_Tantalum_SMD:CP_Tantalum_Case-A_EIA-3216-18_Hand" H 5150 14950 50  0001 C CNN
 F 3 "~" H 5150 14950 50  0001 C CNN
 	1    5150 14950
@@
 OSC32_OUT
 $Comp
-L Device:Crystal 16MHz
+L Device:Crystal OSC?
 U 1 1 5B92DDF6
 P 6350 14650
-F 0 "16MHz" H 6350 14918 50  0000 C CNN
-F 1 "Crystal" H 6350 14827 50  0000 C CNN
+F 0 "OSC?" H 6350 14918 50  0000 C CNN
+F 1 "16MHz" H 6350 14827 50  0000 C CNN
 F 2 "" H 6350 14650 50  0001 C CNN
 F 3 "~" H 6350 14650 50  0001 C CNN
@@
 	6650 14650 6650 14300
 $Comp
-L Device:CP1 22pF
+L Device:CP1 C?
 U 1 1 5B92DE01
 P 6050 14950
-F 0 "22pF" H 6165 14996 50  0000 L CNN
-F 1 "CP1" H 6165 14905 50  0000 L CNN
-F 2 "" H 6050 14950 50  0001 C CNN
+F 0 "C?" H 6165 14996 50  0000 L CNN
+F 1 "22pF" H 6165 14905 50  0000 L CNN
+F 2 "Capacitors_Tantalum_SMD:CP_Tantalum_Case-A_EIA-3216-18_Hand" H 6050 14950 50  0001 C CNN
 F 3 "~" H 6050 14950 50  0001 C CNN
 	1    6050 14950
@@
 $EndComp
 $Comp
-L Device:CP1 22pF
+L Device:CP1 C?
 U 1 1 5B92DE08
 P 6650 14950
-F 0 "22pF" H 6765 14996 50  0000 L CNN
-F 1 "CP1" H 6765 14905 50  0000 L CNN
-F 2 "" H 6650 14950 50  0001 C CNN
+F 0 "C?" H 6765 14996 50  0000 L CNN
+F 1 "22pF" H 6765 14905 50  0000 L CNN
+F 2 "Capacitors_Tantalum_SMD:CP_Tantalum_Case-A_EIA-3216-18_Hand" H 6650 14950 50  0001 C CNN
 F 3 "~" H 6650 14950 50  0001 C CNN
 	1    6650 14950
@@
 Vcap2
 $Comp
-L Device:CP1 2.2uF
+L Device:CP1 C?
 U 1 1 5B8B38D1
 P 13400 2900
-F 0 "2.2uF" H 13515 2946 50  0000 L CNN
-F 1 "CP1" H 13515 2855 50  0000 L CNN
-F 2 "" H 13400 2900 50  0001 C CNN
+F 0 "C?" H 13515 2946 50  0000 L CNN
+F 1 "2.2uF" H 13515 2855 50  0000 L CNN
+F 2 "Capacitors_Tantalum_SMD:CP_Tantalum_Case-A_EIA-3216-18_Hand" H 13400 2900 50  0001 C CNN
 F 3 "~" H 13400 2900 50  0001 C CNN
 	1    13400 2900
@@
 	13400 3250 13400 3050
 $Comp
-L Device:CP1 2.2uF
+L Device:CP1 C?
 U 1 1 5B8B3709
 P 12900 2900
-F 0 "2.2uF" H 13015 2946 50  0000 L CNN
-F 1 "CP1" H 13015 2855 50  0000 L CNN
-F 2 "" H 12900 2900 50  0001 C CNN
+F 0 "C?" H 13015 2946 50  0000 L CNN
+F 1 "2.2uF" H 13015 2855 50  0000 L CNN
+F 2 "Capacitors_Tantalum_SMD:CP_Tantalum_Case-A_EIA-3216-18_Hand" H 12900 2900 50  0001 C CNN
 F 3 "~" H 12900 2900 50  0001 C CNN
 	1    12900 2900
@@
 F 0 "C?" H 1815 2946 50  0000 L CNN
 F 1 "100nF" H 1815 2855 50  0000 L CNN
-F 2 "" H 1700 2900 50  0001 C CNN
+F 2 "Capacitors_Tantalum_SMD:CP_Tantalum_Case-A_EIA-3216-18_Hand" H 1700 2900 50  0001 C CNN
 F 3 "~" H 1700 2900 50  0001 C CNN
 	1    1700 2900
@@
 F 0 "L?" H 10400 2815 50  0000 C CNN
 F 1 "INDUCTOR" H 10400 2724 50  0000 C CNN
-F 2 "" H 10400 2600 50  0001 C CNN
+F 2 "Inductors_SMD:L_0805_HandSoldering" H 10400 2600 50  0001 C CNN
 F 3 "" H 10400 2600 50  0001 C CNN
 	1    10400 2600
@@
 F 0 "C?" H 9365 2946 50  0000 L CNN
 F 1 "100nF" H 9365 2855 50  0000 L CNN
-F 2 "" H 9250 2900 50  0001 C CNN
+F 2 "Capacitors_Tantalum_SMD:CP_Tantalum_Case-A_EIA-3216-18_Hand" H 9250 2900 50  0001 C CNN
 F 3 "~" H 9250 2900 50  0001 C CNN
 	1    9250 2900
@@
 F 0 "C?" H 2215 2946 50  0000 L CNN
 F 1 "100nF" H 2215 2855 50  0000 L CNN
-F 2 "" H 2100 2900 50  0001 C CNN
+F 2 "Capacitors_Tantalum_SMD:CP_Tantalum_Case-A_EIA-3216-18_Hand" H 2100 2900 50  0001 C CNN
 F 3 "~" H 2100 2900 50  0001 C CNN
 	1    2100 2900
@@
 F 0 "C?" H 2615 2946 50  0000 L CNN
 F 1 "100nF" H 2615 2855 50  0000 L CNN
-F 2 "" H 2500 2900 50  0001 C CNN
+F 2 "Capacitors_Tantalum_SMD:CP_Tantalum_Case-A_EIA-3216-18_Hand" H 2500 2900 50  0001 C CNN
 F 3 "~" H 2500 2900 50  0001 C CNN
 	1    2500 2900
@@
 F 0 "C?" H 3015 2946 50  0000 L CNN
 F 1 "100nF" H 3015 2855 50  0000 L CNN
-F 2 "" H 2900 2900 50  0001 C CNN
+F 2 "Capacitors_Tantalum_SMD:CP_Tantalum_Case-A_EIA-3216-18_Hand" H 2900 2900 50  0001 C CNN
 F 3 "~" H 2900 2900 50  0001 C CNN
 	1    2900 2900
@@
 F 0 "C?" H 3415 2946 50  0000 L CNN
 F 1 "100nF" H 3415 2855 50  0000 L CNN
-F 2 "" H 3300 2900 50  0001 C CNN
+F 2 "Capacitors_Tantalum_SMD:CP_Tantalum_Case-A_EIA-3216-18_Hand" H 3300 2900 50  0001 C CNN
 F 3 "~" H 3300 2900 50  0001 C CNN
 	1    3300 2900
@@
 F 0 "C?" H 3815 2946 50  0000 L CNN
 F 1 "100nF" H 3815 2855 50  0000 L CNN
-F 2 "" H 3700 2900 50  0001 C CNN
+F 2 "Capacitors_Tantalum_SMD:CP_Tantalum_Case-A_EIA-3216-18_Hand" H 3700 2900 50  0001 C CNN
 F 3 "~" H 3700 2900 50  0001 C CNN
 	1    3700 2900
@@
 F 0 "C?" H 4215 2946 50  0000 L CNN
 F 1 "100nF" H 4215 2855 50  0000 L CNN
-F 2 "" H 4100 2900 50  0001 C CNN
+F 2 "Capacitors_Tantalum_SMD:CP_Tantalum_Case-A_EIA-3216-18_Hand" H 4100 2900 50  0001 C CNN
 F 3 "~" H 4100 2900 50  0001 C CNN
 	1    4100 2900
@@
 F 0 "C?" H 4615 2946 50  0000 L CNN
 F 1 "100nF" H 4615 2855 50  0000 L CNN
-F 2 "" H 4500 2900 50  0001 C CNN
+F 2 "Capacitors_Tantalum_SMD:CP_Tantalum_Case-A_EIA-3216-18_Hand" H 4500 2900 50  0001 C CNN
 F 3 "~" H 4500 2900 50  0001 C CNN
 	1    4500 2900
@@
 F 0 "C?" H 5015 2946 50  0000 L CNN
 F 1 "100nF" H 5015 2855 50  0000 L CNN
-F 2 "" H 4900 2900 50  0001 C CNN
+F 2 "Capacitors_Tantalum_SMD:CP_Tantalum_Case-A_EIA-3216-18_Hand" H 4900 2900 50  0001 C CNN
 F 3 "~" H 4900 2900 50  0001 C CNN
 	1    4900 2900
@@
 F 0 "C?" H 5415 2946 50  0000 L CNN
 F 1 "100nF" H 5415 2855 50  0000 L CNN
-F 2 "" H 5300 2900 50  0001 C CNN
+F 2 "Capacitors_Tantalum_SMD:CP_Tantalum_Case-A_EIA-3216-18_Hand" H 5300 2900 50  0001 C CNN
 F 3 "~" H 5300 2900 50  0001 C CNN
 	1    5300 2900
@@
 F 0 "C?" H 5815 2946 50  0000 L CNN
 F 1 "100nF" H 5815 2855 50  0000 L CNN
-F 2 "" H 5700 2900 50  0001 C CNN
+F 2 "Capacitors_Tantalum_SMD:CP_Tantalum_Case-A_EIA-3216-18_Hand" H 5700 2900 50  0001 C CNN
 F 3 "~" H 5700 2900 50  0001 C CNN
 	1    5700 2900
@@
 F 0 "C?" H 6215 2946 50  0000 L CNN
 F 1 "100nF" H 6215 2855 50  0000 L CNN
-F 2 "" H 6100 2900 50  0001 C CNN
+F 2 "Capacitors_Tantalum_SMD:CP_Tantalum_Case-A_EIA-3216-18_Hand" H 6100 2900 50  0001 C CNN
 F 3 "~" H 6100 2900 50  0001 C CNN
 	1    6100 2900
@@
 F 0 "C?" H 6615 2946 50  0000 L CNN
 F 1 "4.7uF" H 6615 2855 50  0000 L CNN
-F 2 "" H 6500 2900 50  0001 C CNN
+F 2 "Capacitors_Tantalum_SMD:CP_Tantalum_Case-A_EIA-3216-18_Hand" H 6500 2900 50  0001 C CNN
 F 3 "~" H 6500 2900 50  0001 C CNN
 	1    6500 2900
@@
 P 20400 7750
 F 0 "R?" H 20470 7796 50  0000 L CNN
-F 1 "10K" H 20470 7705 50  0000 L CNN
-F 2 "" V 20330 7750 50  0001 C CNN
+F 1 "10k" H 20470 7705 50  0000 L CNN
+F 2 "Resistors_SMD:R_0603_HandSoldering" V 20330 7750 50  0001 C CNN
 F 3 "" H 20400 7750 50  0001 C CNN
 	1    20400 7750
@@
 P 20400 8400
 F 0 "R?" H 20470 8446 50  0000 L CNN
-F 1 "10K" H 20470 8355 50  0000 L CNN
-F 2 "" V 20330 8400 50  0001 C CNN
+F 1 "10k" H 20470 8355 50  0000 L CNN
+F 2 "Resistors_SMD:R_0603_HandSoldering" V 20330 8400 50  0001 C CNN
 F 3 "" H 20400 8400 50  0001 C CNN
 	1    20400 8400
@@
 P 18900 8300
 F 0 "R?" H 18830 8254 50  0000 R CNN
-F 1 "1K" H 18830 8345 50  0000 R CNN
-F 2 "" V 18830 8300 50  0001 C CNN
+F 1 "1k" H 18830 8345 50  0000 R CNN
+F 2 "Resistors_SMD:R_0603_HandSoldering" V 18830 8300 50  0001 C CNN
 F 3 "" H 18900 8300 50  0001 C CNN
 	1    18900 8300
@@
 F 0 "D?" V 18938 8683 50  0000 R CNN
 F 1 "LED_PRB" V 18847 8683 50  0000 R CNN
-F 2 "" H 18900 8800 50  0001 C CNN
+F 2 "LEDs:LED_0603_HandSoldering" H 18900 8800 50  0001 C CNN
 F 3 "" H 18900 8800 50  0001 C CNN
 	1    18900 8800
