File: kicad/STM32F446ZETx.sch (KiCad schematic (older format))
At the start: 30 parts

Commit message: footprints y JTAG
Parts:
- L1: renamed from L?; footprint (none) -> Inductors_SMD:L_0805_HandSoldering
- gave numbers to parts that had none: 29
Connections:
- net labels added: JNRST, JTAG[5...0], JTCK, JTDI, JTDO, JTMS, JTRST, SPI1_MISO, SPI1_MOSI, SPI1_SCK, SPI1_SS, VCAP1, VCAP2, VREF
- net labels removed: FMC[15:0], NRST, VREF+, Vcap1, Vcap2
- wire segments 154 -> 167

Commit message: STM32F446ZETx.sch
Connections:
- net labels added: FMC_NAVD
- net labels removed: FMC_NL
- wire segments 167 -> 169
Changed lines of the file:
@@
 EESchema Schematic File Version 4
-LIBS:power
-LIBS:74xx
 LIBS:stm32f446zetx
 LIBS:design_emb-cache
@@
 Text Label 5750 11350 0    60   ~ 0
 FMC_NBL1
-Wire Wire Line
-	15650 8550 16350 8550
-Text HLabel 16350 8550 2    60   Input ~ 0
-FMC_NL
 Text Label 15800 8550 0    60   ~ 0
-FMC_NL
+FMC_NAVD
 Wire Wire Line
 	6250 8750 5700 8750
@@
 PROBE LED
 Wire Wire Line
-	15650 11550 17250 11550
-Wire Wire Line
-	15650 11650 17250 11650
-Wire Wire Line
-	15650 11750 17250 11750
-Wire Wire Line
-	15650 11850 17250 11850
-Wire Wire Line
-	15650 11950 17250 11950
-Entry Wire Line
-	17250 11550 17350 11650
-Entry Wire Line
-	17250 11650 17350 11750
-Entry Wire Line
-	17250 11750 17350 11850
-Entry Wire Line
-	17250 11850 17350 11950
-Entry Wire Line
-	17250 11950 17350 12050
+	15650 11550 17500 11550
+Wire Wire Line
+	15650 11650 17500 11650
+Wire Wire Line
+	15650 11750 17500 11750
+Wire Wire Line
+	15650 11850 17500 11850
+Wire Wire Line
+	15650 11950 17500 11950
+Entry Wire Line
+	17500 11550 17600 11650
+Entry Wire Line
+	17500 11650 17600 11750
+Entry Wire Line
+	17500 11750 17600 11850
+Entry Wire Line
+	17500 11850 17600 11950
+Entry Wire Line
+	17500 11950 17600 12050
 Wire Bus Line
-	17350 11450 17550 11450
-Text HLabel 17550 11450 2    60   Input ~ 0
+	17600 11450 17800 11450
+Text HLabel 17800 11450 2    60   Input ~ 0
 Cont[5...0]
 Wire Wire Line
@@
 Text Label 6650 14550 1    60   ~ 0
 OSC_OUT
+Entry Wire Line
+	17500 11450 17600 11550
+Wire Wire Line
+	17300 8550 17300 11450
+Wire Wire Line
+	17300 11450 17500 11450
+Wire Wire Line
+	15650 8550 17300 8550
 Wire Bus Line
 	16600 12450 16600 12650
 Wire Wire Line
 	15650 12350 16500 12350
-Wire Bus Line
-	17350 11450 17350 12050
 Wire Bus Line
 	16400 11350 16400 12850
@@
 	5600 9050 5600 11750
 Wire Bus Line
+	17600 11450 17600 12050
+Wire Bus Line
 	18200 5700 18200 6550

Commit message: STM32F446ZETx.sch
Parts:
- removed R2: 10k, Resistors_SMD:R_0603_HandSoldering, symbol device:R
- added J?: Conn_01x03, symbol conn:Conn_01x03
Connections:
- wire segments 169 -> 173
Changed lines of the file:
@@
 	10050 2600 10150 2600
-$Comp
-L device:R R2
-U 1 1 5B9CAABB
-P 20400 7750
-F 0 "R2" H 20470 7796 50  0000 L CNN
-F 1 "10k" H 20470 7705 50  0000 L CNN
-F 2 "Resistors_SMD:R_0603_HandSoldering" V 20330 7750 50  0001 C CNN
-F 3 "" H 20400 7750 50  0001 C CNN
-	1    20400 7750
-	1    0    0    -1
-$EndComp
 $Comp
 L device:R R3
@@
 	1    0    0    -1
 $EndComp
-Wire Wire Line
-	20400 7900 20400 8050
 Wire Wire Line
 	20400 8050 19950 8050
@@
 Text Notes 700  1050 0    197  ~ 39
 STM32F446ZETx
-Text Notes 20850 7750 3    79   ~ 0
+Text Notes 20850 8050 3    79   ~ 0
 BOOT SELECT
 Text Notes 18650 8900 1    79   ~ 0
@@
 Wire Wire Line
 	15650 8550 17300 8550
+Text HLabel 5950 6250 0    60   Input ~ 0
+VDD_3V3
+Wire Wire Line
+	6250 6250 5950 6250
+$Comp
+L conn:Conn_01x03 J?
+U 1 1 5BB39C3D
+P 20800 7700
+F 0 "J?" H 20880 7742 50  0000 L CNN
+F 1 "Conn_01x03" H 20880 7651 50  0000 L CNN
+F 2 "" H 20800 7700 50  0001 C CNN
+F 3 "~" H 20800 7700 50  0001 C CNN
+	1    20800 7700
+	1    0    0    -1
+$EndComp
+Wire Wire Line
+	20400 7600 20600 7600
+Wire Wire Line
+	20600 7700 20400 7700
+Wire Wire Line
+	20400 7700 20400 8050
+$Comp
+L power:GND #PWR?
+U 1 1 5BB7B71B
+P 20600 7900
+F 0 "#PWR?" H 20600 7650 50  0001 C CNN
+F 1 "GND" H 20605 7727 50  0000 C CNN
+F 2 "" H 20600 7900 50  0001 C CNN
+F 3 "" H 20600 7900 50  0001 C CNN
+	1    20600 7900
+	1    0    0    -1
+$EndComp
+Wire Wire Line
+	20600 7900 20600 7800
+Wire Wire Line
+	15650 12350 16500 12350
 Wire Bus Line
 	16600 12450 16600 12650
-Wire Wire Line
-	15650 12350 16500 12350
 Wire Bus Line
 	16400 11350 16400 12850

Commit message: boot1 jack
Parts:
- added R?: 10k, Resistors_SMD:R_0603_HandSoldering, symbol device:R
Connections:
- net labels removed: FMC_NE2
- wire segments 173 -> 171
Changed lines of the file:
@@
 EESchema Schematic File Version 4
+LIBS:power
+LIBS:74xx
 LIBS:stm32f446zetx
 LIBS:design_emb-cache
@@
 FMC_NAVD
 Wire Wire Line
-	6250 8750 5700 8750
-Text HLabel 5700 8750 0    60   Input ~ 0
-FMC_NE2
-Text Label 5750 8750 0    60   ~ 0
-FMC_NE2
-Wire Wire Line
 	10350 5550 10450 5550
 Connection ~ 10450 5550
@@
 L device:R R3
 U 1 1 5B9CABDE
-P 20400 8400
-F 0 "R3" H 20470 8446 50  0000 L CNN
-F 1 "10k" H 20470 8355 50  0000 L CNN
-F 2 "Resistors_SMD:R_0603_HandSoldering" V 20330 8400 50  0001 C CNN
-F 3 "" H 20400 8400 50  0001 C CNN
-	1    20400 8400
-	1    0    0    -1
-$EndComp
-Wire Wire Line
-	20400 8050 19950 8050
-Connection ~ 20400 8050
-Wire Wire Line
-	20400 8050 20400 8250
+P 20500 8150
+F 0 "R3" H 20570 8196 50  0000 L CNN
+F 1 "10k" H 20570 8105 50  0000 L CNN
+F 2 "Resistors_SMD:R_0603_HandSoldering" V 20430 8150 50  0001 C CNN
+F 3 "" H 20500 8150 50  0001 C CNN
+	1    20500 8150
+	1    0    0    -1
+$EndComp
+Wire Wire Line
+	20500 7800 20500 8000
 Text Label 15850 8050 0    60   ~ 0
 BOOT1
-Text Label 20000 8050 0    60   ~ 0
+Text Label 20000 7700 0    60   ~ 0
 BOOT1
 Wire Wire Line
-	20400 7600 20400 7450
-Wire Wire Line
-	20400 8550 20400 8700
-Text HLabel 20400 7450 1    60   Input ~ 0
+	20500 8300 20500 8450
+Text HLabel 20500 6950 1    60   Input ~ 0
 VDD_3V3
 $Comp
 L power:GND #PWR010
 U 1 1 5B9EC896
-P 20400 8700
-F 0 "#PWR010" H 20400 8450 50  0001 C CNN
-F 1 "GND" H 20405 8527 50  0000 C CNN
-F 2 "" H 20400 8700 50  0001 C CNN
-F 3 "" H 20400 8700 50  0001 C CNN
-	1    20400 8700
+P 20500 8450
+F 0 "#PWR010" H 20500 8200 50  0001 C CNN
+F 1 "GND" H 20505 8277 50  0000 C CNN
+F 2 "" H 20500 8450 50  0001 C CNN
+F 3 "" H 20500 8450 50  0001 C CNN
+	1    20500 8450
 	1    0    0    -1
 $EndComp
@@
 $EndComp
 Wire Wire Line
-	20400 7600 20600 7600
-Wire Wire Line
-	20600 7700 20400 7700
-Wire Wire Line
-	20400 7700 20400 8050
-$Comp
-L power:GND #PWR?
-U 1 1 5BB7B71B
-P 20600 7900
-F 0 "#PWR?" H 20600 7650 50  0001 C CNN
-F 1 "GND" H 20605 7727 50  0000 C CNN
-F 2 "" H 20600 7900 50  0001 C CNN
-F 3 "" H 20600 7900 50  0001 C CNN
-	1    20600 7900
-	1    0    0    -1
-$EndComp
-Wire Wire Line
-	20600 7900 20600 7800
+	19950 7700 20600 7700
+$Comp
+L device:R R?
+U 1 1 5BACE777
+P 20500 7300
+F 0 "R?" H 20570 7346 50  0000 L CNN
+F 1 "10k" H 20570 7255 50  0000 L CNN
+F 2 "Resistors_SMD:R_0603_HandSoldering" V 20430 7300 50  0001 C CNN
+F 3 "" H 20500 7300 50  0001 C CNN
+	1    20500 7300
+	1    0    0    -1
+$EndComp
+Wire Wire Line
+	20500 6950 20500 7150
+Wire Wire Line
+	20500 7450 20500 7600
+Wire Wire Line
+	20600 7600 20500 7600
+Wire Wire Line
+	20600 7800 20500 7800
 Wire Wire Line
 	15650 12350 16500 12350

Commit message: footprints
Parts:
- J4: renamed from J?; footprint (none) -> Connectors:PINHEAD1-3
- gave numbers to parts that had none: 1
Changed lines of the file:
@@
 	6250 6250 5950 6250
 $Comp
-L conn:Conn_01x03 J?
+L conn:Conn_01x03 J4
 U 1 1 5BB39C3D
 P 20800 7700
-F 0 "J?" H 20880 7742 50  0000 L CNN
+F 0 "J4" H 20880 7742 50  0000 L CNN
 F 1 "Conn_01x03" H 20880 7651 50  0000 L CNN
-F 2 "" H 20800 7700 50  0001 C CNN
+F 2 "Connectors:PINHEAD1-3" H 20800 7700 50  0001 C CNN
 F 3 "~" H 20800 7700 50  0001 C CNN
 	1    20800 7700
@@
 	19950 7700 20600 7700
 $Comp
-L device:R R?
+L device:R R2
 U 1 1 5BACE777
 P 20500 7300
-F 0 "R?" H 20570 7346 50  0000 L CNN
+F 0 "R2" H 20570 7346 50  0000 L CNN
 F 1 "10k" H 20570 7255 50  0000 L CNN
 F 2 "Resistors_SMD:R_0603_HandSoldering" V 20430 7300 50  0001 C CNN

Commit message: perifericos stm32
Connections:
- net labels added: OUT_REL1, OUT_REL2
- wire segments 171 -> 173
Changed lines of the file:
@@
 $Descr A2 23386 16535
 encoding utf-8
-Sheet 2 5
+Sheet 2 6
 Title ""
 Date ""
@@
 	20600 7800 20500 7800
 Wire Wire Line
+	6250 7850 5800 7850
+Wire Wire Line
+	6250 7950 5800 7950
+Wire Wire Line
 	15650 12350 16500 12350
 Wire Bus Line
@@
 Wire Bus Line
 	5550 11850 5550 12650
+Text HLabel 5800 7850 0    61   Input ~ 0
+OUT_REL1
+Text HLabel 5800 7950 0    61   Input ~ 0
+OUT_REL2
 $EndSCHEMATC

Commit message: corrección footprints
Parts:
- removed OSC1: 32.768kHz, symbol Device:Crystal
- removed OSC2: 16MHz, symbol Device:Crystal
- added J6: Conn_02x10_Counter_Clockwise, Socket_Strips:Socket_Strip_Straight_2x10_Pitch2.54mm, symbol conn:Conn_02x10_Counter_Clockwise
- added OSC1: 32.768MHz, ABMM2-32.768MHZ:ABMM2-32.768MHZ-E2F-T, symbol device:Crystal_GND24
- added OSC2: 12MHz, Crystals:Crystal_SMD_Abracon_ABM8G-4pin_3.2x2.5mm, symbol device:Crystal_GND24
- C11, C9: value 22pF -> 18pF
- C14, C17: value 22pF -> 10pF
- U3: footprint Package_QFP:LQFP-144_20x20mm_P0.5mm -> Housings_QFP:LQFP-144_20x20mm_Pitch0.5mm
Connections:
- net labels added: USR1, USR10, USR11, USR12, USR13, USR14, USR15, USR16, USR17, USR18, USR2, USR3, USR4, USR5, USR6, USR7, USR8, USR9
- net labels removed: SPI1_MISO, SPI1_MOSI, SPI1_SCK, SPI1_SS, SPI_CS, SPI_MISO, SPI_MOSI, SPI_SCK
- wire segments 173 -> 208

Commit message: fp-lib-table
Parts:
- C1, C10, C11, C12, C13, C14, C15, C16, C17, C18, C19, C2, C20, C21, C3, C4, C5, C6, C7, C8, C9: footprint Capacitors_Tantalum_SMD:CP_Tantalum_Case-A_EIA-3216-18_Hand -> Capacitors_SMD:C_0603_HandSoldering
Changed lines of the file:
@@
 F 0 "C19" H 9815 2946 50  0000 L CNN
 F 1 "1uF" H 9815 2855 50  0000 L CNN
-F 2 "Capacitors_Tantalum_SMD:CP_Tantalum_Case-A_EIA-3216-18_Hand" H 9700 2900 50  0001 C CNN
+F 2 "Capacitors_SMD:C_0603_HandSoldering" H 9700 2900 50  0001 C CNN
 F 3 "~" H 9700 2900 50  0001 C CNN
 	1    9700 2900
@@
 F 0 "C9" H 4665 14996 50  0000 L CNN
 F 1 "18pF" H 4665 14905 50  0000 L CNN
-F 2 "Capacitors_Tantalum_SMD:CP_Tantalum_Case-A_EIA-3216-18_Hand" H 4550 14950 50  0001 C CNN
+F 2 "Capacitors_SMD:C_0603_HandSoldering" H 4550 14950 50  0001 C CNN
 F 3 "~" H 4550 14950 50  0001 C CNN
 	1    4550 14950
@@
 F 0 "C11" H 5265 14996 50  0000 L CNN
 F 1 "18pF" H 5265 14905 50  0000 L CNN
-F 2 "Capacitors_Tantalum_SMD:CP_Tantalum_Case-A_EIA-3216-18_Hand" H 5150 14950 50  0001 C CNN
+F 2 "Capacitors_SMD:C_0603_HandSoldering" H 5150 14950 50  0001 C CNN
 F 3 "~" H 5150 14950 50  0001 C CNN
 	1    5150 14950
@@
 F 0 "C14" H 6165 14996 50  0000 L CNN
 F 1 "10pF" H 6165 14905 50  0000 L CNN
-F 2 "Capacitors_Tantalum_SMD:CP_Tantalum_Case-A_EIA-3216-18_Hand" H 6050 14950 50  0001 C CNN
+F 2 "Capacitors_SMD:C_0603_HandSoldering" H 6050 14950 50  0001 C CNN
 F 3 "~" H 6050 14950 50  0001 C CNN
 	1    6050 14950
@@
 F 0 "C17" H 6765 14996 50  0000 L CNN
 F 1 "10pF" H 6765 14905 50  0000 L CNN
-F 2 "Capacitors_Tantalum_SMD:CP_Tantalum_Case-A_EIA-3216-18_Hand" H 6650 14950 50  0001 C CNN
+F 2 "Capacitors_SMD:C_0603_HandSoldering" H 6650 14950 50  0001 C CNN
 F 3 "~" H 6650 14950 50  0001 C CNN
 	1    6650 14950
@@
 F 0 "C21" H 13515 2946 50  0000 L CNN
 F 1 "2.2uF" H 13515 2855 50  0000 L CNN
-F 2 "Capacitors_Tantalum_SMD:CP_Tantalum_Case-A_EIA-3216-18_Hand" H 13400 2900 50  0001 C CNN
+F 2 "Capacitors_SMD:C_0603_HandSoldering" H 13400 2900 50  0001 C CNN
 F 3 "~" H 13400 2900 50  0001 C CNN
 	1    13400 2900
@@
 F 0 "C20" H 13015 2946 50  0000 L CNN
 F 1 "2.2uF" H 13015 2855 50  0000 L CNN
-F 2 "Capacitors_Tantalum_SMD:CP_Tantalum_Case-A_EIA-3216-18_Hand" H 12900 2900 50  0001 C CNN
+F 2 "Capacitors_SMD:C_0603_HandSoldering" H 12900 2900 50  0001 C CNN
 F 3 "~" H 12900 2900 50  0001 C CNN
 	1    12900 2900
@@
 F 0 "C1" H 1815 2946 50  0000 L CNN
 F 1 "100nF" H 1815 2855 50  0000 L CNN
-F 2 "Capacitors_Tantalum_SMD:CP_Tantalum_Case-A_EIA-3216-18_Hand" H 1700 2900 50  0001 C CNN
+F 2 "Capacitors_SMD:C_0603_HandSoldering" H 1700 2900 50  0001 C CNN
 F 3 "~" H 1700 2900 50  0001 C CNN
 	1    1700 2900
@@
 F 0 "C18" H 9365 2946 50  0000 L CNN
 F 1 "100nF" H 9365 2855 50  0000 L CNN
-F 2 "Capacitors_Tantalum_SMD:CP_Tantalum_Case-A_EIA-3216-18_Hand" H 9250 2900 50  0001 C CNN
+F 2 "Capacitors_SMD:C_0603_HandSoldering" H 9250 2900 50  0001 C CNN
 F 3 "~" H 9250 2900 50  0001 C CNN
 	1    9250 2900
@@
 F 0 "C2" H 2215 2946 50  0000 L CNN
 F 1 "100nF" H 2215 2855 50  0000 L CNN
-F 2 "Capacitors_Tantalum_SMD:CP_Tantalum_Case-A_EIA-3216-18_Hand" H 2100 2900 50  0001 C CNN
+F 2 "Capacitors_SMD:C_0603_HandSoldering" H 2100 2900 50  0001 C CNN
 F 3 "~" H 2100 2900 50  0001 C CNN
 	1    2100 2900
@@
 F 0 "C3" H 2615 2946 50  0000 L CNN
 F 1 "100nF" H 2615 2855 50  0000 L CNN
-F 2 "Capacitors_Tantalum_SMD:CP_Tantalum_Case-A_EIA-3216-18_Hand" H 2500 2900 50  0001 C CNN
+F 2 "Capacitors_SMD:C_0603_HandSoldering" H 2500 2900 50  0001 C CNN
 F 3 "~" H 2500 2900 50  0001 C CNN
 	1    2500 2900
@@
 F 0 "C4" H 3015 2946 50  0000 L CNN
 F 1 "100nF" H 3015 2855 50  0000 L CNN
-F 2 "Capacitors_Tantalum_SMD:CP_Tantalum_Case-A_EIA-3216-18_Hand" H 2900 2900 50  0001 C CNN
+F 2 "Capacitors_SMD:C_0603_HandSoldering" H 2900 2900 50  0001 C CNN
 F 3 "~" H 2900 2900 50  0001 C CNN
 	1    2900 2900
@@
 F 0 "C5" H 3415 2946 50  0000 L CNN
 F 1 "100nF" H 3415 2855 50  0000 L CNN
-F 2 "Capacitors_Tantalum_SMD:CP_Tantalum_Case-A_EIA-3216-18_Hand" H 3300 2900 50  0001 C CNN
+F 2 "Capacitors_SMD:C_0603_HandSoldering" H 3300 2900 50  0001 C CNN
 F 3 "~" H 3300 2900 50  0001 C CNN
 	1    3300 2900
@@
 F 0 "C6" H 3815 2946 50  0000 L CNN
 F 1 "100nF" H 3815 2855 50  0000 L CNN
-F 2 "Capacitors_Tantalum_SMD:CP_Tantalum_Case-A_EIA-3216-18_Hand" H 3700 2900 50  0001 C CNN
+F 2 "Capacitors_SMD:C_0603_HandSoldering" H 3700 2900 50  0001 C CNN
 F 3 "~" H 3700 2900 50  0001 C CNN
 	1    3700 2900
@@
 F 0 "C7" H 4215 2946 50  0000 L CNN
 F 1 "100nF" H 4215 2855 50  0000 L CNN
-F 2 "Capacitors_Tantalum_SMD:CP_Tantalum_Case-A_EIA-3216-18_Hand" H 4100 2900 50  0001 C CNN
+F 2 "Capacitors_SMD:C_0603_HandSoldering" H 4100 2900 50  0001 C CNN
 F 3 "~" H 4100 2900 50  0001 C CNN
 	1    4100 2900
@@
 F 0 "C8" H 4615 2946 50  0000 L CNN
 F 1 "100nF" H 4615 2855 50  0000 L CNN
-F 2 "Capacitors_Tantalum_SMD:CP_Tantalum_Case-A_EIA-3216-18_Hand" H 4500 2900 50  0001 C CNN
+F 2 "Capacitors_SMD:C_0603_HandSoldering" H 4500 2900 50  0001 C CNN
 F 3 "~" H 4500 2900 50  0001 C CNN
 	1    4500 2900
@@
 F 0 "C10" H 5015 2946 50  0000 L CNN
 F 1 "100nF" H 5015 2855 50  0000 L CNN
-F 2 "Capacitors_Tantalum_SMD:CP_Tantalum_Case-A_EIA-3216-18_Hand" H 4900 2900 50  0001 C CNN
+F 2 "Capacitors_SMD:C_0603_HandSoldering" H 4900 2900 50  0001 C CNN
 F 3 "~" H 4900 2900 50  0001 C CNN
 	1    4900 2900
@@
 F 0 "C12" H 5415 2946 50  0000 L CNN
 F 1 "100nF" H 5415 2855 50  0000 L CNN
-F 2 "Capacitors_Tantalum_SMD:CP_Tantalum_Case-A_EIA-3216-18_Hand" H 5300 2900 50  0001 C CNN
+F 2 "Capacitors_SMD:C_0603_HandSoldering" H 5300 2900 50  0001 C CNN
 F 3 "~" H 5300 2900 50  0001 C CNN
 	1    5300 2900
@@
 F 0 "C13" H 5815 2946 50  0000 L CNN
 F 1 "100nF" H 5815 2855 50  0000 L CNN
-F 2 "Capacitors_Tantalum_SMD:CP_Tantalum_Case-A_EIA-3216-18_Hand" H 5700 2900 50  0001 C CNN
+F 2 "Capacitors_SMD:C_0603_HandSoldering" H 5700 2900 50  0001 C CNN
 F 3 "~" H 5700 2900 50  0001 C CNN
 	1    5700 2900
@@
 F 0 "C15" H 6215 2946 50  0000 L CNN
 F 1 "100nF" H 6215 2855 50  0000 L CNN
-F 2 "Capacitors_Tantalum_SMD:CP_Tantalum_Case-A_EIA-3216-18_Hand" H 6100 2900 50  0001 C CNN
+F 2 "Capacitors_SMD:C_0603_HandSoldering" H 6100 2900 50  0001 C CNN
 F 3 "~" H 6100 2900 50  0001 C CNN
 	1    6100 2900
@@
 F 0 "C16" H 6615 2946 50  0000 L CNN
 F 1 "4.7uF" H 6615 2855 50  0000 L CNN
-F 2 "Capacitors_Tantalum_SMD:CP_Tantalum_Case-A_EIA-3216-18_Hand" H 6500 2900 50  0001 C CNN
+F 2 "Capacitors_SMD:C_0603_HandSoldering" H 6500 2900 50  0001 C CNN
 F 3 "~" H 6500 2900 50  0001 C CNN
 	1    6500 2900
