File: kicad/STM32F446ZETx.sch (KiCad schematic (older format))
At the start: 32 parts, among them J4 Conn_01x03, J6 Conn_02x10_Counter_Clockwise, U3 STM32F446ZETx

Commit message: buses JTAG, FMC_AD y CTRL
Connections:
- net labels added: CTRL0, CTRL1, CTRL2, CTRL3, CTRL4, CTRL5, CTRL[5...0], FMCAD0, FMCAD1, FMCAD10, FMCAD11, FMCAD12, FMCAD13, FMCAD14, FMCAD15, FMCAD2, FMCAD3, FMCAD4, FMCAD5, FMCAD6, FMCAD7, FMCAD8, FMCAD9, FMCAD[15...0], JNRST_S, JTAG0, JTAG1, JTAG2, JTAG3, JTAG4, JTAG5, JTCK_S, JTDI_S, JTDO_S, JTMS_S, JTRST_S
- net labels removed: Cont[5...0], FMC_AD[15:0], JNRST, JTCK, JTDI, JTDO, JTMS, JTRST, UART5_RX
- wire segments 208 -> 224

Commit message: design_emb.bak
Connections:
- net labels added: FMCA16, FMCA17, FMCA18, FMCA[24:16], FMCNBL0, FMCNBL1, FMCNBL[1:0], FMC_A16, FMC_A17, FMC_A18, VDD3V3
- net labels removed: FMC_A[24:16], FMC_NBL[1:0]
- wire segments 224 -> 228
Changed lines of the file:
@@
 EESchema Schematic File Version 4
-LIBS:power
-LIBS:74xx
 LIBS:stm32f446zetx
 LIBS:design_emb-cache
@@
 FMC_NE1
 Wire Wire Line
-	6250 11850 5700 11850
-Wire Wire Line
-	6250 11750 5700 11750
-Entry Wire Line
-	5600 11650 5700 11750
-Wire Wire Line
-	6250 11650 5700 11650
-Entry Wire Line
-	5600 11550 5700 11650
-Wire Wire Line
-	6250 11550 5700 11550
-Entry Wire Line
-	5600 11450 5700 11550
-Wire Wire Line
-	6250 11450 5700 11450
-Entry Wire Line
-	5600 11350 5700 11450
+	6250 11750 4900 11750
+Entry Wire Line
+	4800 11650 4900 11750
+Wire Wire Line
+	6250 11650 4900 11650
+Entry Wire Line
+	4800 11550 4900 11650
+Wire Wire Line
+	6250 11550 4900 11550
+Entry Wire Line
+	4800 11450 4900 11550
+Wire Wire Line
+	6250 11450 4900 11450
+Entry Wire Line
+	4800 11350 4900 11450
 Text Label 5800 11550 0    60   ~ 0
 FMC_A19
@@
 FMC_A23
 Wire Bus Line
-	5600 9050 5300 9050
-Text HLabel 5300 9050 0    60   Input ~ 0
-FMC_A[24:16]
-Wire Wire Line
-	6250 9150 5700 9150
+	4800 9050 4550 9050
+Text HLabel 4550 9050 0    60   Input ~ 0
+FMCA[24:16]
+Wire Wire Line
+	6250 9150 4900 9150
 Text Label 5750 9150 0    60   ~ 0
 FMC_A24
-Wire Wire Line
-	6250 11350 5650 11350
-Wire Wire Line
-	6250 11250 5650 11250
-Entry Wire Line
-	5550 11150 5650 11250
-Entry Wire Line
-	5550 11250 5650 11350
+Entry Wire Line
+	4150 10850 4250 10950
+Entry Wire Line
+	4150 10950 4250 11050
 Wire Bus Line
-	5550 11250 5550 11150
+	4150 10950 4150 10850
 Wire Bus Line
-	5550 11150 5300 11150
-Text HLabel 5300 11150 0    60   Input ~ 0
-FMC_NBL[1:0]
-Wire Wire Line
-	15650 12450 16500 12450
-Wire Wire Line
-	15650 12550 16500 12550
-Entry Wire Line
-	16500 12350 16600 12450
-Entry Wire Line
-	16500 12450 16600 12550
-Entry Wire Line
-	16500 12550 16600 12650
-Wire Bus Line
-	16600 12450 16700 12450
-Text HLabel 16700 12450 2    60   Input ~ 0
-FMC_A[24:16]
+	4150 10850 3900 10850
+Text HLabel 3900 10850 0    60   Input ~ 0
+FMCNBL[1:0]
+Wire Wire Line
+	15650 12450 17050 12450
+Wire Wire Line
+	15650 12550 17050 12550
+Entry Wire Line
+	17050 12350 17150 12450
+Entry Wire Line
+	17050 12450 17150 12550
+Entry Wire Line
+	17050 12550 17150 12650
 Text Label 5750 11250 0    60   ~ 0
 FMC_NBL0
@@
 	11350 13250 11350 13500
 Entry Wire Line
-	5600 9050 5700 9150
+	4800 9050 4900 9150
 $Comp
 L power:GND #PWR0101
@@
 	1700 2600 2100 2600
 Text HLabel 1500 2600 0    60   Input ~ 0
-VDD_3V3
+VDD3V3
 Wire Wire Line
 	15650 11450 16150 11450
@@
 	1    0    0    -1
 $EndComp
-Text HLabel 9000 2600 0    60   Input ~ 0
-VDD_3V3
 Text Notes 7850 2300 0    98   ~ 0
 100nF , 1uF - Ceramic/tantalum capacitors
@@
 	20500 8300 20500 8450
 Text HLabel 20500 6950 1    60   Input ~ 0
-VDD_3V3
+VDD3V3
 $Comp
 L power:GND #PWR010
@@
 Wire Wire Line
 	21200 13000 20700 13000
-Text HLabel 19700 12100 0    60   Input ~ 0
-VDD_3V3
 $Comp
 L power:GND #PWR043
@@
 	20750 5350 21050 5350
 Wire Wire Line
-	15650 12350 16500 12350
+	15650 12350 17050 12350
 Text Label 19300 9800 0    60   ~ 0
 FMC_DA0
@@
 Entry Wire Line
 	17500 11950 17600 11850
-Text Label 20000 11300 0    60   ~ 0
+Text Label 19950 9800 0    60   ~ 0
 FMCAD0
-Text Label 20000 11200 0    60   ~ 0
+Text Label 19950 9900 0    60   ~ 0
 FMCAD1
-Text Label 20000 11100 0    60   ~ 0
+Text Label 19950 10000 0    60   ~ 0
 FMCAD2
-Text Label 20000 11000 0    60   ~ 0
+Text Label 19950 10100 0    60   ~ 0
 FMCAD3
-Text Label 20000 10900 0    60   ~ 0
+Text Label 19950 10200 0    60   ~ 0
 FMCAD4
-Text Label 20000 10800 0    60   ~ 0
+Text Label 19950 10300 0    60   ~ 0
 FMCAD5
-Text Label 20000 10700 0    60   ~ 0
+Text Label 19950 10400 0    60   ~ 0
 FMCAD6
-Text Label 20000 10600 0    60   ~ 0
+Text Label 19950 10500 0    60   ~ 0
 FMCAD7
-Text Label 20000 10500 0    60   ~ 0
+Text Label 19950 10600 0    60   ~ 0
 FMCAD8
-Text Label 20000 10400 0    60   ~ 0
+Text Label 19950 10700 0    60   ~ 0
 FMCAD9
-Text Label 20000 10300 0    60   ~ 0
+Text Label 19950 10800 0    60   ~ 0
 FMCAD10
-Text Label 20000 10200 0    60   ~ 0
+Text Label 19950 10900 0    60   ~ 0
 FMCAD11
-Text Label 20000 10100 0    60   ~ 0
+Text Label 19950 11000 0    60   ~ 0
 FMCAD12
-Text Label 20000 10000 0    60   ~ 0
+Text Label 19950 11100 0    60   ~ 0
 FMCAD13
-Text Label 20000 9900 0    60   ~ 0
+Text Label 19950 11200 0    60   ~ 0
 FMCAD14
-Text Label 20000 9800 0    60   ~ 0
+Text Label 19950 11300 0    60   ~ 0
 FMCAD15
 Wire Bus Line
-	16600 12450 16600 12650
+	17150 12450 17350 12450
+Text Label 15700 12350 0    60   ~ 0
+FMC_A16
+Text Label 15700 12450 0    60   ~ 0
+FMC_A17
+Text Label 15700 12550 0    60   ~ 0
+FMC_A18
+Text HLabel 17350 12450 2    60   Input ~ 0
+FMCA[24:16]
+Text Label 16450 12350 0    60   ~ 0
+FMCA16
+Text Label 16450 12450 0    60   ~ 0
+FMCA17
+Text Label 16450 12550 0    60   ~ 0
+FMCA18
+Wire Wire Line
+	6250 11350 5050 11350
+Wire Wire Line
+	5050 11350 5050 11050
+Wire Wire Line
+	5050 11050 4250 11050
+Wire Wire Line
+	6250 11250 5150 11250
+Wire Wire Line
+	5150 11250 5150 10950
+Wire Wire Line
+	5150 10950 4250 10950
+Text Label 5250 11250 0    60   ~ 0
+FMCNBL0
+Text Label 5250 11350 0    60   ~ 0
+FMCNBL1
+Wire Wire Line
+	4900 11850 6250 11850
+Entry Wire Line
+	4800 11750 4900 11850
+Text HLabel 9000 2600 0    60   Input ~ 0
+VDD3V3
+Text HLabel 19700 12100 0    60   Input ~ 0
+VDD3V3
+Wire Bus Line
+	17150 12450 17150 12650
+Wire Bus Line
+	20750 5350 20750 5850
 Wire Bus Line
 	17600 11350 17600 11850
 Wire Bus Line
-	20750 5350 20750 5850
-Wire Bus Line
-	5600 9050 5600 11750
+	4800 9050 4800 11850
 Wire Bus Line
 	20600 9700 20600 11200

Commit message: design_emb.sch
Connections:
- net labels added: FMCA19, FMCA20, FMCA21, FMCA22, FMCA23, FMCA24, FMCA[24...16], FMCNBL[1...0], UART4_RX, UART4_TX
- net labels removed: FMCA[24:16], FMCNBL[1:0], UART5_TX
- wire segments 228 -> 240
Changed lines of the file:
@@
 FMC_NE1
 Wire Wire Line
-	6250 11750 4900 11750
-Entry Wire Line
-	4800 11650 4900 11750
-Wire Wire Line
-	6250 11650 4900 11650
-Entry Wire Line
-	4800 11550 4900 11650
-Wire Wire Line
-	6250 11550 4900 11550
-Entry Wire Line
-	4800 11450 4900 11550
-Wire Wire Line
-	6250 11450 4900 11450
-Entry Wire Line
-	4800 11350 4900 11450
+	4500 11600 3150 11600
+Entry Wire Line
+	3050 11500 3150 11600
+Wire Wire Line
+	4500 11500 3150 11500
+Entry Wire Line
+	3050 11400 3150 11500
+Wire Wire Line
+	4500 11400 3150 11400
+Entry Wire Line
+	3050 11300 3150 11400
+Wire Wire Line
+	4500 11300 3150 11300
+Entry Wire Line
+	3050 11200 3150 11300
 Text Label 5800 11550 0    60   ~ 0
 FMC_A19
@@
 FMC_A23
 Wire Bus Line
-	4800 9050 4550 9050
-Text HLabel 4550 9050 0    60   Input ~ 0
-FMCA[24:16]
-Wire Wire Line
-	6250 9150 4900 9150
+	3050 8900 2800 8900
+Text HLabel 2800 8900 0    60   BiDi ~ 0
+FMCA[24...16]
+Wire Wire Line
+	4500 9000 3150 9000
 Text Label 5750 9150 0    60   ~ 0
 FMC_A24
 Entry Wire Line
-	4150 10850 4250 10950
-Entry Wire Line
-	4150 10950 4250 11050
+	2650 12000 2750 12100
+Entry Wire Line
+	2650 12100 2750 12200
 Wire Bus Line
-	4150 10950 4150 10850
+	2650 12100 2650 12000
 Wire Bus Line
-	4150 10850 3900 10850
-Text HLabel 3900 10850 0    60   Input ~ 0
-FMCNBL[1:0]
-Wire Wire Line
-	15650 12450 17050 12450
-Wire Wire Line
-	15650 12550 17050 12550
-Entry Wire Line
-	17050 12350 17150 12450
-Entry Wire Line
-	17050 12450 17150 12550
-Entry Wire Line
-	17050 12550 17150 12650
+	2650 12000 2400 12000
+Text HLabel 2400 12000 0    60   BiDi ~ 0
+FMCNBL[1...0]
+Wire Wire Line
+	16650 13050 18050 13050
+Wire Wire Line
+	16650 13150 18050 13150
+Entry Wire Line
+	18050 12950 18150 13050
+Entry Wire Line
+	18050 13050 18150 13150
+Entry Wire Line
+	18050 13150 18150 13250
 Text Label 5750 11250 0    60   ~ 0
 FMC_NBL0
@@
 	11350 13250 11350 13500
 Entry Wire Line
-	4800 9050 4900 9150
+	3050 8900 3150 9000
 $Comp
 L power:GND #PWR0101
@@
 	15650 8050 16400 8050
 Wire Wire Line
-	15650 10750 16150 10750
-Text HLabel 16150 10750 2    60   Output ~ 0
-UART5_TX
+	15650 10550 16150 10550
+Text HLabel 16150 10550 2    60   Output ~ 0
+UART4_TX
 Wire Wire Line
 	15650 10950 16250 10950
@@
 	20750 5350 21050 5350
 Wire Wire Line
-	15650 12350 17050 12350
+	16650 12950 18050 12950
 Text Label 19300 9800 0    60   ~ 0
 FMC_DA0
@@
 FMCAD15
 Wire Bus Line
-	17150 12450 17350 12450
+	18150 13050 18350 13050
 Text Label 15700 12350 0    60   ~ 0
 FMC_A16
@@
 Text Label 15700 12550 0    60   ~ 0
 FMC_A18
-Text HLabel 17350 12450 2    60   Input ~ 0
-FMCA[24:16]
-Text Label 16450 12350 0    60   ~ 0
+Text HLabel 18350 13050 2    60   BiDi ~ 0
+FMCA[24...16]
+Text Label 17450 12950 0    60   ~ 0
 FMCA16
-Text Label 16450 12450 0    60   ~ 0
+Text Label 17450 13050 0    60   ~ 0
 FMCA17
-Text Label 16450 12550 0    60   ~ 0
+Text Label 17450 13150 0    60   ~ 0
 FMCA18
 Wire Wire Line
-	6250 11350 5050 11350
-Wire Wire Line
-	5050 11350 5050 11050
-Wire Wire Line
-	5050 11050 4250 11050
-Wire Wire Line
-	6250 11250 5150 11250
-Wire Wire Line
-	5150 11250 5150 10950
-Wire Wire Line
-	5150 10950 4250 10950
-Text Label 5250 11250 0    60   ~ 0
+	4200 12500 3000 12500
+Wire Wire Line
+	3000 12500 3000 12200
+Wire Wire Line
+	3000 12200 2750 12200
+Wire Wire Line
+	4200 12400 3100 12400
+Wire Wire Line
+	3100 12400 3100 12100
+Wire Wire Line
+	3100 12100 2750 12100
+Text Label 3200 12400 0    60   ~ 0
 FMCNBL0
-Text Label 5250 11350 0    60   ~ 0
+Text Label 3200 12500 0    60   ~ 0
 FMCNBL1
 Wire Wire Line
-	4900 11850 6250 11850
-Entry Wire Line
-	4800 11750 4900 11850
+	3150 11700 4500 11700
+Entry Wire Line
+	3050 11600 3150 11700
 Text HLabel 9000 2600 0    60   Input ~ 0
 VDD3V3
 Text HLabel 19700 12100 0    60   Input ~ 0
 VDD3V3
+Text Label 4200 12400 0    60   ~ 0
+FMC_NBL0
+Text Label 4200 12500 0    60   ~ 0
+FMC_NBL1
+Wire Wire Line
+	6250 11350 5050 11350
+Wire Wire Line
+	6250 11250 5150 11250
+Text Label 4050 11400 0    60   ~ 0
+FMC_A19
+Text Label 4050 11500 0    60   ~ 0
+FMC_A20
+Text Label 4050 11600 0    60   ~ 0
+FMC_A21
+Text Label 4050 11700 0    60   ~ 0
+FMC_A22
+Text Label 4050 11300 0    60   ~ 0
+FMC_A23
+Text Label 4000 9000 0    60   ~ 0
+FMC_A24
+Text Label 3350 9000 0    60   ~ 0
+FMCA24
+Text Label 3350 11300 0    60   ~ 0
+FMCA23
+Text Label 3350 11400 0    60   ~ 0
+FMCA19
+Text Label 3350 11500 0    60   ~ 0
+FMCA20
+Text Label 3350 11600 0    60   ~ 0
+FMCA21
+Text Label 3350 11700 0    60   ~ 0
+FMCA22
+Wire Wire Line
+	6250 11750 4900 11750
+Wire Wire Line
+	6250 11650 4900 11650
+Wire Wire Line
+	6250 11550 4900 11550
+Wire Wire Line
+	6250 11450 4900 11450
+Wire Wire Line
+	4900 11850 6250 11850
+Wire Wire Line
+	6250 9150 4900 9150
+Text Label 16650 12950 0    60   ~ 0
+FMC_A16
+Text Label 16650 13050 0    60   ~ 0
+FMC_A17
+Text Label 16650 13150 0    60   ~ 0
+FMC_A18
+Wire Wire Line
+	15650 12450 17050 12450
+Wire Wire Line
+	15650 12550 17050 12550
+Wire Wire Line
+	15650 12350 17050 12350
+Wire Wire Line
+	15650 10650 16150 10650
+Text HLabel 16150 10650 2    60   Input ~ 0
+UART4_RX
 Wire Bus Line
-	17150 12450 17150 12650
+	18150 13050 18150 13250
 Wire Bus Line
 	20750 5350 20750 5850
@@
 	17600 11350 17600 11850
 Wire Bus Line
-	4800 9050 4800 11850
+	3050 8900 3050 11700
 Wire Bus Line
 	20600 9700 20600 11200

Commit message: design_emb.sch
Connections:
- net labels added: FMC_NB0, FMC_NB1
- net labels removed: FMCNBL[1...0], FMC_NBL0, FMC_NBL1, VDD_3V3
- wire segments 240 -> 237
Changed lines of the file:
@@
 FMC_NE1
 Wire Wire Line
-	4500 11600 3150 11600
-Entry Wire Line
-	3050 11500 3150 11600
-Wire Wire Line
-	4500 11500 3150 11500
-Entry Wire Line
-	3050 11400 3150 11500
-Wire Wire Line
-	4500 11400 3150 11400
-Entry Wire Line
-	3050 11300 3150 11400
-Wire Wire Line
-	4500 11300 3150 11300
-Entry Wire Line
-	3050 11200 3150 11300
+	3450 10100 2100 10100
+Entry Wire Line
+	2000 10000 2100 10100
+Wire Wire Line
+	3450 10000 2100 10000
+Entry Wire Line
+	2000 9900 2100 10000
+Wire Wire Line
+	3450 9900 2100 9900
+Entry Wire Line
+	2000 9800 2100 9900
+Wire Wire Line
+	3450 9800 2100 9800
+Entry Wire Line
+	2000 9700 2100 9800
 Text Label 5800 11550 0    60   ~ 0
 FMC_A19
@@
 FMC_A23
 Wire Bus Line
-	3050 8900 2800 8900
-Text HLabel 2800 8900 0    60   BiDi ~ 0
+	2000 7400 1750 7400
+Text HLabel 1750 7400 0    60   BiDi ~ 0
 FMCA[24...16]
 Wire Wire Line
-	4500 9000 3150 9000
+	3450 7500 2100 7500
 Text Label 5750 9150 0    60   ~ 0
 FMC_A24
-Entry Wire Line
-	2650 12000 2750 12100
-Entry Wire Line
-	2650 12100 2750 12200
-Wire Bus Line
-	2650 12100 2650 12000
-Wire Bus Line
-	2650 12000 2400 12000
-Text HLabel 2400 12000 0    60   BiDi ~ 0
-FMCNBL[1...0]
 Wire Wire Line
 	16650 13050 18050 13050
@@
 	18050 13150 18150 13250
 Text Label 5750 11250 0    60   ~ 0
-FMC_NBL0
+FMC_NB0
 Text Label 5750 11350 0    60   ~ 0
-FMC_NBL1
+FMC_NB1
 Text Label 15800 8550 0    60   ~ 0
 FMC_NAVD
@@
 	11350 13250 11350 13500
 Entry Wire Line
-	3050 8900 3150 9000
+	2000 7400 2100 7500
 $Comp
 L power:GND #PWR0101
@@
 Text HLabel 1500 2600 0    60   Input ~ 0
 VDD3V3
-Wire Wire Line
-	15650 11450 16150 11450
 Wire Wire Line
 	12900 2600 13050 2600
@@
 	15650 8550 17300 8550
 Text HLabel 5950 6250 0    60   Input ~ 0
-VDD_3V3
+VDD3V3
 Wire Wire Line
 	6250 6250 5950 6250
@@
 FMCA18
 Wire Wire Line
-	4200 12500 3000 12500
-Wire Wire Line
-	3000 12500 3000 12200
-Wire Wire Line
-	3000 12200 2750 12200
-Wire Wire Line
-	4200 12400 3100 12400
-Wire Wire Line
-	3100 12400 3100 12100
-Wire Wire Line
-	3100 12100 2750 12100
-Text Label 3200 12400 0    60   ~ 0
+	3850 11350 3850 11050
+Wire Wire Line
+	3850 11050 3550 11050
+Wire Wire Line
+	3950 11250 3950 10950
+Wire Wire Line
+	3950 10950 3550 10950
+Text Label 4050 11250 0    60   ~ 0
 FMCNBL0
-Text Label 3200 12500 0    60   ~ 0
+Text Label 4050 11350 0    60   ~ 0
 FMCNBL1
 Wire Wire Line
-	3150 11700 4500 11700
-Entry Wire Line
-	3050 11600 3150 11700
+	2100 10200 3450 10200
+Entry Wire Line
+	2000 10100 2100 10200
 Text HLabel 9000 2600 0    60   Input ~ 0
 VDD3V3
 Text HLabel 19700 12100 0    60   Input ~ 0
 VDD3V3
-Text Label 4200 12400 0    60   ~ 0
-FMC_NBL0
-Text Label 4200 12500 0    60   ~ 0
-FMC_NBL1
-Wire Wire Line
-	6250 11350 5050 11350
-Wire Wire Line
-	6250 11250 5150 11250
-Text Label 4050 11400 0    60   ~ 0
+Text Label 3000 9900 0    60   ~ 0
 FMC_A19
-Text Label 4050 11500 0    60   ~ 0
+Text Label 3000 10000 0    60   ~ 0
 FMC_A20
-Text Label 4050 11600 0    60   ~ 0
+Text Label 3000 10100 0    60   ~ 0
 FMC_A21
-Text Label 4050 11700 0    60   ~ 0
+Text Label 3000 10200 0    60   ~ 0
 FMC_A22
-Text Label 4050 11300 0    60   ~ 0
+Text Label 3000 9800 0    60   ~ 0
 FMC_A23
-Text Label 4000 9000 0    60   ~ 0
+Text Label 2950 7500 0    60   ~ 0
 FMC_A24
-Text Label 3350 9000 0    60   ~ 0
+Text Label 2300 7500 0    60   ~ 0
 FMCA24
-Text Label 3350 11300 0    60   ~ 0
+Text Label 2300 9800 0    60   ~ 0
 FMCA23
-Text Label 3350 11400 0    60   ~ 0
+Text Label 2300 9900 0    60   ~ 0
 FMCA19
-Text Label 3350 11500 0    60   ~ 0
+Text Label 2300 10000 0    60   ~ 0
 FMCA20
-Text Label 3350 11600 0    60   ~ 0
+Text Label 2300 10100 0    60   ~ 0
 FMCA21
-Text Label 3350 11700 0    60   ~ 0
+Text Label 2300 10200 0    60   ~ 0
 FMCA22
 Wire Wire Line
@@
 Text HLabel 16150 10650 2    60   Input ~ 0
 UART4_RX
+Wire Wire Line
+	3850 11350 6250 11350
+Wire Wire Line
+	3950 11250 6250 11250
+Text HLabel 3550 10950 0    60   BiDi ~ 0
+FMCNBL0
+Text HLabel 3550 11050 0    60   BiDi ~ 0
+FMCNBL1
 Wire Bus Line
 	18150 13050 18150 13250
 Wire Bus Line
+	17600 11350 17600 11850
+Wire Bus Line
 	20750 5350 20750 5850
 Wire Bus Line
-	17600 11350 17600 11850
-Wire Bus Line
-	3050 8900 3050 11700
+	2000 7400 2000 10200
 Wire Bus Line
 	20600 9700 20600 11200

Commit message: bus SPI, FMC_A Y FMC_NBL
Connections:
- net labels added: FMCNBL[1.0]
- wire segments 237 -> 233
Other:
- moved on the sheet: U3
