File: kicad/power.sch (KiCad schematic (older format))
At the start: 4 parts

Commit message: reguladores y conexión a stm32
Parts:
- removed J?: USB_OTG, symbol conn:USB_OTG
- added C? (x3): 0.1uF, symbol device:CP1
- added C? (x4): 1uF, symbol device:CP1
- added D?: LED, symbol device:LED
- added R?: 1k, symbol Device:R
- added SW?: SW_SPST, symbol Switch:SW_SPST
- added U?: TLV1117LV33DCYR, DCY4, symbol TLV1117LV33DCYR:TLV1117LV33DCYR
- added U?: TLV1117LV12DCYR, DCY4, symbol TLV1117LV33DCYR:TLV1117LV12DCYR
Connections:
- net labels added: +1V2_FPGA, +3V3, +3V3_FPGA, VDDA
- net labels removed: +3v3
- wire segments 5 -> 27
Other:
- note added: "+5VDC\n"
- note added: "POWER SUPPLY\n\n"
- note added: "XR5 or XR7-type ceramic capacitors are recommended."

Commit message: leds de prueba
Parts:
- D?: value LED -> LED_ON
Changed lines of the file:
@@
 P 7100 1950
 F 0 "D?" V 7138 1833 50  0000 R CNN
-F 1 "LED" V 7047 1833 50  0000 R CNN
+F 1 "LED_ON" V 7047 1833 50  0000 R CNN
 F 2 "" H 7100 1950 50  0001 C CNN
 F 3 "" H 7100 1950 50  0001 C CNN

Commit message: anotaciones
Parts:
- added J?: Barrel_Jack, symbol conn:Barrel_Jack
Other:
- note added: "PROBE LED"
Changed lines of the file:
@@
 EESchema Schematic File Version 4
+LIBS:power
+LIBS:74xx
 LIBS:stm32f446zetx
+LIBS:design_emb-cache
 EELAYER 26 0
 EELAYER END
@@
 L device:LED D?
 U 1 1 5B99282B
-P 7100 1950
-F 0 "D?" V 7138 1833 50  0000 R CNN
-F 1 "LED_ON" V 7047 1833 50  0000 R CNN
-F 2 "" H 7100 1950 50  0001 C CNN
-F 3 "" H 7100 1950 50  0001 C CNN
-	1    7100 1950
+P 7600 1950
+F 0 "D?" V 7638 1833 50  0000 R CNN
+F 1 "LED_ON" V 7547 1833 50  0000 R CNN
+F 2 "" H 7600 1950 50  0001 C CNN
+F 3 "" H 7600 1950 50  0001 C CNN
+	1    7600 1950
 	0    -1   -1   0
 $EndComp
 Wire Wire Line
-	7100 1800 7100 1700
-Wire Wire Line
-	7100 1700 6950 1700
-Text HLabel 6950 1700 0    60   Input ~ 0
+	7600 1800 7600 1700
+Wire Wire Line
+	7600 1700 7450 1700
+Text HLabel 7450 1700 0    60   Input ~ 0
 +3V3
 $Comp
 L Device:R R?
 U 1 1 5B99299C
-P 7100 2400
-F 0 "R?" H 7170 2446 50  0000 L CNN
-F 1 "1k" H 7170 2355 50  0000 L CNN
-F 2 "" V 7030 2400 50  0001 C CNN
-F 3 "~" H 7100 2400 50  0001 C CNN
-	1    7100 2400
-	1    0    0    -1
-$EndComp
-Wire Wire Line
-	7100 2100 7100 2250
+P 7600 2400
+F 0 "R?" H 7670 2446 50  0000 L CNN
+F 1 "1k" H 7670 2355 50  0000 L CNN
+F 2 "" V 7530 2400 50  0001 C CNN
+F 3 "~" H 7600 2400 50  0001 C CNN
+	1    7600 2400
+	1    0    0    -1
+$EndComp
+Wire Wire Line
+	7600 2100 7600 2250
 $Comp
 L power:GND #PWR?
 U 1 1 5B992A60
-P 7100 2700
-F 0 "#PWR?" H 7100 2450 50  0001 C CNN
-F 1 "GND" H 7105 2527 50  0000 C CNN
-F 2 "" H 7100 2700 50  0001 C CNN
-F 3 "" H 7100 2700 50  0001 C CNN
-	1    7100 2700
-	1    0    0    -1
-$EndComp
-Wire Wire Line
-	7100 2550 7100 2700
+P 7600 2700
+F 0 "#PWR?" H 7600 2450 50  0001 C CNN
+F 1 "GND" H 7605 2527 50  0000 C CNN
+F 2 "" H 7600 2700 50  0001 C CNN
+F 3 "" H 7600 2700 50  0001 C CNN
+	1    7600 2700
+	1    0    0    -1
+$EndComp
+Wire Wire Line
+	7600 2550 7600 2700
 Wire Wire Line
 	5600 1850 5600 2000
@@
 Text HLabel 6100 3650 2    60   Output ~ 0
 +3V3_FPGA
+$Comp
+L conn:Barrel_Jack J?
+U 1 1 5B9BF6D3
+P 1350 3250
+F 0 "J?" H 1428 3575 50  0000 C CNN
+F 1 "Barrel_Jack" H 1428 3484 50  0000 C CNN
+F 2 "" H 1400 3210 50  0001 C CNN
+F 3 "~" H 1400 3210 50  0001 C CNN
+	1    1350 3250
+	1    0    0    -1
+$EndComp
+Text Notes 7400 2550 1    79   ~ 0
+PROBE LED
 $EndSCHEMATC

Commit message: footprints resistencias y condensadores
Parts:
- C? (x9): footprint (none) -> Capacitors_Tantalum_SMD:CP_Tantalum_Case-A_EIA-3216-18_Hand
- D?: footprint (none) -> LEDs:LED_0603_HandSoldering
- R?: footprint (none) -> Resistors_SMD:R_0603_HandSoldering
Changed lines of the file:
@@
 EESchema Schematic File Version 4
+LIBS:power
+LIBS:74xx
 LIBS:stm32f446zetx
 LIBS:design_emb-cache
@@
 F 0 "C?" H 4315 2196 50  0000 L CNN
 F 1 "1uF" H 4315 2105 50  0000 L CNN
-F 2 "" H 4200 2150 50  0001 C CNN
+F 2 "Capacitors_Tantalum_SMD:CP_Tantalum_Case-A_EIA-3216-18_Hand" H 4200 2150 50  0001 C CNN
 F 3 "" H 4200 2150 50  0001 C CNN
 	1    4200 2150
@@
 F 0 "C?" H 5715 2196 50  0000 L CNN
 F 1 "1uF" H 5715 2105 50  0000 L CNN
-F 2 "" H 5600 2150 50  0001 C CNN
+F 2 "Capacitors_Tantalum_SMD:CP_Tantalum_Case-A_EIA-3216-18_Hand" H 5600 2150 50  0001 C CNN
 F 3 "" H 5600 2150 50  0001 C CNN
 	1    5600 2150
@@
 F 0 "D?" V 7638 1833 50  0000 R CNN
 F 1 "LED_ON" V 7547 1833 50  0000 R CNN
-F 2 "" H 7600 1950 50  0001 C CNN
+F 2 "LEDs:LED_0603_HandSoldering" H 7600 1950 50  0001 C CNN
 F 3 "" H 7600 1950 50  0001 C CNN
 	1    7600 1950
@@
 F 0 "R?" H 7670 2446 50  0000 L CNN
 F 1 "1k" H 7670 2355 50  0000 L CNN
-F 2 "" V 7530 2400 50  0001 C CNN
+F 2 "Resistors_SMD:R_0603_HandSoldering" V 7530 2400 50  0001 C CNN
 F 3 "~" H 7600 2400 50  0001 C CNN
 	1    7600 2400
@@
 F 0 "C?" H 6065 2196 50  0000 L CNN
 F 1 "0.1uF" H 6065 2105 50  0000 L CNN
-F 2 "" H 5950 2150 50  0001 C CNN
+F 2 "Capacitors_Tantalum_SMD:CP_Tantalum_Case-A_EIA-3216-18_Hand" H 5950 2150 50  0001 C CNN
 F 3 "" H 5950 2150 50  0001 C CNN
 	1    5950 2150
@@
 F 0 "C?" H 4365 4146 50  0000 L CNN
 F 1 "1uF" H 4365 4055 50  0000 L CNN
-F 2 "" H 4250 4100 50  0001 C CNN
+F 2 "Capacitors_Tantalum_SMD:CP_Tantalum_Case-A_EIA-3216-18_Hand" H 4250 4100 50  0001 C CNN
 F 3 "" H 4250 4100 50  0001 C CNN
 	1    4250 4100
@@
 F 0 "C?" H 5765 4146 50  0000 L CNN
 F 1 "1uF" H 5765 4055 50  0000 L CNN
-F 2 "" H 5650 4100 50  0001 C CNN
+F 2 "Capacitors_Tantalum_SMD:CP_Tantalum_Case-A_EIA-3216-18_Hand" H 5650 4100 50  0001 C CNN
 F 3 "" H 5650 4100 50  0001 C CNN
 	1    5650 4100
@@
 F 0 "C?" H 6115 4146 50  0000 L CNN
 F 1 "0.1uF" H 6115 4055 50  0000 L CNN
-F 2 "" H 6000 4100 50  0001 C CNN
+F 2 "Capacitors_Tantalum_SMD:CP_Tantalum_Case-A_EIA-3216-18_Hand" H 6000 4100 50  0001 C CNN
 F 3 "" H 6000 4100 50  0001 C CNN
 	1    6000 4100
@@
 F 0 "C?" H 4365 5696 50  0000 L CNN
 F 1 "1uF" H 4365 5605 50  0000 L CNN
-F 2 "" H 4250 5650 50  0001 C CNN
+F 2 "Capacitors_Tantalum_SMD:CP_Tantalum_Case-A_EIA-3216-18_Hand" H 4250 5650 50  0001 C CNN
 F 3 "" H 4250 5650 50  0001 C CNN
 	1    4250 5650
@@
 F 0 "C?" H 5765 5696 50  0000 L CNN
 F 1 "1uF" H 5765 5605 50  0000 L CNN
-F 2 "" H 5650 5650 50  0001 C CNN
+F 2 "Capacitors_Tantalum_SMD:CP_Tantalum_Case-A_EIA-3216-18_Hand" H 5650 5650 50  0001 C CNN
 F 3 "" H 5650 5650 50  0001 C CNN
 	1    5650 5650
@@
 F 0 "C?" H 6115 5696 50  0000 L CNN
 F 1 "0.1uF" H 6115 5605 50  0000 L CNN
-F 2 "" H 6000 5650 50  0001 C CNN
+F 2 "Capacitors_Tantalum_SMD:CP_Tantalum_Case-A_EIA-3216-18_Hand" H 6000 5650 50  0001 C CNN
 F 3 "" H 6000 5650 50  0001 C CNN
 	1    6000 5650
