File: kicad/fpga.sch (KiCad schematic (older format))
At the start: 16 parts

Commit message: design_emb.sch
Connections:
- net labels added: FMC_NBL0, FMC_NBL1
- net labels removed: ENABLE0, ENABLE1
Changed lines of the file:
@@
 Cont[5...0]
 Text Label 14450 8400 0    60   ~ 0
-ENABLE0
+FMC_NBL0
 Wire Wire Line
 	14400 8400 14900 8400
@@
 	14400 8500 14900 8500
 Text Label 14450 8500 0    60   ~ 0
-ENABLE1
+FMC_NBL1
 Entry Wire Line
 	14900 8400 15000 8300

Commit message: footprints resistencias y condensadores
Parts:
- removed 100nF (x6): C, symbol device:C
- added C? (x6): 100nF, Capacitors_Tantalum_SMD:CP_Tantalum_Case-A_EIA-3216-18_Hand, symbol device:CP1
- C? (x7): renamed from 100nF; value C -> 100nF; footprint (none) -> Capacitors_Tantalum_SMD:CP_Tantalum_Case-A_EIA-3216-18_Hand; symbol device:C -> device:CP1
- D?: footprint (none) -> LEDs:LED_0603_HandSoldering
- R?: value 1000 -> 1k; footprint (none) -> Resistors_SMD:R_0603_HandSoldering
Changed lines of the file:
@@
 EESchema Schematic File Version 4
+LIBS:power
+LIBS:74xx
 LIBS:stm32f446zetx
 LIBS:design_emb-cache
@@
 P 8900 10600
 F 0 "R?" V 8693 10600 50  0000 C CNN
-F 1 "1000" V 8784 10600 50  0000 C CNN
-F 2 "" V 8830 10600 50  0001 C CNN
+F 1 "1k" V 8784 10600 50  0000 C CNN
+F 2 "Resistors_SMD:R_0603_HandSoldering" V 8830 10600 50  0001 C CNN
 F 3 "" H 8900 10600 50  0001 C CNN
 	1    8900 10600
@@
 F 0 "D?" H 8441 10816 50  0000 C CNN
 F 1 "LED" H 8441 10725 50  0000 C CNN
-F 2 "" H 8450 10600 50  0001 C CNN
+F 2 "LEDs:LED_0603_HandSoldering" H 8450 10600 50  0001 C CNN
 F 3 "" H 8450 10600 50  0001 C CNN
 	1    8450 10600
@@
 NoConn ~ 12100 3300
 $Comp
-L device:C 100nF
+L device:CP1 C?
 U 1 1 5B9B30D6
 P 10800 2800
-F 0 "100nF" H 10800 2900 50  0000 L CNN
-F 1 "C" H 10915 2755 50  0000 L CNN
-F 2 "" H 10838 2650 50  0001 C CNN
+F 0 "C?" H 10800 2900 50  0000 L CNN
+F 1 "100nF" H 10915 2755 50  0000 L CNN
+F 2 "Capacitors_Tantalum_SMD:CP_Tantalum_Case-A_EIA-3216-18_Hand" H 10838 2650 50  0001 C CNN
 F 3 "" H 10800 2800 50  0001 C CNN
 	1    10800 2800
@@
 $EndComp
 $Comp
-L device:C 100nF
+L device:CP1 C?
 U 1 1 5B9DB436
 P 10550 2800
-F 0 "100nF" H 10550 2900 50  0000 L CNN
-F 1 "C" H 10665 2755 50  0000 L CNN
-F 2 "" H 10588 2650 50  0001 C CNN
+F 0 "C?" H 10550 2900 50  0000 L CNN
+F 1 "100nF" H 10665 2755 50  0000 L CNN
+F 2 "Capacitors_Tantalum_SMD:CP_Tantalum_Case-A_EIA-3216-18_Hand" H 10588 2650 50  0001 C CNN
 F 3 "" H 10550 2800 50  0001 C CNN
 	1    10550 2800
@@
 $EndComp
 $Comp
-L device:C 100nF
+L device:CP1 C?
 U 1 1 5B9E993D
 P 10300 2800
-F 0 "100nF" H 10300 2900 50  0000 L CNN
-F 1 "C" H 10415 2755 50  0000 L CNN
-F 2 "" H 10338 2650 50  0001 C CNN
+F 0 "C?" H 10300 2900 50  0000 L CNN
+F 1 "100nF" H 10415 2755 50  0000 L CNN
+F 2 "Capacitors_Tantalum_SMD:CP_Tantalum_Case-A_EIA-3216-18_Hand" H 10338 2650 50  0001 C CNN
 F 3 "" H 10300 2800 50  0001 C CNN
 	1    10300 2800
@@
 $EndComp
 $Comp
-L device:C 100nF
+L device:CP1 C?
 U 1 1 5B9E9944
 P 10050 2800
-F 0 "100nF" H 10050 2900 50  0000 L CNN
-F 1 "C" H 10165 2755 50  0000 L CNN
-F 2 "" H 10088 2650 50  0001 C CNN
+F 0 "C?" H 10050 2900 50  0000 L CNN
+F 1 "100nF" H 10165 2755 50  0000 L CNN
+F 2 "Capacitors_Tantalum_SMD:CP_Tantalum_Case-A_EIA-3216-18_Hand" H 10088 2650 50  0001 C CNN
 F 3 "" H 10050 2800 50  0001 C CNN
 	1    10050 2800
@@
 $EndComp
 $Comp
-L device:C 100nF
+L device:CP1 C?
 U 1 1 5B9ED2C9
 P 9800 2800
-F 0 "100nF" H 9800 2900 50  0000 L CNN
-F 1 "C" H 9915 2755 50  0000 L CNN
-F 2 "" H 9838 2650 50  0001 C CNN
+F 0 "C?" H 9800 2900 50  0000 L CNN
+F 1 "100nF" H 9915 2755 50  0000 L CNN
+F 2 "Capacitors_Tantalum_SMD:CP_Tantalum_Case-A_EIA-3216-18_Hand" H 9838 2650 50  0001 C CNN
 F 3 "" H 9800 2800 50  0001 C CNN
 	1    9800 2800
@@
 $EndComp
 $Comp
-L device:C 100nF
-U 1 1 5BA67665
-P 14100 2800
-F 0 "100nF" H 14100 2900 50  0000 L CNN
-F 1 "C" H 14215 2755 50  0000 L CNN
-F 2 "" H 14138 2650 50  0001 C CNN
-F 3 "" H 14100 2800 50  0001 C CNN
-	1    14100 2800
-	1    0    0    -1
-$EndComp
-$Comp
-L device:C 100nF
-U 1 1 5BA6766C
-P 13850 2800
-F 0 "100nF" H 13850 2900 50  0000 L CNN
-F 1 "C" H 13965 2755 50  0000 L CNN
-F 2 "" H 13888 2650 50  0001 C CNN
-F 3 "" H 13850 2800 50  0001 C CNN
-	1    13850 2800
-	1    0    0    -1
-$EndComp
-$Comp
-L device:C 100nF
-U 1 1 5BA67673
-P 13600 2800
-F 0 "100nF" H 13600 2900 50  0000 L CNN
-F 1 "C" H 13715 2755 50  0000 L CNN
-F 2 "" H 13638 2650 50  0001 C CNN
-F 3 "" H 13600 2800 50  0001 C CNN
-	1    13600 2800
-	1    0    0    -1
-$EndComp
-$Comp
-L device:C 100nF
+L device:CP1 C?
 U 1 1 5BA6767A
 P 13350 2800
-F 0 "100nF" H 13350 2900 50  0000 L CNN
-F 1 "C" H 13465 2755 50  0000 L CNN
-F 2 "" H 13388 2650 50  0001 C CNN
+F 0 "C?" H 13350 2900 50  0000 L CNN
+F 1 "100nF" H 13465 2755 50  0000 L CNN
+F 2 "Capacitors_Tantalum_SMD:CP_Tantalum_Case-A_EIA-3216-18_Hand" H 13388 2650 50  0001 C CNN
 F 3 "" H 13350 2800 50  0001 C CNN
 	1    13350 2800
@@
 $EndComp
 $Comp
-L device:C 100nF
+L device:CP1 C?
 U 1 1 5BA67681
 P 13100 2800
-F 0 "100nF" H 13100 2900 50  0000 L CNN
-F 1 "C" H 13215 2755 50  0000 L CNN
-F 2 "" H 13138 2650 50  0001 C CNN
+F 0 "C?" H 13100 2900 50  0000 L CNN
+F 1 "100nF" H 13215 2755 50  0000 L CNN
+F 2 "Capacitors_Tantalum_SMD:CP_Tantalum_Case-A_EIA-3216-18_Hand" H 13138 2650 50  0001 C CNN
 F 3 "" H 13100 2800 50  0001 C CNN
 	1    13100 2800
@@
 Wire Wire Line
 	13350 2650 13100 2650
-Connection ~ 13600 2650
-Wire Wire Line
-	13600 2650 13350 2650
-Connection ~ 13850 2650
-Wire Wire Line
-	13850 2650 13600 2650
-Wire Wire Line
-	14100 2650 13850 2650
 Wire Wire Line
 	13100 2950 13350 2950
 Connection ~ 13350 2950
-Wire Wire Line
-	13350 2950 13600 2950
-Connection ~ 13600 2950
-Wire Wire Line
-	13600 2950 13850 2950
 $Comp
 L power:GND #PWR?
@@
 	1    0    0    -1
 $EndComp
-$Comp
-L device:C 100nF
-U 1 1 5BA6E0FB
-P 14350 2800
-F 0 "100nF" H 14350 2900 50  0000 L CNN
-F 1 "C" H 14465 2755 50  0000 L CNN
-F 2 "" H 14388 2650 50  0001 C CNN
-F 3 "" H 14350 2800 50  0001 C CNN
-	1    14350 2800
-	1    0    0    -1
-$EndComp
-$Comp
-L device:C 100nF
-U 1 1 5BA74BA0
-P 14600 2800
-F 0 "100nF" H 14600 2900 50  0000 L CNN
-F 1 "C" H 14715 2755 50  0000 L CNN
-F 2 "" H 14638 2650 50  0001 C CNN
-F 3 "" H 14600 2800 50  0001 C CNN
-	1    14600 2800
-	1    0    0    -1
-$EndComp
-Wire Wire Line
-	14100 2650 14350 2650
 Connection ~ 14100 2650
-Connection ~ 14350 2650
-Wire Wire Line
-	14350 2650 14600 2650
-$Comp
-L device:C 100nF
-U 1 1 5BA893EC
-P 14850 2800
-F 0 "100nF" H 14850 2900 50  0000 L CNN
-F 1 "C" H 14965 2755 50  0000 L CNN
-F 2 "" H 14888 2650 50  0001 C CNN
-F 3 "" H 14850 2800 50  0001 C CNN
-	1    14850 2800
-	1    0    0    -1
-$EndComp
-Wire Wire Line
-	14600 2650 14850 2650
-Connection ~ 14600 2650
 Text HLabel 13850 2450 0    60   Input ~ 0
 +3V3_FPGA
@@
 Wire Wire Line
 	14100 2450 13850 2450
-Wire Wire Line
-	13850 2950 14100 2950
-Connection ~ 13850 2950
 Connection ~ 14100 2950
-Wire Wire Line
-	14100 2950 14350 2950
-Connection ~ 14350 2950
-Wire Wire Line
-	14350 2950 14600 2950
-Connection ~ 14600 2950
-Wire Wire Line
-	14600 2950 14850 2950
 Text HLabel 7500 10650 0    60   BiDi ~ 0
 ICE40_SPI[3...0]
@@
 Text HLabel 8250 10850 0    60   BiDi ~ 0
 RESET_B
+Wire Wire Line
+	14100 2650 14350 2650
+Wire Wire Line
+	14100 2950 14350 2950
+Wire Wire Line
+	13350 2650 13600 2650
+Wire Wire Line
+	13350 2950 13600 2950
 Wire Bus Line
 	15000 8200 15000 8500
@@
 Wire Bus Line
 	20050 3800 20050 5500
+$Comp
+L device:CP1 C?
+U 1 1 5BA2D18B
+P 13600 2800
+F 0 "C?" H 13600 2900 50  0000 L CNN
+F 1 "100nF" H 13715 2755 50  0000 L CNN
+F 2 "Capacitors_Tantalum_SMD:CP_Tantalum_Case-A_EIA-3216-18_Hand" H 13638 2650 50  0001 C CNN
+F 3 "" H 13600 2800 50  0001 C CNN
+	1    13600 2800
+	1    0    0    -1
+$EndComp
+Connection ~ 13600 2650
+Wire Wire Line
+	13600 2650 13850 2650
+Connection ~ 13600 2950
+Wire Wire Line
+	13600 2950 13850 2950
+$Comp
+L device:CP1 C?
+U 1 1 5BA2D2CF
+P 13850 2800
+F 0 "C?" H 13850 2900 50  0000 L CNN
+F 1 "100nF" H 13965 2755 50  0000 L CNN
+F 2 "Capacitors_Tantalum_SMD:CP_Tantalum_Case-A_EIA-3216-18_Hand" H 13888 2650 50  0001 C CNN
+F 3 "" H 13850 2800 50  0001 C CNN
+	1    13850 2800
+	1    0    0    -1
+$EndComp
+Connection ~ 13850 2650
+Wire Wire Line
+	13850 2650 14100 2650
+Connection ~ 13850 2950
+Wire Wire Line
+	13850 2950 14100 2950
+$Comp
+L device:CP1 C?
+U 1 1 5BA2D301
+P 14100 2800
+F 0 "C?" H 14100 2900 50  0000 L CNN
+F 1 "100nF" H 14215 2755 50  0000 L CNN
+F 2 "Capacitors_Tantalum_SMD:CP_Tantalum_Case-A_EIA-3216-18_Hand" H 14138 2650 50  0001 C CNN
+F 3 "" H 14100 2800 50  0001 C CNN
+	1    14100 2800
+	1    0    0    -1
+$EndComp
+$Comp
+L device:CP1 C?
+U 1 1 5BA2D331
+P 14350 2800
+F 0 "C?" H 14350 2900 50  0000 L CNN
+F 1 "100nF" H 14465 2755 50  0000 L CNN
+F 2 "Capacitors_Tantalum_SMD:CP_Tantalum_Case-A_EIA-3216-18_Hand" H 14388 2650 50  0001 C CNN
+F 3 "" H 14350 2800 50  0001 C CNN
+	1    14350 2800
+	1    0    0    -1
+$EndComp
+Connection ~ 14350 2650
+Wire Wire Line
+	14350 2650 14600 2650
+Connection ~ 14350 2950
+Wire Wire Line
+	14350 2950 14600 2950
+$Comp
+L device:CP1 C?
+U 1 1 5BA2D367
+P 14600 2800
+F 0 "C?" H 14600 2900 50  0000 L CNN
+F 1 "100nF" H 14715 2755 50  0000 L CNN
+F 2 "Capacitors_Tantalum_SMD:CP_Tantalum_Case-A_EIA-3216-18_Hand" H 14638 2650 50  0001 C CNN
+F 3 "" H 14600 2800 50  0001 C CNN
+	1    14600 2800
+	1    0    0    -1
+$EndComp
+Connection ~ 14600 2650
+Wire Wire Line
+	14600 2650 14850 2650
+Connection ~ 14600 2950
+Wire Wire Line
+	14600 2950 14850 2950
+$Comp
+L device:CP1 C?
+U 1 1 5BA2D39F
+P 14850 2800
+F 0 "C?" H 14850 2900 50  0000 L CNN
+F 1 "100nF" H 14965 2755 50  0000 L CNN
+F 2 "Capacitors_Tantalum_SMD:CP_Tantalum_Case-A_EIA-3216-18_Hand" H 14888 2650 50  0001 C CNN
+F 3 "" H 14850 2800 50  0001 C CNN
+	1    14850 2800
+	1    0    0    -1
+$EndComp
 $EndSCHEMATC

Commit message: design_emb.sch
Parts:
- added C? (x2): 100nF, Capacitors_Tantalum_SMD:CP_Tantalum_Case-A_EIA-3216-18_Hand, symbol device:CP1
- added D?: 1N5817, Diodes_THT:D_DO-41_SOD81_Horizontal_RM10, symbol diode:1N5817
- added R?: 10k, symbol device:R
- added SW?: SW_Push, symbol switches:SW_Push
Connections:
- net labels added: CRESET_B
- wire segments 135 -> 151
Changed lines of the file:
@@
 EESchema Schematic File Version 4
-LIBS:power
-LIBS:74xx
 LIBS:stm32f446zetx
 LIBS:design_emb-cache
@@
 Wire Wire Line
 	13350 2950 13600 2950
+$Comp
+L device:CP1 C?
+U 1 1 5BA2D18B
+P 13600 2800
+F 0 "C?" H 13600 2900 50  0000 L CNN
+F 1 "100nF" H 13715 2755 50  0000 L CNN
+F 2 "Capacitors_Tantalum_SMD:CP_Tantalum_Case-A_EIA-3216-18_Hand" H 13638 2650 50  0001 C CNN
+F 3 "" H 13600 2800 50  0001 C CNN
+	1    13600 2800
+	1    0    0    -1
+$EndComp
+Connection ~ 13600 2650
+Wire Wire Line
+	13600 2650 13850 2650
+Connection ~ 13600 2950
+Wire Wire Line
+	13600 2950 13850 2950
+$Comp
+L device:CP1 C?
+U 1 1 5BA2D2CF
+P 13850 2800
+F 0 "C?" H 13850 2900 50  0000 L CNN
+F 1 "100nF" H 13965 2755 50  0000 L CNN
+F 2 "Capacitors_Tantalum_SMD:CP_Tantalum_Case-A_EIA-3216-18_Hand" H 13888 2650 50  0001 C CNN
+F 3 "" H 13850 2800 50  0001 C CNN
+	1    13850 2800
+	1    0    0    -1
+$EndComp
+Connection ~ 13850 2650
+Wire Wire Line
+	13850 2650 14100 2650
+Connection ~ 13850 2950
+Wire Wire Line
+	13850 2950 14100 2950
+$Comp
+L device:CP1 C?
+U 1 1 5BA2D301
+P 14100 2800
+F 0 "C?" H 14100 2900 50  0000 L CNN
+F 1 "100nF" H 14215 2755 50  0000 L CNN
+F 2 "Capacitors_Tantalum_SMD:CP_Tantalum_Case-A_EIA-3216-18_Hand" H 14138 2650 50  0001 C CNN
+F 3 "" H 14100 2800 50  0001 C CNN
+	1    14100 2800
+	1    0    0    -1
+$EndComp
+$Comp
+L device:CP1 C?
+U 1 1 5BA2D331
+P 14350 2800
+F 0 "C?" H 14350 2900 50  0000 L CNN
+F 1 "100nF" H 14465 2755 50  0000 L CNN
+F 2 "Capacitors_Tantalum_SMD:CP_Tantalum_Case-A_EIA-3216-18_Hand" H 14388 2650 50  0001 C CNN
+F 3 "" H 14350 2800 50  0001 C CNN
+	1    14350 2800
+	1    0    0    -1
+$EndComp
+Connection ~ 14350 2650
+Wire Wire Line
+	14350 2650 14600 2650
+Connection ~ 14350 2950
+Wire Wire Line
+	14350 2950 14600 2950
+$Comp
+L device:CP1 C?
+U 1 1 5BA2D367
+P 14600 2800
+F 0 "C?" H 14600 2900 50  0000 L CNN
+F 1 "100nF" H 14715 2755 50  0000 L CNN
+F 2 "Capacitors_Tantalum_SMD:CP_Tantalum_Case-A_EIA-3216-18_Hand" H 14638 2650 50  0001 C CNN
+F 3 "" H 14600 2800 50  0001 C CNN
+	1    14600 2800
+	1    0    0    -1
+$EndComp
+Connection ~ 14600 2650
+Wire Wire Line
+	14600 2650 14850 2650
+Connection ~ 14600 2950
+Wire Wire Line
+	14600 2950 14850 2950
+$Comp
+L device:CP1 C?
+U 1 1 5BA2D39F
+P 14850 2800
+F 0 "C?" H 14850 2900 50  0000 L CNN
+F 1 "100nF" H 14965 2755 50  0000 L CNN
+F 2 "Capacitors_Tantalum_SMD:CP_Tantalum_Case-A_EIA-3216-18_Hand" H 14888 2650 50  0001 C CNN
+F 3 "" H 14850 2800 50  0001 C CNN
+	1    14850 2800
+	1    0    0    -1
+$EndComp
+$Comp
+L diode:1N5817 D?
+U 1 1 5BA35AEC
+P 12000 3150
+F 0 "D?" V 12046 3229 50  0000 L CNN
+F 1 "1N5817" V 11955 3229 50  0000 L CNN
+F 2 "Diodes_THT:D_DO-41_SOD81_Horizontal_RM10" H 12000 2975 50  0001 C CNN
+F 3 "http://www.vishay.com/docs/88525/1n5817.pdf" H 12000 3150 50  0001 C CNN
+	1    12000 3150
+	0    1    -1   0
+$EndComp
+$Comp
+L device:CP1 C?
+U 1 1 5BA4B6D7
+P 12550 2800
+F 0 "C?" H 12550 2900 50  0000 L CNN
+F 1 "100nF" H 12665 2755 50  0000 L CNN
+F 2 "Capacitors_Tantalum_SMD:CP_Tantalum_Case-A_EIA-3216-18_Hand" H 12588 2650 50  0001 C CNN
+F 3 "" H 12550 2800 50  0001 C CNN
+	1    12550 2800
+	1    0    0    -1
+$EndComp
+Wire Wire Line
+	12000 3050 12000 3000
+Wire Wire Line
+	12000 2650 12550 2650
+Connection ~ 12000 3000
+Wire Wire Line
+	12000 3000 12000 2650
+Wire Wire Line
+	12550 2650 13100 2650
+Connection ~ 12550 2650
+Connection ~ 13100 2650
+Wire Wire Line
+	12550 2950 13100 2950
+Connection ~ 13100 2950
+$Comp
+L device:R R?
+U 1 1 5BA62067
+P 16950 2950
+F 0 "R?" V 16743 2950 50  0000 C CNN
+F 1 "10k" V 16834 2950 50  0000 C CNN
+F 2 "" V 16880 2950 50  0001 C CNN
+F 3 "" H 16950 2950 50  0001 C CNN
+	1    16950 2950
+	0    1    1    0
+$EndComp
+Text HLabel 16600 2950 0    60   Input ~ 0
++3V3_FPGA
+Wire Wire Line
+	16600 2950 16800 2950
+$Comp
+L device:CP1 C?
+U 1 1 5BA7293B
+P 17250 3250
+F 0 "C?" H 17250 3350 50  0000 L CNN
+F 1 "100nF" H 17365 3205 50  0000 L CNN
+F 2 "Capacitors_Tantalum_SMD:CP_Tantalum_Case-A_EIA-3216-18_Hand" H 17288 3100 50  0001 C CNN
+F 3 "" H 17250 3250 50  0001 C CNN
+	1    17250 3250
+	1    0    0    -1
+$EndComp
+$Comp
+L switches:SW_Push SW?
+U 1 1 5BA7A69B
+P 17700 3200
+F 0 "SW?" V 17654 3348 50  0000 L CNN
+F 1 "SW_Push" V 17745 3348 50  0000 L CNN
+F 2 "" H 17700 3400 50  0001 C CNN
+F 3 "" H 17700 3400 50  0001 C CNN
+	1    17700 3200
+	0    1    1    0
+$EndComp
+Wire Wire Line
+	17100 2950 17250 2950
+Wire Wire Line
+	17700 2950 17700 3000
+Wire Wire Line
+	17250 3100 17250 2950
+Connection ~ 17250 2950
+Wire Wire Line
+	17250 2950 17700 2950
+Wire Wire Line
+	17250 3400 17250 3450
+Wire Wire Line
+	17250 3450 17500 3450
+Wire Wire Line
+	17700 3450 17700 3400
+Wire Wire Line
+	17500 3450 17500 3600
+Connection ~ 17500 3450
+Wire Wire Line
+	17500 3450 17700 3450
+$Comp
+L power:GND #PWR?
+U 1 1 5BAAA046
+P 17500 3600
+F 0 "#PWR?" H 17500 3350 50  0001 C CNN
+F 1 "GND" H 17505 3427 50  0000 C CNN
+F 2 "" H 17500 3600 50  0001 C CNN
+F 3 "" H 17500 3600 50  0001 C CNN
+	1    17500 3600
+	1    0    0    -1
+$EndComp
+Connection ~ 17700 2950
+Text Label 17800 2950 0    60   ~ 0
+CRESET_B
+Wire Wire Line
+	17700 2950 18350 2950
 Wire Bus Line
 	15000 8200 15000 8500
@@
 Wire Bus Line
 	20050 3800 20050 5500
-$Comp
-L device:CP1 C?
-U 1 1 5BA2D18B
-P 13600 2800
-F 0 "C?" H 13600 2900 50  0000 L CNN
-F 1 "100nF" H 13715 2755 50  0000 L CNN
-F 2 "Capacitors_Tantalum_SMD:CP_Tantalum_Case-A_EIA-3216-18_Hand" H 13638 2650 50  0001 C CNN
-F 3 "" H 13600 2800 50  0001 C CNN
-	1    13600 2800
-	1    0    0    -1
-$EndComp
-Connection ~ 13600 2650
-Wire Wire Line
-	13600 2650 13850 2650
-Connection ~ 13600 2950
-Wire Wire Line
-	13600 2950 13850 2950
-$Comp
-L device:CP1 C?
-U 1 1 5BA2D2CF
-P 13850 2800
-F 0 "C?" H 13850 2900 50  0000 L CNN
-F 1 "100nF" H 13965 2755 50  0000 L CNN
-F 2 "Capacitors_Tantalum_SMD:CP_Tantalum_Case-A_EIA-3216-18_Hand" H 13888 2650 50  0001 C CNN
-F 3 "" H 13850 2800 50  0001 C CNN
-	1    13850 2800
-	1    0    0    -1
-$EndComp
-Connection ~ 13850 2650
-Wire Wire Line
-	13850 2650 14100 2650
-Connection ~ 13850 2950
-Wire Wire Line
-	13850 2950 14100 2950
-$Comp
-L device:CP1 C?
-U 1 1 5BA2D301
-P 14100 2800
-F 0 "C?" H 14100 2900 50  0000 L CNN
-F 1 "100nF" H 14215 2755 50  0000 L CNN
-F 2 "Capacitors_Tantalum_SMD:CP_Tantalum_Case-A_EIA-3216-18_Hand" H 14138 2650 50  0001 C CNN
-F 3 "" H 14100 2800 50  0001 C CNN
-	1    14100 2800
-	1    0    0    -1
-$EndComp
-$Comp
-L device:CP1 C?
-U 1 1 5BA2D331
-P 14350 2800
-F 0 "C?" H 14350 2900 50  0000 L CNN
-F 1 "100nF" H 14465 2755 50  0000 L CNN
-F 2 "Capacitors_Tantalum_SMD:CP_Tantalum_Case-A_EIA-3216-18_Hand" H 14388 2650 50  0001 C CNN
-F 3 "" H 14350 2800 50  0001 C CNN
-	1    14350 2800
-	1    0    0    -1
-$EndComp
-Connection ~ 14350 2650
-Wire Wire Line
-	14350 2650 14600 2650
-Connection ~ 14350 2950
-Wire Wire Line
-	14350 2950 14600 2950
-$Comp
-L device:CP1 C?
-U 1 1 5BA2D367
-P 14600 2800
-F 0 "C?" H 14600 2900 50  0000 L CNN
-F 1 "100nF" H 14715 2755 50  0000 L CNN
-F 2 "Capacitors_Tantalum_SMD:CP_Tantalum_Case-A_EIA-3216-18_Hand" H 14638 2650 50  0001 C CNN
-F 3 "" H 14600 2800 50  0001 C CNN
-	1    14600 2800
-	1    0    0    -1
-$EndComp
-Connection ~ 14600 2650
-Wire Wire Line
-	14600 2650 14850 2650
-Connection ~ 14600 2950
-Wire Wire Line
-	14600 2950 14850 2950
-$Comp
-L device:CP1 C?
-U 1 1 5BA2D39F
-P 14850 2800
-F 0 "C?" H 14850 2900 50  0000 L CNN
-F 1 "100nF" H 14965 2755 50  0000 L CNN
-F 2 "Capacitors_Tantalum_SMD:CP_Tantalum_Case-A_EIA-3216-18_Hand" H 14888 2650 50  0001 C CNN
-F 3 "" H 14850 2800 50  0001 C CNN
-	1    14850 2800
-	1    0    0    -1
-$EndComp
 $EndSCHEMATC
