File: kicad/fpga.sch (KiCad schematic (older format))
At the start: 21 parts

Commit message: footprints y JTAG
Parts:
- gave numbers to parts that had none: 21
Connections:
- net labels removed: ICE40_RESETB, RESET_B
Changed lines of the file:
@@
 EESchema Schematic File Version 4
+LIBS:power
+LIBS:74xx
 LIBS:stm32f446zetx
 LIBS:design_emb-cache
@@
 Text Label 8350 11350 0    60   ~ 0
 SPI_SS
-Text Label 8350 10850 0    60   ~ 0
-ICE40_RESETB
-Wire Wire Line
-	8250 10850 9250 10850
 Wire Wire Line
 	7700 11050 9250 11050
@@
 	12300 12000 12450 12000
 $Comp
-L power:GND #PWR?
+L power:GND #PWR013
 U 1 1 5B997ACB
 P 11950 12150
-F 0 "#PWR?" H 11950 11900 50  0001 C CNN
+F 0 "#PWR013" H 11950 11900 50  0001 C CNN
 F 1 "GND" H 11955 11977 50  0000 C CNN
 F 2 "" H 11950 12150 50  0001 C CNN
@@
 	9250 10600 9050 10600
 $Comp
-L device:R R?
+L device:R R4
 U 1 1 5B996733
 P 8900 10600
-F 0 "R?" V 8693 10600 50  0000 C CNN
+F 0 "R4" V 8693 10600 50  0000 C CNN
 F 1 "1k" V 8784 10600 50  0000 C CNN
 F 2 "Resistors_SMD:R_0603_HandSoldering" V 8830 10600 50  0001 C CNN
@@
 $EndComp
 $Comp
-L device:LED D?
+L device:LED D2
 U 1 1 5B99718C
 P 8450 10600
-F 0 "D?" H 8441 10816 50  0000 C CNN
+F 0 "D2" H 8441 10816 50  0000 C CNN
 F 1 "LED" H 8441 10725 50  0000 C CNN
 F 2 "LEDs:LED_0603_HandSoldering" H 8450 10600 50  0001 C CNN
@@
 	8750 10600 8600 10600
 $Comp
-L power:GND #PWR?
+L power:GND #PWR011
 U 1 1 5B997740
 P 8200 10600
-F 0 "#PWR?" H 8200 10350 50  0001 C CNN
+F 0 "#PWR011" H 8200 10350 50  0001 C CNN
 F 1 "GND" V 8205 10472 50  0000 R CNN
 F 2 "" H 8200 10600 50  0001 C CNN
@@
 NoConn ~ 12100 3300
 $Comp
-L device:CP1 C?
+L device:CP1 C26
 U 1 1 5B9B30D6
 P 10800 2800
-F 0 "C?" H 10800 2900 50  0000 L CNN
+F 0 "C26" H 10800 2900 50  0000 L CNN
 F 1 "100nF" H 10915 2755 50  0000 L CNN
 F 2 "Capacitors_Tantalum_SMD:CP_Tantalum_Case-A_EIA-3216-18_Hand" H 10838 2650 50  0001 C CNN
@@
 $EndComp
 $Comp
-L device:CP1 C?
+L device:CP1 C25
 U 1 1 5B9DB436
 P 10550 2800
-F 0 "C?" H 10550 2900 50  0000 L CNN
+F 0 "C25" H 10550 2900 50  0000 L CNN
 F 1 "100nF" H 10665 2755 50  0000 L CNN
 F 2 "Capacitors_Tantalum_SMD:CP_Tantalum_Case-A_EIA-3216-18_Hand" H 10588 2650 50  0001 C CNN
@@
 $EndComp
 $Comp
-L device:CP1 C?
+L device:CP1 C24
 U 1 1 5B9E993D
 P 10300 2800
-F 0 "C?" H 10300 2900 50  0000 L CNN
+F 0 "C24" H 10300 2900 50  0000 L CNN
 F 1 "100nF" H 10415 2755 50  0000 L CNN
 F 2 "Capacitors_Tantalum_SMD:CP_Tantalum_Case-A_EIA-3216-18_Hand" H 10338 2650 50  0001 C CNN
@@
 $EndComp
 $Comp
-L device:CP1 C?
+L device:CP1 C23
 U 1 1 5B9E9944
 P 10050 2800
-F 0 "C?" H 10050 2900 50  0000 L CNN
+F 0 "C23" H 10050 2900 50  0000 L CNN
 F 1 "100nF" H 10165 2755 50  0000 L CNN
 F 2 "Capacitors_Tantalum_SMD:CP_Tantalum_Case-A_EIA-3216-18_Hand" H 10088 2650 50  0001 C CNN
@@
 $EndComp
 $Comp
-L device:CP1 C?
+L device:CP1 C22
 U 1 1 5B9ED2C9
 P 9800 2800
-F 0 "C?" H 9800 2900 50  0000 L CNN
+F 0 "C22" H 9800 2900 50  0000 L CNN
 F 1 "100nF" H 9915 2755 50  0000 L CNN
 F 2 "Capacitors_Tantalum_SMD:CP_Tantalum_Case-A_EIA-3216-18_Hand" H 9838 2650 50  0001 C CNN
@@
 	10550 2950 10800 2950
 $Comp
-L power:GND #PWR?
+L power:GND #PWR012
 U 1 1 5B9F89E5
 P 10300 2950
-F 0 "#PWR?" H 10300 2700 50  0001 C CNN
+F 0 "#PWR012" H 10300 2700 50  0001 C CNN
 F 1 "GND" H 10305 2777 50  0000 C CNN
 F 2 "" H 10300 2950 50  0001 C CNN
@@
 	9100 10150 9000 10150
 $Comp
-L ICE40HC1k:ICE40HX1K U?
+L ICE40HC1k:ICE40HX1K U4
 U 1 1 5B8D3D93
 P 11900 7200
-F 0 "U?" H 11825 11278 50  0000 C CNN
+F 0 "U4" H 11825 11278 50  0000 C CNN
 F 1 "ICE40HX1K" H 11825 11187 50  0000 C CNN
 F 2 "Package_QFP:TQFP-144_20x20mm_P0.5mm" H 14100 10975 50  0001 R TNN
@@
 $EndComp
 $Comp
-L device:CP1 C?
+L device:CP1 C29
 U 1 1 5BA6767A
 P 13350 2800
-F 0 "C?" H 13350 2900 50  0000 L CNN
+F 0 "C29" H 13350 2900 50  0000 L CNN
 F 1 "100nF" H 13465 2755 50  0000 L CNN
 F 2 "Capacitors_Tantalum_SMD:CP_Tantalum_Case-A_EIA-3216-18_Hand" H 13388 2650 50  0001 C CNN
@@
 $EndComp
 $Comp
-L device:CP1 C?
+L device:CP1 C28
 U 1 1 5BA67681
 P 13100 2800
-F 0 "C?" H 13100 2900 50  0000 L CNN
+F 0 "C28" H 13100 2900 50  0000 L CNN
 F 1 "100nF" H 13215 2755 50  0000 L CNN
 F 2 "Capacitors_Tantalum_SMD:CP_Tantalum_Case-A_EIA-3216-18_Hand" H 13138 2650 50  0001 C CNN
@@
 Connection ~ 13350 2950
 $Comp
-L power:GND #PWR?
+L power:GND #PWR014
 U 1 1 5BA67698
 P 14100 2950
-F 0 "#PWR?" H 14100 2700 50  0001 C CNN
+F 0 "#PWR014" H 14100 2700 50  0001 C CNN
 F 1 "GND" H 14105 2777 50  0000 C CNN
 F 2 "" H 14100 2950 50  0001 C CNN
@@
 Wire Bus Line
 	7600 10650 7500 10650
-Text HLabel 8250 10850 0    60   BiDi ~ 0
-RESET_B
 Wire Wire Line
 	14100 2650 14350 2650
@@
 	13350 2950 13600 2950
 $Comp
-L device:CP1 C?
+L device:CP1 C30
 U 1 1 5BA2D18B
 P 13600 2800
-F 0 "C?" H 13600 2900 50  0000 L CNN
+F 0 "C30" H 13600 2900 50  0000 L CNN
 F 1 "100nF" H 13715 2755 50  0000 L CNN
 F 2 "Capacitors_Tantalum_SMD:CP_Tantalum_Case-A_EIA-3216-18_Hand" H 13638 2650 50  0001 C CNN
@@
 	13600 2950 13850 2950
 $Comp
-L device:CP1 C?
+L device:CP1 C31
 U 1 1 5BA2D2CF
 P 13850 2800
-F 0 "C?" H 13850 2900 50  0000 L CNN
+F 0 "C31" H 13850 2900 50  0000 L CNN
 F 1 "100nF" H 13965 2755 50  0000 L CNN
 F 2 "Capacitors_Tantalum_SMD:CP_Tantalum_Case-A_EIA-3216-18_Hand" H 13888 2650 50  0001 C CNN
@@
 	13850 2950 14100 2950
 $Comp
-L device:CP1 C?
+L device:CP1 C32
 U 1 1 5BA2D301
 P 14100 2800
-F 0 "C?" H 14100 2900 50  0000 L CNN
+F 0 "C32" H 14100 2900 50  0000 L CNN
 F 1 "100nF" H 14215 2755 50  0000 L CNN
 F 2 "Capacitors_Tantalum_SMD:CP_Tantalum_Case-A_EIA-3216-18_Hand" H 14138 2650 50  0001 C CNN
@@
 $EndComp
 $Comp
-L device:CP1 C?
+L device:CP1 C33
 U 1 1 5BA2D331
 P 14350 2800
-F 0 "C?" H 14350 2900 50  0000 L CNN
+F 0 "C33" H 14350 2900 50  0000 L CNN
 F 1 "100nF" H 14465 2755 50  0000 L CNN
 F 2 "Capacitors_Tantalum_SMD:CP_Tantalum_Case-A_EIA-3216-18_Hand" H 14388 2650 50  0001 C CNN
@@
 	14350 2950 14600 2950
 $Comp
-L device:CP1 C?
+L device:CP1 C34
 U 1 1 5BA2D367
 P 14600 2800
-F 0 "C?" H 14600 2900 50  0000 L CNN
+F 0 "C34" H 14600 2900 50  0000 L CNN
 F 1 "100nF" H 14715 2755 50  0000 L CNN
 F 2 "Capacitors_Tantalum_SMD:CP_Tantalum_Case-A_EIA-3216-18_Hand" H 14638 2650 50  0001 C CNN
@@
 	14600 2950 14850 2950
 $Comp
-L device:CP1 C?
+L device:CP1 C35
 U 1 1 5BA2D39F
 P 14850 2800
-F 0 "C?" H 14850 2900 50  0000 L CNN
+F 0 "C35" H 14850 2900 50  0000 L CNN
 F 1 "100nF" H 14965 2755 50  0000 L CNN
 F 2 "Capacitors_Tantalum_SMD:CP_Tantalum_Case-A_EIA-3216-18_Hand" H 14888 2650 50  0001 C CNN
@@
 $EndComp
 $Comp
-L diode:1N5817 D?
+L diode:1N5817 D3
 U 1 1 5BA35AEC
 P 12000 3150
-F 0 "D?" V 12046 3229 50  0000 L CNN
+F 0 "D3" V 12046 3229 50  0000 L CNN
 F 1 "1N5817" V 11955 3229 50  0000 L CNN
 F 2 "Diodes_THT:D_DO-41_SOD81_Horizontal_RM10" H 12000 2975 50  0001 C CNN
@@
 $EndComp
 $Comp
-L device:CP1 C?
+L device:CP1 C27
 U 1 1 5BA4B6D7
 P 12550 2800
-F 0 "C?" H 12550 2900 50  0000 L CNN
+F 0 "C27" H 12550 2900 50  0000 L CNN
 F 1 "100nF" H 12665 2755 50  0000 L CNN
 F 2 "Capacitors_Tantalum_SMD:CP_Tantalum_Case-A_EIA-3216-18_Hand" H 12588 2650 50  0001 C CNN
@@
 Connection ~ 13100 2950
 $Comp
-L device:R R?
+L device:R R5
 U 1 1 5BA62067
 P 16950 2950
-F 0 "R?" V 16743 2950 50  0000 C CNN
+F 0 "R5" V 16743 2950 50  0000 C CNN
 F 1 "10k" V 16834 2950 50  0000 C CNN
 F 2 "" V 16880 2950 50  0001 C CNN
@@
 	16600 2950 16800 2950
 $Comp
-L device:CP1 C?
+L device:CP1 C36
 U 1 1 5BA7293B
 P 17250 3250
-F 0 "C?" H 17250 3350 50  0000 L CNN
+F 0 "C36" H 17250 3350 50  0000 L CNN
 F 1 "100nF" H 17365 3205 50  0000 L CNN
 F 2 "Capacitors_Tantalum_SMD:CP_Tantalum_Case-A_EIA-3216-18_Hand" H 17288 3100 50  0001 C CNN
@@
 $EndComp
 $Comp
-L switches:SW_Push SW?
+L switches:SW_Push SW1
 U 1 1 5BA7A69B
 P 17700 3200
-F 0 "SW?" V 17654 3348 50  0000 L CNN
+F 0 "SW1" V 17654 3348 50  0000 L CNN
 F 1 "SW_Push" V 17745 3348 50  0000 L CNN
 F 2 "" H 17700 3400 50  0001 C CNN
@@
 	17500 3450 17700 3450
 $Comp
-L power:GND #PWR?
+L power:GND #PWR015
 U 1 1 5BAAA046
 P 17500 3600
-F 0 "#PWR?" H 17500 3350 50  0001 C CNN
+F 0 "#PWR015" H 17500 3350 50  0001 C CNN
 F 1 "GND" H 17505 3427 50  0000 C CNN
 F 2 "" H 17500 3600 50  0001 C CNN
@@
 Wire Wire Line
 	17700 2950 18350 2950
+Wire Wire Line
+	9250 10850 8350 10850
 Wire Bus Line
 	15000 8200 15000 8500
@@
 Wire Bus Line
 	20050 3800 20050 5500
+Text Label 8600 10850 0    60   ~ 0
+CRESET_B
 $EndSCHEMATC

Commit message: footprints
Parts:
- R5: footprint (none) -> Resistors_SMD:R_0603_HandSoldering
Changed lines of the file:
@@
 F 0 "R5" V 16743 2950 50  0000 C CNN
 F 1 "10k" V 16834 2950 50  0000 C CNN
-F 2 "" V 16880 2950 50  0001 C CNN
+F 2 "Resistors_SMD:R_0603_HandSoldering" V 16880 2950 50  0001 C CNN
 F 3 "" H 16950 2950 50  0001 C CNN
 	1    16950 2950

Commit message: fpga.sch
Parts:
- added C?: 100nF, Capacitors_Tantalum_SMD:CP_Tantalum_Case-A_EIA-3216-18_Hand, symbol device:CP1
- added J? (x2): Conn_01x10, symbol conn:Conn_01x10
Connections:
- net labels added: GPIO0, GPIO1, GPIO10, GPIO11, GPIO12, GPIO13, GPIO14, GPIO15, GPIO16, GPIO17, GPIO18, GPIO19, GPIO2, GPIO3, GPIO4, GPIO5, GPIO6, GPIO7, GPIO8, GPIO9
- wire segments 151 -> 186
Changed lines of the file:
@@
 EESchema Schematic File Version 4
-LIBS:power
-LIBS:74xx
 LIBS:stm32f446zetx
 LIBS:design_emb-cache
@@
 Text HLabel 9000 10150 0    60   Input ~ 0
 +3V3_FPGA
-Text HLabel 8900 6850 0    60   Input ~ 0
+Text HLabel 8900 6900 0    60   Input ~ 0
 +3V3_FPGA
-Text HLabel 8900 6950 0    60   Input ~ 0
+Text HLabel 8900 7000 0    60   Input ~ 0
 +3V3_FPGA
 Wire Wire Line
-	8900 6850 9250 6850
-Wire Wire Line
-	8900 6950 9250 6950
+	8900 6900 9250 6900
+Wire Wire Line
+	8900 7000 9250 7000
 Wire Wire Line
 	9250 10400 9000 10400
@@
 	12000 3000 12000 2650
 Wire Wire Line
-	12550 2650 13100 2650
+	12550 2650 12850 2650
 Connection ~ 12550 2650
 Connection ~ 13100 2650
 Wire Wire Line
-	12550 2950 13100 2950
+	12550 2950 12850 2950
 Connection ~ 13100 2950
 $Comp
@@
 Wire Wire Line
 	9250 10850 8350 10850
+Text Label 8600 10850 0    60   ~ 0
+CRESET_B
+$Comp
+L device:CP1 C?
+U 1 1 5BADC284
+P 12850 2800
+F 0 "C?" H 12850 2900 50  0000 L CNN
+F 1 "100nF" H 12965 2755 50  0000 L CNN
+F 2 "Capacitors_Tantalum_SMD:CP_Tantalum_Case-A_EIA-3216-18_Hand" H 12888 2650 50  0001 C CNN
+F 3 "" H 12850 2800 50  0001 C CNN
+	1    12850 2800
+	1    0    0    -1
+$EndComp
+Connection ~ 12850 2650
+Wire Wire Line
+	12850 2650 13100 2650
+Connection ~ 12850 2950
+Wire Wire Line
+	12850 2950 13100 2950
+Wire Wire Line
+	9250 4200 8700 4200
+Wire Wire Line
+	9250 4300 8700 4300
+Wire Wire Line
+	9250 4400 8700 4400
+Wire Wire Line
+	9250 4500 8700 4500
+Wire Wire Line
+	9250 4600 8700 4600
+Wire Wire Line
+	9250 4700 8700 4700
+Wire Wire Line
+	9250 4800 8700 4800
+Wire Wire Line
+	9250 4900 8700 4900
+Wire Wire Line
+	9250 5000 8700 5000
+Wire Wire Line
+	9250 5100 8700 5100
+Text Label 8800 4200 0    60   ~ 0
+GPIO0
+Text Label 8800 4300 0    60   ~ 0
+GPIO1
+Text Label 8800 4400 0    60   ~ 0
+GPIO2
+Text Label 8800 4500 0    60   ~ 0
+GPIO3
+Text Label 8800 4600 0    60   ~ 0
+GPIO4
+Text Label 8800 4700 0    60   ~ 0
+GPIO5
+Text Label 8800 4800 0    60   ~ 0
+GPIO6
+Text Label 8800 4900 0    60   ~ 0
+GPIO7
+Text Label 8800 5000 0    60   ~ 0
+GPIO8
+Text Label 8800 5100 0    60   ~ 0
+GPIO9
+$Comp
+L conn:Conn_01x10 J?
+U 1 1 5BB3EB2A
+P 8500 4600
+F 0 "J?" H 8420 5217 50  0000 C CNN
+F 1 "Conn_01x10" H 8420 5126 50  0000 C CNN
+F 2 "" H 8500 4600 50  0001 C CNN
+F 3 "~" H 8500 4600 50  0001 C CNN
+	1    8500 4600
+	-1   0    0    -1
+$EndComp
+Wire Wire Line
+	14400 4250 15150 4250
+Wire Wire Line
+	14400 4350 15150 4350
+Wire Wire Line
+	14400 4450 15150 4450
+Wire Wire Line
+	14400 4550 15150 4550
+Wire Wire Line
+	14400 4750 14450 4750
+Wire Wire Line
+	14450 4750 14450 4650
+Wire Wire Line
+	14450 4650 15150 4650
+Wire Wire Line
+	14400 4850 14500 4850
+Wire Wire Line
+	14500 4850 14500 4750
+Wire Wire Line
+	14500 4750 15150 4750
+Wire Wire Line
+	14400 4950 14550 4950
+Wire Wire Line
+	14550 4950 14550 4850
+Wire Wire Line
+	14550 4850 15150 4850
+Wire Wire Line
+	14400 5050 14600 5050
+Wire Wire Line
+	14600 5050 14600 4950
+Wire Wire Line
+	14600 4950 15150 4950
+Wire Wire Line
+	14400 5550 14650 5550
+Wire Wire Line
+	14650 5550 14650 5050
+Wire Wire Line
+	14650 5050 15150 5050
+Wire Wire Line
+	14400 5650 14700 5650
+Wire Wire Line
+	14700 5650 14700 5150
+Wire Wire Line
+	14700 5150 15150 5150
+$Comp
+L conn:Conn_01x10 J?
+U 1 1 5BBC8CFA
+P 15350 4650
+F 0 "J?" H 15430 4642 50  0000 L CNN
+F 1 "Conn_01x10" H 15430 4551 50  0000 L CNN
+F 2 "" H 15350 4650 50  0001 C CNN
+F 3 "~" H 15350 4650 50  0001 C CNN
+	1    15350 4650
+	1    0    0    -1
+$EndComp
+Text Label 14700 4250 0    60   ~ 0
+GPIO10
+Text Label 14700 4350 0    60   ~ 0
+GPIO11
+Text Label 14700 4450 0    60   ~ 0
+GPIO12
+Text Label 14700 4550 0    60   ~ 0
+GPIO13
+Text Label 14700 4650 0    60   ~ 0
+GPIO14
+Text Label 14700 4750 0    60   ~ 0
+GPIO15
+Text Label 14700 4850 0    60   ~ 0
+GPIO16
+Text Label 14700 4950 0    60   ~ 0
+GPIO17
+Text Label 14700 5050 0    60   ~ 0
+GPIO18
+Text Label 14750 5150 0    60   ~ 0
+GPIO19
+Text HLabel 9100 11550 0    60   Input ~ 0
++3V3_FPGA
+Wire Wire Line
+	9100 11550 9250 11550
 Wire Bus Line
 	15000 8200 15000 8500
@@
 Wire Bus Line
 	20050 3800 20050 5500
-Text Label 8600 10850 0    60   ~ 0
-CRESET_B
 $EndSCHEMATC

Commit message: fpga.sch
Parts:
- removed J? (x2): Conn_01x10, symbol conn:Conn_01x10
- added J?: Conn_02x11_Counter_Clockwise, symbol conn:Conn_02x11_Counter_Clockwise
Connections:
- wire segments 186 -> 212
Changed lines of the file:
@@
 	12850 2950 13100 2950
 Wire Wire Line
-	9250 4200 8700 4200
-Wire Wire Line
-	9250 4300 8700 4300
-Wire Wire Line
-	9250 4400 8700 4400
-Wire Wire Line
-	9250 4500 8700 4500
-Wire Wire Line
-	9250 4600 8700 4600
-Wire Wire Line
-	9250 4700 8700 4700
-Wire Wire Line
-	9250 4800 8700 4800
-Wire Wire Line
-	9250 4900 8700 4900
-Wire Wire Line
-	9250 5000 8700 5000
-Wire Wire Line
-	9250 5100 8700 5100
-Text Label 8800 4200 0    60   ~ 0
+	9250 4200 8400 4200
+Wire Wire Line
+	9250 4300 8400 4300
+Wire Wire Line
+	9250 4400 8400 4400
+Wire Wire Line
+	9250 4500 8400 4500
+Wire Wire Line
+	9250 4600 8400 4600
+Wire Wire Line
+	9250 4700 8400 4700
+Wire Wire Line
+	9250 4800 8400 4800
+Wire Wire Line
+	9250 4900 8400 4900
+Wire Wire Line
+	9250 5000 8400 5000
+Wire Wire Line
+	9250 5100 8400 5100
+Text Label 8500 4200 0    60   ~ 0
 GPIO0
-Text Label 8800 4300 0    60   ~ 0
+Text Label 8500 4300 0    60   ~ 0
 GPIO1
-Text Label 8800 4400 0    60   ~ 0
+Text Label 8500 4400 0    60   ~ 0
 GPIO2
-Text Label 8800 4500 0    60   ~ 0
+Text Label 8500 4500 0    60   ~ 0
 GPIO3
-Text Label 8800 4600 0    60   ~ 0
+Text Label 8500 4600 0    60   ~ 0
 GPIO4
-Text Label 8800 4700 0    60   ~ 0
+Text Label 8500 4700 0    60   ~ 0
 GPIO5
-Text Label 8800 4800 0    60   ~ 0
+Text Label 8500 4800 0    60   ~ 0
 GPIO6
-Text Label 8800 4900 0    60   ~ 0
+Text Label 8500 4900 0    60   ~ 0
 GPIO7
-Text Label 8800 5000 0    60   ~ 0
+Text Label 8500 5000 0    60   ~ 0
 GPIO8
-Text Label 8800 5100 0    60   ~ 0
+Text Label 8500 5100 0    60   ~ 0
 GPIO9
-$Comp
-L conn:Conn_01x10 J?
-U 1 1 5BB3EB2A
-P 8500 4600
-F 0 "J?" H 8420 5217 50  0000 C CNN
-F 1 "Conn_01x10" H 8420 5126 50  0000 C CNN
-F 2 "" H 8500 4600 50  0001 C CNN
-F 3 "~" H 8500 4600 50  0001 C CNN
-	1    8500 4600
-	-1   0    0    -1
-$EndComp
 Wire Wire Line
 	14400 4250 15150 4250
@@
 Wire Wire Line
 	14700 5150 15150 5150
-$Comp
-L conn:Conn_01x10 J?
-U 1 1 5BBC8CFA
-P 15350 4650
-F 0 "J?" H 15430 4642 50  0000 L CNN
-F 1 "Conn_01x10" H 15430 4551 50  0000 L CNN
-F 2 "" H 15350 4650 50  0001 C CNN
-F 3 "~" H 15350 4650 50  0001 C CNN
-	1    15350 4650
-	1    0    0    -1
-$EndComp
 Text Label 14700 4250 0    60   ~ 0
 GPIO10
@@
 Wire Wire Line
 	9100 11550 9250 11550
+$Comp
+L conn:Conn_02x11_Counter_Clockwise J?
+U 1 1 5BC29906
+P 8100 4600
+F 0 "J?" H 8150 5317 50  0000 C CNN
+F 1 "Conn_02x11_Counter_Clockwise" H 8150 5226 50  0000 C CNN
+F 2 "" H 8100 4600 50  0001 C CNN
+F 3 "~" H 8100 4600 50  0001 C CNN
+	1    8100 4600
+	1    0    0    -1
+$EndComp
+Text HLabel 8850 4100 2    60   Input ~ 0
++3V3_FPGA
+Wire Wire Line
+	8400 4100 8850 4100
+Wire Wire Line
+	7150 4200 7900 4200
+Wire Wire Line
+	7150 4300 7900 4300
+Wire Wire Line
+	7150 4400 7900 4400
+Wire Wire Line
+	7150 4500 7900 4500
+Wire Wire Line
+	7150 4700 7200 4700
+Wire Wire Line
+	7200 4700 7200 4600
+Wire Wire Line
+	7200 4600 7900 4600
+Wire Wire Line
+	7150 4800 7250 4800
+Wire Wire Line
+	7250 4800 7250 4700
+Wire Wire Line
+	7250 4700 7900 4700
+Wire Wire Line
+	7150 4900 7300 4900
+Wire Wire Line
+	7300 4900 7300 4800
+Wire Wire Line
+	7300 4800 7900 4800
+Wire Wire Line
+	7150 5000 7350 5000
+Wire Wire Line
+	7350 5000 7350 4900
+Wire Wire Line
+	7350 4900 7900 4900
+Wire Wire Line
+	7150 5500 7400 5500
+Wire Wire Line
+	7400 5500 7400 5000
+Wire Wire Line
+	7400 5000 7900 5000
+Wire Wire Line
+	7150 5600 7450 5600
+Wire Wire Line
+	7450 5600 7450 5100
+Wire Wire Line
+	7450 5100 7900 5100
+Text Label 7450 4200 0    60   ~ 0
+GPIO10
+Text Label 7450 4300 0    60   ~ 0
+GPIO11
+Text Label 7450 4400 0    60   ~ 0
+GPIO12
+Text Label 7450 4500 0    60   ~ 0
+GPIO13
+Text Label 7450 4600 0    60   ~ 0
+GPIO14
+Text Label 7450 4700 0    60   ~ 0
+GPIO15
+Text Label 7450 4800 0    60   ~ 0
+GPIO16
+Text Label 7450 4900 0    60   ~ 0
+GPIO17
+Text Label 7450 5000 0    60   ~ 0
+GPIO18
+Text Label 7500 5100 0    60   ~ 0
+GPIO19
+Wire Wire Line
+	7900 4100 7450 4100
+Wire Wire Line
+	7450 4100 7450 3850
+Wire Wire Line
+	7450 3850 7400 3850
+$Comp
+L power:GND #PWR?
+U 1 1 5BCDECEA
+P 7400 3850
+F 0 "#PWR?" H 7400 3600 50  0001 C CNN
+F 1 "GND" H 7405 3677 50  0000 C CNN
+F 2 "" H 7400 3850 50  0001 C CNN
+F 3 "" H 7400 3850 50  0001 C CNN
+	1    7400 3850
+	0    1    1    0
+$EndComp
 Wire Bus Line
 	15000 8200 15000 8500

Commit message: perifericos stm32
Connections:
- wire segments 212 -> 211
Changed lines of the file:
@@
 EESchema Schematic File Version 4
+LIBS:power
+LIBS:74xx
 LIBS:stm32f446zetx
 LIBS:design_emb-cache
@@
 $Descr A2 23386 16535
 encoding utf-8
-Sheet 3 5
+Sheet 3 6
 Title ""
 Date ""
@@
 $EndComp
 Wire Wire Line
-	12000 3050 12000 3000
-Wire Wire Line
 	12000 2650 12550 2650
-Connection ~ 12000 3000
 Wire Wire Line
 	12000 3000 12000 2650
