File: kicad/fpga.sch (KiCad schematic (older format))
At the start: 23 parts, among them SW1 SW_Push, U4 ICE40HX1K

Commit message: fpga.sch
Parts:
- added C?: 100nF, dgk_footprints:0603, symbol device:CP1
- added R?: 10k, Resistors_SMD:R_0603_HandSoldering, symbol device:R
- added R? (x2): 4.7k, Resistors_SMD:R_0603_HandSoldering, symbol device:R
- added U?: S25FL116KOXNFIQ-11, dgk_footprints:WSON-8_2x2mm, symbol Flash:S25FL116KOXNFIQ-11
- gave numbers to parts that had none: 2
Connections:
- wire segments 211 -> 224
Changed lines of the file:
@@
 EESchema Schematic File Version 4
-LIBS:power
-LIBS:74xx
 LIBS:stm32f446zetx
 LIBS:design_emb-cache
@@
 CRESET_B
 $Comp
-L device:CP1 C?
+L device:CP1 C1
 U 1 1 5BADC284
 P 12850 2800
-F 0 "C?" H 12850 2900 50  0000 L CNN
+F 0 "C1" H 12850 2900 50  0000 L CNN
 F 1 "100nF" H 12965 2755 50  0000 L CNN
 F 2 "Capacitors_Tantalum_SMD:CP_Tantalum_Case-A_EIA-3216-18_Hand" H 12888 2650 50  0001 C CNN
@@
 	9100 11550 9250 11550
 $Comp
-L conn:Conn_02x11_Counter_Clockwise J?
+L conn:Conn_02x11_Counter_Clockwise J5
 U 1 1 5BC29906
 P 8100 4600
-F 0 "J?" H 8150 5317 50  0000 C CNN
+F 0 "J5" H 8150 5317 50  0000 C CNN
 F 1 "Conn_02x11_Counter_Clockwise" H 8150 5226 50  0000 C CNN
 F 2 "" H 8100 4600 50  0001 C CNN
@@
 	7450 3850 7400 3850
 $Comp
-L power:GND #PWR?
+L power:GND #PWR0113
 U 1 1 5BCDECEA
 P 7400 3850
-F 0 "#PWR?" H 7400 3600 50  0001 C CNN
+F 0 "#PWR0113" H 7400 3600 50  0001 C CNN
 F 1 "GND" H 7405 3677 50  0000 C CNN
 F 2 "" H 7400 3850 50  0001 C CNN
@@
 	0    1    1    0
 $EndComp
+Text HLabel 19500 8350 0    60   Input ~ 0
++3V3_FPGA
+$Comp
+L power:GND #PWR?
+U 1 1 5BB66E4F
+P 19500 9750
+F 0 "#PWR?" H 19500 9500 50  0001 C CNN
+F 1 "GND" H 19505 9577 50  0000 C CNN
+F 2 "" H 19500 9750 50  0001 C CNN
+F 3 "" H 19500 9750 50  0001 C CNN
+	1    19500 9750
+	1    0    0    -1
+$EndComp
+Wire Wire Line
+	19500 9750 19500 9700
+Text Label 20800 9200 0    60   ~ 0
+SPI_MISO
+Text Label 18400 9350 0    60   ~ 0
+SPI_MOSI
+Text Label 20450 9350 0    60   ~ 0
+SPI_SCLK
+Text Label 18400 9200 0    60   ~ 0
+SPI_SS
+Wire Wire Line
+	20150 9200 20550 9200
+$Comp
+L device:CP1 C?
+U 1 1 5BC11EAD
+P 19700 8500
+F 0 "C?" H 19700 8600 50  0000 L CNN
+F 1 "100nF" H 19815 8455 50  0000 L CNN
+F 2 "dgk_footprints:0603" H 19738 8350 50  0001 C CNN
+F 3 "" H 19700 8500 50  0001 C CNN
+	1    19700 8500
+	1    0    0    -1
+$EndComp
+Wire Wire Line
+	19700 8350 19500 8350
+Text HLabel 21300 9350 2    60   Input ~ 0
++3V3_FPGA
+$Comp
+L device:R R?
+U 1 1 5BC2563C
+P 21100 9350
+F 0 "R?" V 21200 9350 50  0000 C CNN
+F 1 "10k" V 21250 9350 50  0000 C CNN
+F 2 "Resistors_SMD:R_0603_HandSoldering" V 21030 9350 50  0001 C CNN
+F 3 "" H 21100 9350 50  0001 C CNN
+	1    21100 9350
+	0    -1   1    0
+$EndComp
+Wire Wire Line
+	20150 9350 20950 9350
+Wire Wire Line
+	21250 9350 21300 9350
+$Comp
+L Flash:S25FL116KOXNFIQ-11 U?
+U 1 1 5BB4EC35
+P 19500 9700
+F 0 "U?" H 19525 10600 60  0000 C CNN
+F 1 "S25FL116KOXNFIQ-11" H 19525 10494 60  0000 C CNN
+F 2 "dgk_footprints:WSON-8_2x2mm" H 19500 9700 60  0001 C CNN
+F 3 "" H 19500 9700 60  0001 C CNN
+	1    19500 9700
+	1    0    0    -1
+$EndComp
+Wire Wire Line
+	17750 9200 18900 9200
+Wire Wire Line
+	17750 9350 17950 9350
+$Comp
+L power:GND #PWR?
+U 1 1 5BC3509B
+P 19700 8700
+F 0 "#PWR?" H 19700 8450 50  0001 C CNN
+F 1 "GND" H 19705 8527 50  0000 C CNN
+F 2 "" H 19700 8700 50  0001 C CNN
+F 3 "" H 19700 8700 50  0001 C CNN
+	1    19700 8700
+	1    0    0    -1
+$EndComp
+Wire Wire Line
+	19700 8700 19700 8650
+Wire Wire Line
+	19500 8350 19500 9000
+Text HLabel 18700 9500 0    60   Input ~ 0
++3V3_FPGA
+Text HLabel 20350 9500 2    60   Input ~ 0
++3V3_FPGA
+Wire Wire Line
+	20350 9500 20150 9500
+Wire Wire Line
+	18900 9500 18700 9500
+$Comp
+L device:R R?
+U 1 1 5BCE0714
+P 20550 9050
+F 0 "R?" V 20650 9050 50  0000 C CNN
+F 1 "4.7k" V 20700 9050 50  0000 C CNN
+F 2 "Resistors_SMD:R_0603_HandSoldering" V 20480 9050 50  0001 C CNN
+F 3 "" H 20550 9050 50  0001 C CNN
+	1    20550 9050
+	-1   0    0    -1
+$EndComp
+$Comp
+L device:R R?
+U 1 1 5BCE07AD
+P 17950 9500
+F 0 "R?" V 18050 9500 50  0000 C CNN
+F 1 "4.7k" V 18100 9500 50  0000 C CNN
+F 2 "Resistors_SMD:R_0603_HandSoldering" V 17880 9500 50  0001 C CNN
+F 3 "" H 17950 9500 50  0001 C CNN
+	1    17950 9500
+	-1   0    0    -1
+$EndComp
+Connection ~ 20550 9200
+Wire Wire Line
+	20550 9200 21300 9200
+Connection ~ 17950 9350
+Wire Wire Line
+	17950 9350 18900 9350
+Text HLabel 20550 8900 1    60   Input ~ 0
++3V3_FPGA
 Wire Bus Line
 	15000 8200 15000 8500
@@
 Wire Bus Line
 	20050 3800 20050 5500
+Text HLabel 17950 9650 2    60   Input ~ 0
++3V3_FPGA
 $EndSCHEMATC

Commit message: corrección footprints
Parts:
- J5: footprint (none) -> Socket_Strips:Socket_Strip_Straight_2x11_Pitch2.54mm
- U4: footprint Package_QFP:TQFP-144_20x20mm_P0.5mm -> Housings_QFP:LQFP-144_20x20mm_Pitch0.5mm
- gave numbers to parts that had none: 4
- renumbered C1 to C53
Changed lines of the file:
@@
 EESchema Schematic File Version 4
+LIBS:power
+LIBS:74xx
 LIBS:stm32f446zetx
 LIBS:design_emb-cache
@@
 F 0 "U4" H 11825 11278 50  0000 C CNN
 F 1 "ICE40HX1K" H 11825 11187 50  0000 C CNN
-F 2 "Package_QFP:TQFP-144_20x20mm_P0.5mm" H 14100 10975 50  0001 R TNN
+F 2 "Housings_QFP:LQFP-144_20x20mm_Pitch0.5mm" H 14100 10975 50  0001 R TNN
 F 3 "http://www.latticesemi.com/~/media/LatticeSemi/Documents/DataSheets/iCE/iCE40LPHXFamilyDataSheet.pdf" H 9450 10925 50  0001 C CNN
 	1    11900 7200
@@
 CRESET_B
 $Comp
-L device:CP1 C1
+L device:CP1 C53
 U 1 1 5BADC284
 P 12850 2800
-F 0 "C1" H 12850 2900 50  0000 L CNN
+F 0 "C53" H 12850 2900 50  0000 L CNN
 F 1 "100nF" H 12965 2755 50  0000 L CNN
 F 2 "Capacitors_Tantalum_SMD:CP_Tantalum_Case-A_EIA-3216-18_Hand" H 12888 2650 50  0001 C CNN
@@
 F 0 "J5" H 8150 5317 50  0000 C CNN
 F 1 "Conn_02x11_Counter_Clockwise" H 8150 5226 50  0000 C CNN
-F 2 "" H 8100 4600 50  0001 C CNN
+F 2 "Socket_Strips:Socket_Strip_Straight_2x11_Pitch2.54mm" H 8100 4600 50  0001 C CNN
 F 3 "~" H 8100 4600 50  0001 C CNN
 	1    8100 4600
@@
 +3V3_FPGA
 $Comp
-L power:GND #PWR?
+L power:GND #PWR044
 U 1 1 5BB66E4F
 P 19500 9750
-F 0 "#PWR?" H 19500 9500 50  0001 C CNN
+F 0 "#PWR044" H 19500 9500 50  0001 C CNN
 F 1 "GND" H 19505 9577 50  0000 C CNN
 F 2 "" H 19500 9750 50  0001 C CNN
@@
 	20150 9200 20550 9200
 $Comp
-L device:CP1 C?
+L device:CP1 C52
 U 1 1 5BC11EAD
 P 19700 8500
-F 0 "C?" H 19700 8600 50  0000 L CNN
+F 0 "C52" H 19700 8600 50  0000 L CNN
 F 1 "100nF" H 19815 8455 50  0000 L CNN
 F 2 "dgk_footprints:0603" H 19738 8350 50  0001 C CNN
@@
 +3V3_FPGA
 $Comp
-L device:R R?
+L device:R R11
 U 1 1 5BC2563C
 P 21100 9350
-F 0 "R?" V 21200 9350 50  0000 C CNN
+F 0 "R11" V 21200 9350 50  0000 C CNN
 F 1 "10k" V 21250 9350 50  0000 C CNN
 F 2 "Resistors_SMD:R_0603_HandSoldering" V 21030 9350 50  0001 C CNN
@@
 	17750 9350 17950 9350
 $Comp
-L power:GND #PWR?
+L power:GND #PWR045
 U 1 1 5BC3509B
 P 19700 8700
-F 0 "#PWR?" H 19700 8450 50  0001 C CNN
+F 0 "#PWR045" H 19700 8450 50  0001 C CNN
 F 1 "GND" H 19705 8527 50  0000 C CNN
 F 2 "" H 19700 8700 50  0001 C CNN
@@
 	18900 9500 18700 9500
 $Comp
-L device:R R?
+L device:R R10
 U 1 1 5BCE0714
 P 20550 9050
-F 0 "R?" V 20650 9050 50  0000 C CNN
+F 0 "R10" V 20650 9050 50  0000 C CNN
 F 1 "4.7k" V 20700 9050 50  0000 C CNN
 F 2 "Resistors_SMD:R_0603_HandSoldering" V 20480 9050 50  0001 C CNN
@@
 $EndComp
 $Comp
-L device:R R?
+L device:R R9
 U 1 1 5BCE07AD
 P 17950 9500
-F 0 "R?" V 18050 9500 50  0000 C CNN
+F 0 "R9" V 18050 9500 50  0000 C CNN
 F 1 "4.7k" V 18100 9500 50  0000 C CNN
 F 2 "Resistors_SMD:R_0603_HandSoldering" V 17880 9500 50  0001 C CNN
@@
 	17950 9350 18900 9350
 Text HLabel 20550 8900 1    60   Input ~ 0
++3V3_FPGA
+Text HLabel 17950 9650 2    60   Input ~ 0
 +3V3_FPGA
 Wire Bus Line
@@
 Wire Bus Line
 	20050 3800 20050 5500
-Text HLabel 17950 9650 2    60   Input ~ 0
-+3V3_FPGA
 $EndSCHEMATC

Commit message: fp-lib-table
Parts:
- C22, C23, C24, C25, C26, C27, C28, C29, C30, C31, C32, C33, C34, C35, C36, C53: footprint Capacitors_Tantalum_SMD:CP_Tantalum_Case-A_EIA-3216-18_Hand -> Capacitors_SMD:C_0603_HandSoldering
- C52: footprint dgk_footprints:0603 -> Capacitors_SMD:C_0603_HandSoldering
Changed lines of the file:
@@
 F 0 "C26" H 10800 2900 50  0000 L CNN
 F 1 "100nF" H 10915 2755 50  0000 L CNN
-F 2 "Capacitors_Tantalum_SMD:CP_Tantalum_Case-A_EIA-3216-18_Hand" H 10838 2650 50  0001 C CNN
+F 2 "Capacitors_SMD:C_0603_HandSoldering" H 10838 2650 50  0001 C CNN
 F 3 "" H 10800 2800 50  0001 C CNN
 	1    10800 2800
@@
 F 0 "C25" H 10550 2900 50  0000 L CNN
 F 1 "100nF" H 10665 2755 50  0000 L CNN
-F 2 "Capacitors_Tantalum_SMD:CP_Tantalum_Case-A_EIA-3216-18_Hand" H 10588 2650 50  0001 C CNN
+F 2 "Capacitors_SMD:C_0603_HandSoldering" H 10588 2650 50  0001 C CNN
 F 3 "" H 10550 2800 50  0001 C CNN
 	1    10550 2800
@@
 F 0 "C24" H 10300 2900 50  0000 L CNN
 F 1 "100nF" H 10415 2755 50  0000 L CNN
-F 2 "Capacitors_Tantalum_SMD:CP_Tantalum_Case-A_EIA-3216-18_Hand" H 10338 2650 50  0001 C CNN
+F 2 "Capacitors_SMD:C_0603_HandSoldering" H 10338 2650 50  0001 C CNN
 F 3 "" H 10300 2800 50  0001 C CNN
 	1    10300 2800
@@
 F 0 "C23" H 10050 2900 50  0000 L CNN
 F 1 "100nF" H 10165 2755 50  0000 L CNN
-F 2 "Capacitors_Tantalum_SMD:CP_Tantalum_Case-A_EIA-3216-18_Hand" H 10088 2650 50  0001 C CNN
+F 2 "Capacitors_SMD:C_0603_HandSoldering" H 10088 2650 50  0001 C CNN
 F 3 "" H 10050 2800 50  0001 C CNN
 	1    10050 2800
@@
 F 0 "C22" H 9800 2900 50  0000 L CNN
 F 1 "100nF" H 9915 2755 50  0000 L CNN
-F 2 "Capacitors_Tantalum_SMD:CP_Tantalum_Case-A_EIA-3216-18_Hand" H 9838 2650 50  0001 C CNN
+F 2 "Capacitors_SMD:C_0603_HandSoldering" H 9838 2650 50  0001 C CNN
 F 3 "" H 9800 2800 50  0001 C CNN
 	1    9800 2800
@@
 F 0 "C29" H 13350 2900 50  0000 L CNN
 F 1 "100nF" H 13465 2755 50  0000 L CNN
-F 2 "Capacitors_Tantalum_SMD:CP_Tantalum_Case-A_EIA-3216-18_Hand" H 13388 2650 50  0001 C CNN
+F 2 "Capacitors_SMD:C_0603_HandSoldering" H 13388 2650 50  0001 C CNN
 F 3 "" H 13350 2800 50  0001 C CNN
 	1    13350 2800
@@
 F 0 "C28" H 13100 2900 50  0000 L CNN
 F 1 "100nF" H 13215 2755 50  0000 L CNN
-F 2 "Capacitors_Tantalum_SMD:CP_Tantalum_Case-A_EIA-3216-18_Hand" H 13138 2650 50  0001 C CNN
+F 2 "Capacitors_SMD:C_0603_HandSoldering" H 13138 2650 50  0001 C CNN
 F 3 "" H 13100 2800 50  0001 C CNN
 	1    13100 2800
@@
 F 0 "C30" H 13600 2900 50  0000 L CNN
 F 1 "100nF" H 13715 2755 50  0000 L CNN
-F 2 "Capacitors_Tantalum_SMD:CP_Tantalum_Case-A_EIA-3216-18_Hand" H 13638 2650 50  0001 C CNN
+F 2 "Capacitors_SMD:C_0603_HandSoldering" H 13638 2650 50  0001 C CNN
 F 3 "" H 13600 2800 50  0001 C CNN
 	1    13600 2800
@@
 F 0 "C31" H 13850 2900 50  0000 L CNN
 F 1 "100nF" H 13965 2755 50  0000 L CNN
-F 2 "Capacitors_Tantalum_SMD:CP_Tantalum_Case-A_EIA-3216-18_Hand" H 13888 2650 50  0001 C CNN
+F 2 "Capacitors_SMD:C_0603_HandSoldering" H 13888 2650 50  0001 C CNN
 F 3 "" H 13850 2800 50  0001 C CNN
 	1    13850 2800
@@
 F 0 "C32" H 14100 2900 50  0000 L CNN
 F 1 "100nF" H 14215 2755 50  0000 L CNN
-F 2 "Capacitors_Tantalum_SMD:CP_Tantalum_Case-A_EIA-3216-18_Hand" H 14138 2650 50  0001 C CNN
+F 2 "Capacitors_SMD:C_0603_HandSoldering" H 14138 2650 50  0001 C CNN
 F 3 "" H 14100 2800 50  0001 C CNN
 	1    14100 2800
@@
 F 0 "C33" H 14350 2900 50  0000 L CNN
 F 1 "100nF" H 14465 2755 50  0000 L CNN
-F 2 "Capacitors_Tantalum_SMD:CP_Tantalum_Case-A_EIA-3216-18_Hand" H 14388 2650 50  0001 C CNN
+F 2 "Capacitors_SMD:C_0603_HandSoldering" H 14388 2650 50  0001 C CNN
 F 3 "" H 14350 2800 50  0001 C CNN
 	1    14350 2800
@@
 F 0 "C34" H 14600 2900 50  0000 L CNN
 F 1 "100nF" H 14715 2755 50  0000 L CNN
-F 2 "Capacitors_Tantalum_SMD:CP_Tantalum_Case-A_EIA-3216-18_Hand" H 14638 2650 50  0001 C CNN
+F 2 "Capacitors_SMD:C_0603_HandSoldering" H 14638 2650 50  0001 C CNN
 F 3 "" H 14600 2800 50  0001 C CNN
 	1    14600 2800
@@
 F 0 "C35" H 14850 2900 50  0000 L CNN
 F 1 "100nF" H 14965 2755 50  0000 L CNN
-F 2 "Capacitors_Tantalum_SMD:CP_Tantalum_Case-A_EIA-3216-18_Hand" H 14888 2650 50  0001 C CNN
+F 2 "Capacitors_SMD:C_0603_HandSoldering" H 14888 2650 50  0001 C CNN
 F 3 "" H 14850 2800 50  0001 C CNN
 	1    14850 2800
@@
 F 0 "C27" H 12550 2900 50  0000 L CNN
 F 1 "100nF" H 12665 2755 50  0000 L CNN
-F 2 "Capacitors_Tantalum_SMD:CP_Tantalum_Case-A_EIA-3216-18_Hand" H 12588 2650 50  0001 C CNN
+F 2 "Capacitors_SMD:C_0603_HandSoldering" H 12588 2650 50  0001 C CNN
 F 3 "" H 12550 2800 50  0001 C CNN
 	1    12550 2800
@@
 F 0 "C36" H 17250 3350 50  0000 L CNN
 F 1 "100nF" H 17365 3205 50  0000 L CNN
-F 2 "Capacitors_Tantalum_SMD:CP_Tantalum_Case-A_EIA-3216-18_Hand" H 17288 3100 50  0001 C CNN
+F 2 "Capacitors_SMD:C_0603_HandSoldering" H 17288 3100 50  0001 C CNN
 F 3 "" H 17250 3250 50  0001 C CNN
 	1    17250 3250
@@
 F 0 "C53" H 12850 2900 50  0000 L CNN
 F 1 "100nF" H 12965 2755 50  0000 L CNN
-F 2 "Capacitors_Tantalum_SMD:CP_Tantalum_Case-A_EIA-3216-18_Hand" H 12888 2650 50  0001 C CNN
+F 2 "Capacitors_SMD:C_0603_HandSoldering" H 12888 2650 50  0001 C CNN
 F 3 "" H 12850 2800 50  0001 C CNN
 	1    12850 2800
@@
 F 0 "C52" H 19700 8600 50  0000 L CNN
 F 1 "100nF" H 19815 8455 50  0000 L CNN
-F 2 "dgk_footprints:0603" H 19738 8350 50  0001 C CNN
+F 2 "Capacitors_SMD:C_0603_HandSoldering" H 19738 8350 50  0001 C CNN
 F 3 "" H 19700 8500 50  0001 C CNN
 	1    19700 8500

Commit message: buses JTAG, FMC_AD y CTRL
Parts:
- gave numbers to parts that had none: 1
Connections:
- net labels added: CTRL0, CTRL1, CTRL2, CTRL3, CTRL4, CTRL5, CTRL[5...0], FMCAD0, FMCAD1, FMCAD10, FMCAD11, FMCAD12, FMCAD13, FMCAD14, FMCAD15, FMCAD2, FMCAD3, FMCAD4, FMCAD5, FMCAD6, FMCAD7, FMCAD8, FMCAD9, FMCAD[15...0], FMC_NAVD
- net labels removed: Cont[5...0], FMC_AD[15...0], FMC_DA0, FMC_DA1, FMC_DA10, FMC_DA11, FMC_DA12, FMC_DA13, FMC_DA14, FMC_DA15, FMC_DA2, FMC_DA3, FMC_DA4, FMC_DA5, FMC_DA6, FMC_DA7, FMC_DA8, FMC_DA9
Changed lines of the file:
@@
 	14400 8800 16250 8800
 Text Label 14500 10100 0    60   ~ 0
+FMC_NOE
+Text Label 14500 10200 0    60   ~ 0
+FMC_NWE
+Text Label 14500 10300 0    60   ~ 0
+FMC_NWAIT
+Text Label 14500 10400 0    60   ~ 0
 FMC_NE1
-Text Label 14500 10200 0    60   ~ 0
-FMC_NWAIT
-Text Label 14500 10300 0    60   ~ 0
-FMC_NWE
-Text Label 14500 10400 0    60   ~ 0
-FMC_NOE
-Text Label 14450 8000 0    60   ~ 0
-FMC_CLK
-Entry Wire Line
-	16250 10400 16350 10500
-Entry Wire Line
-	16250 10300 16350 10400
-Entry Wire Line
-	16250 10200 16350 10300
-Entry Wire Line
-	16250 10100 16350 10200
-Entry Wire Line
-	16250 8800 16350 8900
-Entry Wire Line
-	16250 8000 16350 8100
+Text Label 14450 8700 0    60   ~ 0
+FMC_NAVD
 Wire Bus Line
-	16350 8000 16600 8000
-Text HLabel 16600 8000 2    60   Output ~ 0
-Cont[5...0]
+	16350 8600 16600 8600
+Text HLabel 16600 8600 2    60   BiDi ~ 0
+CTRL[5...0]
 Text Label 14450 8400 0    60   ~ 0
 FMC_NBL0
@@
 	14900 8500 15000 8400
 Wire Wire Line
-	14400 8000 16250 8000
+	14400 8700 16250 8700
 Wire Bus Line
 	15000 8200 15100 8200
@@
 Text Label 8850 6300 0    60   ~ 0
 FMC_D15
-Wire Wire Line
-	19950 5500 19400 5500
-Wire Wire Line
-	19400 5400 19950 5400
-Text Label 19500 5400 0    60   ~ 0
-FMC_DA1
-Text Label 19500 5500 0    60   ~ 0
-FMC_DA0
-Wire Wire Line
-	19400 5200 19950 5200
-Wire Wire Line
-	19400 5300 19950 5300
-Text Label 19500 5200 0    60   ~ 0
-FMC_DA3
-Text Label 19500 5300 0    60   ~ 0
-FMC_DA2
-Text Label 19500 5100 0    60   ~ 0
-FMC_DA4
-Text Label 19500 5000 0    60   ~ 0
-FMC_DA5
-Wire Wire Line
-	19400 5100 19950 5100
-Wire Wire Line
-	19400 5000 19950 5000
-Text Label 19500 4900 0    60   ~ 0
-FMC_DA6
-Text Label 19500 4800 0    60   ~ 0
-FMC_DA7
-Text Label 19500 4700 0    60   ~ 0
-FMC_DA8
-Text Label 19500 4600 0    60   ~ 0
-FMC_DA9
-Text Label 19500 4500 0    60   ~ 0
-FMC_DA10
-Text Label 19500 4400 0    60   ~ 0
-FMC_DA11
-Text Label 19500 4300 0    60   ~ 0
-FMC_DA12
-Wire Wire Line
-	19400 4900 19950 4900
-Wire Wire Line
-	19400 4800 19950 4800
-Wire Wire Line
-	19400 4700 19950 4700
-Wire Wire Line
-	19400 4600 19950 4600
-Wire Wire Line
-	19400 4500 19950 4500
-Wire Wire Line
-	19400 4400 19950 4400
-Wire Wire Line
-	19400 4300 19950 4300
-Text Label 19500 4200 0    60   ~ 0
-FMC_DA13
-Text Label 19500 4100 0    60   ~ 0
-FMC_DA14
-Text Label 19500 4000 0    60   ~ 0
-FMC_DA15
-Wire Wire Line
-	19400 4200 19950 4200
-Wire Wire Line
-	19400 4100 19950 4100
-Wire Wire Line
-	19400 4000 19950 4000
 Entry Wire Line
 	19950 5500 20050 5400
@@
 	20050 3800 20250 3800
 Text HLabel 20250 3800 2    60   BiDi ~ 0
-FMC_AD[15...0]
+FMCAD[15...0]
 Wire Wire Line
 	19400 5850 19950 5850
@@
 	21250 9350 21300 9350
 $Comp
-L Flash:S25FL116KOXNFIQ-11 U?
+L Flash:S25FL116KOXNFIQ-11 U10
 U 1 1 5BB4EC35
 P 19500 9700
-F 0 "U?" H 19525 10600 60  0000 C CNN
+F 0 "U10" H 19525 10600 60  0000 C CNN
 F 1 "S25FL116KOXNFIQ-11" H 19525 10494 60  0000 C CNN
 F 2 "dgk_footprints:WSON-8_2x2mm" H 19500 9700 60  0001 C CNN
@@
 Text HLabel 17950 9650 2    60   Input ~ 0
 +3V3_FPGA
+Text Label 15600 8800 0    60   ~ 0
+CTRL1
+Text Label 15600 10100 0    60   ~ 0
+CTRL2
+Text Label 15600 10200 0    60   ~ 0
+CTRL3
+Text Label 15600 10300 0    60   ~ 0
+CTRL4
+Text Label 15600 10400 0    60   ~ 0
+CTRL5
+Wire Wire Line
+	18850 5500 19950 5500
+Wire Wire Line
+	18850 5400 19950 5400
+Wire Wire Line
+	18850 5200 19950 5200
+Wire Wire Line
+	18850 5300 19950 5300
+Wire Wire Line
+	18850 5100 19950 5100
+Wire Wire Line
+	18850 5000 19950 5000
+Wire Wire Line
+	18850 4900 19950 4900
+Wire Wire Line
+	18850 4800 19950 4800
+Wire Wire Line
+	18850 4700 19950 4700
+Wire Wire Line
+	18850 4600 19950 4600
+Wire Wire Line
+	18850 4500 19950 4500
+Wire Wire Line
+	18850 4400 19950 4400
+Wire Wire Line
+	18850 4300 19950 4300
+Wire Wire Line
+	18850 4200 19950 4200
+Wire Wire Line
+	18850 4100 19950 4100
+Wire Wire Line
+	18850 4000 19950 4000
+Text Label 14450 8800 0    60   ~ 0
+FMC_CLK
+Text Label 15600 8700 0    60   ~ 0
+CTRL0
+Entry Wire Line
+	16250 8700 16350 8600
+Entry Wire Line
+	16250 8800 16350 8700
+Entry Wire Line
+	16250 10100 16350 10000
+Entry Wire Line
+	16250 10200 16350 10100
+Entry Wire Line
+	16250 10300 16350 10200
+Entry Wire Line
+	16250 10400 16350 10300
+Text Label 19450 4000 0    60   ~ 0
+FMCAD0
+Text Label 19450 4100 0    60   ~ 0
+FMCAD1
+Text Label 19450 4200 0    60   ~ 0
+FMCAD2
+Text Label 19450 4300 0    60   ~ 0
+FMCAD3
+Text Label 19450 4400 0    60   ~ 0
+FMCAD4
+Text Label 19450 4500 0    60   ~ 0
+FMCAD5
+Text Label 19450 4600 0    60   ~ 0
+FMCAD6
+Text Label 19450 4700 0    60   ~ 0
+FMCAD7
+Text Label 19450 4800 0    60   ~ 0
+FMCAD8
+Text Label 19450 4900 0    60   ~ 0
+FMCAD9
+Text Label 19450 5000 0    60   ~ 0
+FMCAD10
+Text Label 19450 5100 0    60   ~ 0
+FMCAD11
+Text Label 19450 5200 0    60   ~ 0
+FMCAD12
+Text Label 19450 5300 0    60   ~ 0
+FMCAD13
+Text Label 19450 5400 0    60   ~ 0
+FMCAD14
+Text Label 19450 5500 0    60   ~ 0
+FMCAD15
+Text Label 18850 4000 0    60   ~ 0
+FMC_D0
+Text Label 18850 4100 0    60   ~ 0
+FMC_D1
+Text Label 18850 4200 0    60   ~ 0
+FMC_D2
+Text Label 18850 4300 0    60   ~ 0
+FMC_D3
+Text Label 18850 4400 0    60   ~ 0
+FMC_D4
+Text Label 18850 4500 0    60   ~ 0
+FMC_D5
+Text Label 18850 4600 0    60   ~ 0
+FMC_D6
+Text Label 18850 4700 0    60   ~ 0
+FMC_D7
+Text Label 18850 4800 0    60   ~ 0
+FMC_D8
+Text Label 18850 4900 0    60   ~ 0
+FMC_D9
+Text Label 18850 5000 0    60   ~ 0
+FMC_D10
+Text Label 18850 5100 0    60   ~ 0
+FMC_D11
+Text Label 18850 5200 0    60   ~ 0
+FMC_D12
+Text Label 18850 5300 0    60   ~ 0
+FMC_D13
+Text Label 18850 5400 0    60   ~ 0
+FMC_D14
+Text Label 18850 5500 0    60   ~ 0
+FMC_D15
 Wire Bus Line
 	15000 8200 15000 8500
 Wire Bus Line
+	16350 8600 16350 10300
+Wire Bus Line
 	7600 10650 7600 11450
 Wire Bus Line
-	16350 8000 16350 10500
-Wire Bus Line
 	20050 5700 20050 6650
