File: kicad/fpga.sch (KiCad schematic (older format))
At the start: 28 parts, among them J5 Conn_02x11_Counter_Clockwise, SW1 SW_Push, U10 S25FL116KOXNFIQ-11, U4 ICE40HX1K

Commit message: design_emb.sch
Connections:
- net labels added: FMCA16, FMCA17, FMCA18, FMCA19, FMCA20, FMCA21, FMCA22, FMCA23, FMCA24, FMCA[24...16], FMCNBL0, FMCNBL1, ICE40ENABLE[1...0], ICE40SPI[3...0], SPI0, SPI1, SPI2, SPI3
- net labels removed: FMC_A[24...16], ICE40_ENABLE[1...0], ICE40_SPI[3...0]
- wire segments 224 -> 228
Changed lines of the file:
@@
 EESchema Schematic File Version 4
-LIBS:power
-LIBS:74xx
 LIBS:stm32f446zetx
 LIBS:design_emb-cache
@@
 SPI_SS
 Wire Wire Line
-	7700 11050 9250 11050
-Wire Wire Line
-	7700 11150 9250 11150
-Wire Wire Line
-	7700 11250 9250 11250
-Wire Wire Line
-	7700 11350 9250 11350
+	6150 11700 7700 11700
+Wire Wire Line
+	6150 11800 7700 11800
+Wire Wire Line
+	6150 11900 7700 11900
+Wire Wire Line
+	6150 12000 7700 12000
 Wire Wire Line
 	11500 11800 11500 12000
@@
 FMC_NBL0
 Wire Wire Line
-	14400 8400 14900 8400
-Wire Wire Line
-	14400 8500 14900 8500
+	14400 8400 15650 8400
+Wire Wire Line
+	14400 8500 15650 8500
 Text Label 14450 8500 0    60   ~ 0
 FMC_NBL1
 Entry Wire Line
-	14900 8400 15000 8300
-Entry Wire Line
-	14900 8500 15000 8400
+	15650 8400 15750 8300
+Entry Wire Line
+	15650 8500 15750 8400
 Wire Wire Line
 	14400 8700 16250 8700
 Wire Bus Line
-	15000 8200 15100 8200
-Text HLabel 15100 8200 2    60   BiDi ~ 0
-ICE40_ENABLE[1...0]
+	15750 8200 15850 8200
+Text HLabel 15850 8200 2    60   BiDi ~ 0
+ICE40ENABLE[1...0]
 Wire Wire Line
 	9250 5800 8700 5800
@@
 Text HLabel 20250 3800 2    60   BiDi ~ 0
 FMCAD[15...0]
-Wire Wire Line
-	19400 5850 19950 5850
-Wire Wire Line
-	19400 5950 19950 5950
-Wire Wire Line
-	19400 6050 19950 6050
-Wire Wire Line
-	19400 6150 19950 6150
-Wire Wire Line
-	19400 6250 19950 6250
-Wire Wire Line
-	19400 6350 19950 6350
-Wire Wire Line
-	19400 6450 19950 6450
-Wire Wire Line
-	19400 6550 19950 6550
-Wire Wire Line
-	19400 6650 19950 6650
-Text Label 19500 5850 0    60   ~ 0
+Text Label 18850 5950 0    60   ~ 0
 FMC_A16
-Text Label 19500 5950 0    60   ~ 0
+Text Label 18850 6050 0    60   ~ 0
 FMC_A17
-Text Label 19500 6050 0    60   ~ 0
+Text Label 18850 6150 0    60   ~ 0
 FMC_A18
-Text Label 19500 6150 0    60   ~ 0
+Text Label 18850 6250 0    60   ~ 0
 FMC_A19
-Text Label 19500 6250 0    60   ~ 0
+Text Label 18850 6350 0    60   ~ 0
 FMC_A20
-Text Label 19500 6350 0    60   ~ 0
+Text Label 18850 6450 0    60   ~ 0
 FMC_A21
-Text Label 19500 6450 0    60   ~ 0
+Text Label 18850 6550 0    60   ~ 0
 FMC_A22
-Text Label 19500 6550 0    60   ~ 0
+Text Label 18850 6650 0    60   ~ 0
 FMC_A23
-Text Label 19500 6650 0    60   ~ 0
+Text Label 18850 6750 0    60   ~ 0
 FMC_A24
 Entry Wire Line
+	19950 6750 20050 6650
+Entry Wire Line
 	19950 6650 20050 6550
 Entry Wire Line
@@
 Entry Wire Line
 	19950 5950 20050 5850
-Entry Wire Line
-	19950 5850 20050 5750
 Wire Bus Line
-	20050 5700 20250 5700
-Text HLabel 20250 5700 2    60   BiDi ~ 0
-FMC_A[24...16]
+	20050 5800 20250 5800
+Text HLabel 20250 5800 2    60   BiDi ~ 0
+FMCA[24...16]
 Wire Wire Line
 	8700 6200 9250 6200
@@
 	14100 2450 13850 2450
 Connection ~ 14100 2950
-Text HLabel 7500 10650 0    60   BiDi ~ 0
-ICE40_SPI[3...0]
-Entry Wire Line
-	7600 11450 7700 11350
-Entry Wire Line
-	7600 11350 7700 11250
-Entry Wire Line
-	7600 11250 7700 11150
-Entry Wire Line
-	7600 11150 7700 11050
+Text HLabel 5950 11300 0    60   BiDi ~ 0
+ICE40SPI[3...0]
+Entry Wire Line
+	6050 12100 6150 12000
+Entry Wire Line
+	6050 12000 6150 11900
+Entry Wire Line
+	6050 11900 6150 11800
+Entry Wire Line
+	6050 11800 6150 11700
 Wire Bus Line
-	7600 10650 7500 10650
+	6050 11300 5950 11300
 Wire Wire Line
 	14100 2650 14350 2650
@@
 Text Label 18850 5500 0    60   ~ 0
 FMC_D15
+Wire Wire Line
+	18850 5950 19950 5950
+Wire Wire Line
+	18850 6050 19950 6050
+Wire Wire Line
+	18850 6150 19950 6150
+Wire Wire Line
+	18850 6250 19950 6250
+Wire Wire Line
+	18850 6350 19950 6350
+Wire Wire Line
+	18850 6450 19950 6450
+Wire Wire Line
+	18850 6550 19950 6550
+Wire Wire Line
+	18850 6650 19950 6650
+Wire Wire Line
+	18850 6750 19950 6750
+Text Label 19500 5950 0    60   ~ 0
+FMCA16
+Text Label 19500 6050 0    60   ~ 0
+FMCA17
+Text Label 19500 6150 0    60   ~ 0
+FMCA18
+Text Label 19500 6250 0    60   ~ 0
+FMCA19
+Text Label 19500 6350 0    60   ~ 0
+FMCA20
+Text Label 19500 6450 0    60   ~ 0
+FMCA21
+Text Label 19500 6550 0    60   ~ 0
+FMCA22
+Text Label 19500 6650 0    60   ~ 0
+FMCA23
+Text Label 19500 6750 0    60   ~ 0
+FMCA24
+Text Label 15050 8400 0    60   ~ 0
+FMCNBL0
+Text Label 15050 8500 0    60   ~ 0
+FMCNBL1
+Text Label 6250 11700 0    60   ~ 0
+SPI3
+Text Label 6250 11800 0    60   ~ 0
+SPI2
+Text Label 6250 11900 0    60   ~ 0
+SPI1
+Text Label 6250 12000 0    60   ~ 0
+SPI0
+Text Label 7700 11700 0    60   ~ 0
+SPI_MISO
+Text Label 7700 11800 0    60   ~ 0
+SPI_MOSI
+Text Label 7700 11900 0    60   ~ 0
+SPI_SCLK
+Text Label 7700 12000 0    60   ~ 0
+SPI_SS
+Wire Wire Line
+	7700 11050 9250 11050
+Wire Wire Line
+	7700 11150 9250 11150
+Wire Wire Line
+	7700 11250 9250 11250
+Wire Wire Line
+	7700 11350 9250 11350
 Wire Bus Line
-	15000 8200 15000 8500
+	15750 8200 15750 8500
+Wire Bus Line
+	6050 11300 6050 12100
 Wire Bus Line
 	16350 8600 16350 10300
 Wire Bus Line
-	7600 10650 7600 11450
-Wire Bus Line
-	20050 5700 20050 6650
+	20050 5800 20050 6750
 Wire Bus Line
 	20050 3800 20050 5500

Commit message: design_emb.sch
Connections:
- net labels added: FMC_NB0, FMC_NB1, ICESPI[3...0]
- net labels removed: FMC_NBL0, FMC_NBL1, ICE40ENABLE[1...0], ICE40SPI[3...0]
Changed lines of the file:
@@
 CTRL[5...0]
 Text Label 14450 8400 0    60   ~ 0
-FMC_NBL0
-Wire Wire Line
-	14400 8400 15650 8400
-Wire Wire Line
-	14400 8500 15650 8500
+FMC_NB0
 Text Label 14450 8500 0    60   ~ 0
-FMC_NBL1
-Entry Wire Line
-	15650 8400 15750 8300
-Entry Wire Line
-	15650 8500 15750 8400
+FMC_NB1
 Wire Wire Line
 	14400 8700 16250 8700
-Wire Bus Line
-	15750 8200 15850 8200
-Text HLabel 15850 8200 2    60   BiDi ~ 0
-ICE40ENABLE[1...0]
 Wire Wire Line
 	9250 5800 8700 5800
@@
 Connection ~ 14100 2950
 Text HLabel 5950 11300 0    60   BiDi ~ 0
-ICE40SPI[3...0]
+ICESPI[3...0]
 Entry Wire Line
 	6050 12100 6150 12000
@@
 Text Label 19500 6750 0    60   ~ 0
 FMCA24
-Text Label 15050 8400 0    60   ~ 0
+Text Label 16300 8400 0    60   ~ 0
 FMCNBL0
-Text Label 15050 8500 0    60   ~ 0
+Text Label 16300 8500 0    60   ~ 0
 FMCNBL1
 Text Label 6250 11700 0    60   ~ 0
@@
 Wire Wire Line
 	7700 11350 9250 11350
+Wire Wire Line
+	14400 8500 16900 8500
+Wire Wire Line
+	14400 8400 16900 8400
+Text HLabel 16900 8400 2    60   BiDi ~ 0
+FMCNBL0
+Text HLabel 16900 8500 2    60   BiDi ~ 0
+FMCNBL1
 Wire Bus Line
-	15750 8200 15750 8500
+	16350 8600 16350 10300
 Wire Bus Line
 	6050 11300 6050 12100
 Wire Bus Line
-	16350 8600 16350 10300
-Wire Bus Line
 	20050 5800 20050 6750

Commit message: bus SPI, FMC_A Y FMC_NBL
Parts:
- R9: value 4.7k -> 10k
Connections:
- net labels added: ICENBL[1.0]
Changed lines of the file:
@@
 EESchema Schematic File Version 4
+LIBS:power
+LIBS:74xx
 LIBS:stm32f446zetx
 LIBS:design_emb-cache
@@
 SPI_SS
 Wire Wire Line
-	6150 11700 7700 11700
-Wire Wire Line
-	6150 11800 7700 11800
-Wire Wire Line
-	6150 11900 7700 11900
-Wire Wire Line
-	6150 12000 7700 12000
+	9100 13600 7550 13600
+Wire Wire Line
+	9100 13700 7550 13700
+Wire Wire Line
+	9100 13800 7550 13800
+Wire Wire Line
+	9100 13900 7550 13900
 Wire Wire Line
 	11500 11800 11500 12000
@@
 	14100 2450 13850 2450
 Connection ~ 14100 2950
-Text HLabel 5950 11300 0    60   BiDi ~ 0
+Text HLabel 9300 13400 2    60   BiDi ~ 0
 ICESPI[3...0]
-Entry Wire Line
-	6050 12100 6150 12000
-Entry Wire Line
-	6050 12000 6150 11900
-Entry Wire Line
-	6050 11900 6150 11800
-Entry Wire Line
-	6050 11800 6150 11700
 Wire Bus Line
-	6050 11300 5950 11300
+	9200 13400 9300 13400
 Wire Wire Line
 	14100 2650 14350 2650
@@
 P 17950 9500
 F 0 "R9" V 18050 9500 50  0000 C CNN
-F 1 "4.7k" V 18100 9500 50  0000 C CNN
+F 1 "10k" V 18100 9500 50  0000 C CNN
 F 2 "Resistors_SMD:R_0603_HandSoldering" V 17880 9500 50  0001 C CNN
 F 3 "" H 17950 9500 50  0001 C CNN
@@
 Text HLabel 20550 8900 1    60   Input ~ 0
 +3V3_FPGA
-Text HLabel 17950 9650 2    60   Input ~ 0
+Text HLabel 17950 9650 3    60   Input ~ 0
 +3V3_FPGA
 Text Label 15600 8800 0    60   ~ 0
@@
 Text Label 19500 6750 0    60   ~ 0
 FMCA24
-Text Label 16300 8400 0    60   ~ 0
+Text Label 15150 8400 0    60   ~ 0
 FMCNBL0
-Text Label 16300 8500 0    60   ~ 0
+Text Label 15150 8500 0    60   ~ 0
 FMCNBL1
-Text Label 6250 11700 0    60   ~ 0
+Text Label 8850 13900 2    60   ~ 0
 SPI3
-Text Label 6250 11800 0    60   ~ 0
+Text Label 8850 13800 2    60   ~ 0
 SPI2
-Text Label 6250 11900 0    60   ~ 0
+Text Label 8850 13700 2    60   ~ 0
 SPI1
-Text Label 6250 12000 0    60   ~ 0
+Text Label 8850 13600 2    60   ~ 0
 SPI0
-Text Label 7700 11700 0    60   ~ 0
+Text Label 7700 13900 0    60   ~ 0
 SPI_MISO
-Text Label 7700 11800 0    60   ~ 0
+Text Label 7700 13800 0    60   ~ 0
 SPI_MOSI
-Text Label 7700 11900 0    60   ~ 0
+Text Label 7700 13700 0    60   ~ 0
 SPI_SCLK
-Text Label 7700 12000 0    60   ~ 0
+Text Label 7700 13600 0    60   ~ 0
 SPI_SS
 Wire Wire Line
@@
 	7700 11350 9250 11350
 Wire Wire Line
-	14400 8500 16900 8500
-Wire Wire Line
-	14400 8400 16900 8400
-Text HLabel 16900 8400 2    60   BiDi ~ 0
-FMCNBL0
-Text HLabel 16900 8500 2    60   BiDi ~ 0
-FMCNBL1
+	14400 8500 15800 8500
+Wire Wire Line
+	14400 8400 15800 8400
+Entry Wire Line
+	15800 8400 15900 8300
+Entry Wire Line
+	15800 8500 15900 8400
+Wire Bus Line
+	15900 8250 16100 8250
+Text HLabel 16100 8250 2    60   BiDi ~ 0
+ICENBL[1.0]
+Entry Wire Line
+	9200 13800 9100 13900
+Entry Wire Line
+	9200 13700 9100 13800
+Entry Wire Line
+	9200 13600 9100 13700
+Entry Wire Line
+	9200 13500 9100 13600
+Wire Bus Line
+	15900 8250 15900 8400
 Wire Bus Line
 	16350 8600 16350 10300
 Wire Bus Line
-	6050 11300 6050 12100
+	9200 13400 9200 13800
 Wire Bus Line
 	20050 5800 20050 6750

Commit message: fpga.sch
Parts:
- removed R9: 10k, Resistors_SMD:R_0603_HandSoldering, symbol device:R
- R11: value 10k -> 4.7k
Connections:
- wire segments 228 -> 227
Changed lines of the file:
@@
 EESchema Schematic File Version 4
-LIBS:power
-LIBS:74xx
 LIBS:stm32f446zetx
 LIBS:design_emb-cache
@@
 Wire Wire Line
 	19500 9750 19500 9700
-Text Label 20800 9200 0    60   ~ 0
+Text Label 20450 9200 0    60   ~ 0
 SPI_MISO
 Text Label 18400 9350 0    60   ~ 0
@@
 Text Label 18400 9200 0    60   ~ 0
 SPI_SS
-Wire Wire Line
-	20150 9200 20550 9200
 $Comp
 L device:CP1 C52
@@
 P 21100 9350
 F 0 "R11" V 21200 9350 50  0000 C CNN
-F 1 "10k" V 21250 9350 50  0000 C CNN
+F 1 "4.7k" V 21250 9350 50  0000 C CNN
 F 2 "Resistors_SMD:R_0603_HandSoldering" V 21030 9350 50  0001 C CNN
 F 3 "" H 21100 9350 50  0001 C CNN
@@
 $EndComp
 Wire Wire Line
-	17750 9200 18900 9200
-Wire Wire Line
-	17750 9350 17950 9350
+	17750 9200 17950 9200
 $Comp
 L power:GND #PWR045
@@
 L device:R R10
 U 1 1 5BCE0714
-P 20550 9050
-F 0 "R10" V 20650 9050 50  0000 C CNN
-F 1 "4.7k" V 20700 9050 50  0000 C CNN
-F 2 "Resistors_SMD:R_0603_HandSoldering" V 20480 9050 50  0001 C CNN
-F 3 "" H 20550 9050 50  0001 C CNN
-	1    20550 9050
+P 17950 9050
+F 0 "R10" V 18050 9050 50  0000 C CNN
+F 1 "4.7k" V 18100 9050 50  0000 C CNN
+F 2 "Resistors_SMD:R_0603_HandSoldering" V 17880 9050 50  0001 C CNN
+F 3 "" H 17950 9050 50  0001 C CNN
+	1    17950 9050
 	-1   0    0    -1
 $EndComp
-$Comp
-L device:R R9
-U 1 1 5BCE07AD
-P 17950 9500
-F 0 "R9" V 18050 9500 50  0000 C CNN
-F 1 "10k" V 18100 9500 50  0000 C CNN
-F 2 "Resistors_SMD:R_0603_HandSoldering" V 17880 9500 50  0001 C CNN
-F 3 "" H 17950 9500 50  0001 C CNN
-	1    17950 9500
-	-1   0    0    -1
-$EndComp
-Connection ~ 20550 9200
-Wire Wire Line
-	20550 9200 21300 9200
-Connection ~ 17950 9350
-Wire Wire Line
-	17950 9350 18900 9350
-Text HLabel 20550 8900 1    60   Input ~ 0
-+3V3_FPGA
-Text HLabel 17950 9650 3    60   Input ~ 0
+Text HLabel 17950 8900 1    60   Input ~ 0
 +3V3_FPGA
 Text Label 15600 8800 0    60   ~ 0
@@
 Entry Wire Line
 	9200 13500 9100 13600
+Connection ~ 17950 9200
+Wire Wire Line
+	17950 9200 18900 9200
+Wire Wire Line
+	20150 9200 21300 9200
+Wire Wire Line
+	17750 9350 18900 9350
 Wire Bus Line
 	15900 8250 15900 8400
