File: kicad/fpga.sch (KiCad schematic (older format))
At the start: 27 parts, among them J5 Conn_02x11_Counter_Clockwise, SW1 SW_Push, U10 S25FL116KOXNFIQ-11, U4 ICE40HX1K

Commit message: arreglo pines FPGA compatibilidad STM32
Parts:
- U4: footprint Housings_QFP:LQFP-144_20x20mm_Pitch0.5mm -> ICE40LPH:LQFP-144_20x20mm_Pitch0.5mm
Connections:
- net labels added: FMCNBL[1.0], SPI[3...0]
- net labels removed: ICENBL[1.0], ICESPI[3...0]
- wire segments 228 -> 220

Commit message: ruteo
Parts:
- SW1: footprint (none) -> Switch:TACTILE_SWITCH_6mm
Changed lines of the file:
@@
 F 0 "SW1" V 17654 3348 50  0000 L CNN
 F 1 "SW_Push" V 17745 3348 50  0000 L CNN
-F 2 "" H 17700 3400 50  0001 C CNN
-F 3 "" H 17700 3400 50  0001 C CNN
+F 2 "Switch:TACTILE_SWITCH_6mm" H 17700 3400 50  0001 C CNN
+F 3 "https://www.ckswitches.com/media/1471/pts645.pdf" H 17700 3400 50  0001 C CNN
 	1    17700 3200
 	0    1    1    0

Commit message: plano de tierra y modificación de señales
Parts:
- removed C35: 100nF, Capacitors_SMD:C_0603_HandSoldering, symbol device:CP1
- added L7: L, Inductors_SMD:L_0805_HandSoldering, symbol Device:L
Connections:
- net labels added: +3V3
- wire segments 220 -> 218
Changed lines of the file:
@@
 	14400 9300 16250 9300
 Wire Wire Line
-	14400 8900 16250 8900
+	14400 7900 16250 7900
 Text Label 14500 9000 0    60   ~ 0
 FMC_NOE
@@
 	1    0    0    -1
 $EndComp
-Connection ~ 14600 2650
-Wire Wire Line
-	14600 2650 14850 2650
-Connection ~ 14600 2950
-Wire Wire Line
-	14600 2950 14850 2950
-$Comp
-L device:CP1 C35
-U 1 1 5BA2D39F
-P 14850 2800
-F 0 "C35" H 14850 2900 50  0000 L CNN
-F 1 "100nF" H 14965 2755 50  0000 L CNN
-F 2 "Capacitors_SMD:C_0603_HandSoldering" H 14888 2650 50  0001 C CNN
-F 3 "" H 14850 2800 50  0001 C CNN
-	1    14850 2800
-	1    0    0    -1
-$EndComp
 $Comp
 L diode:1N5817 D3
@@
 	1    0    0    -1
 $EndComp
-Text HLabel 3850 4550 0    60   Input ~ 0
+Text HLabel 3550 4550 0    60   Input ~ 0
 +3V3_FPGA
 Wire Wire Line
@@
 $EndComp
 Text HLabel 19500 8350 0    60   Input ~ 0
-+3V3_FPGA
++3V3
 $Comp
 L power:GND #PWR044
@@
 	19700 8350 19500 8350
 Text HLabel 20700 9700 3    60   Input ~ 0
-+3V3_FPGA
++3V3
 $Comp
 L device:R R11
@@
 	19500 8350 19500 9000
 Text HLabel 18700 9500 0    60   Input ~ 0
-+3V3_FPGA
++3V3
 Text HLabel 20400 9500 3    60   Input ~ 0
-+3V3_FPGA
++3V3
 Wire Wire Line
 	20400 9500 20150 9500
@@
 $EndComp
 Text HLabel 18550 8900 1    60   Input ~ 0
-+3V3_FPGA
-Text Label 15600 8900 0    60   ~ 0
++3V3
+Text Label 15600 7900 0    60   ~ 0
 CTRL1
 Text Label 15600 9000 0    60   ~ 0
@@
 Wire Wire Line
 	18850 4000 19950 4000
-Text Label 14500 8900 0    60   ~ 0
+Text Label 14500 7900 0    60   ~ 0
 FMC_CLK
 Text Label 15700 10400 0    60   ~ 0
@@
 Wire Wire Line
 	3850 4550 4750 4550
+$Comp
+L Device:L L7
+U 1 1 5BCA4948
+P 3700 4550
+F 0 "L7" V 3522 4550 50  0000 C CNN
+F 1 "L" V 3613 4550 50  0000 C CNN
+F 2 "Inductors_SMD:L_0805_HandSoldering" H 3700 4550 50  0001 C CNN
+F 3 "~" H 3700 4550 50  0001 C CNN
+	1    3700 4550
+	0    1    1    0
+$EndComp
 Wire Bus Line
 	15900 10550 15900 10700

Commit message: modificación alimentación PLL fpga
Parts:
- added C5: 10uF, Capacitors_SMD:C_0603_HandSoldering, symbol device:CP1
- added R19: 100, Resistors_SMD:R_0603_HandSoldering, symbol device:R
- D3: footprint Diodes_THT:D_DO-41_SOD81_Horizontal_RM10 -> Diodes_SMD:D_SOD-123
Connections:
- net labels added: PLLGND, VCCPLL
- wire segments 218 -> 224
Other:
- note added: "VOLTAGE SUPPLY FILTER PLL RECOMENDED BY FABRICANT\n"
Changed lines of the file:
@@
 Wire Wire Line
 	12300 11800 12300 12000
-Connection ~ 12300 12000
-Wire Wire Line
-	12300 12000 12450 12000
 $Comp
 L power:GND #PWR013
@@
 Wire Wire Line
 	11800 3300 11800 2650
-Wire Wire Line
-	11800 2650 11600 2650
-Connection ~ 11600 2650
 NoConn ~ 14400 9500
 NoConn ~ 14400 9600
@@
 L device:CP1 C26
 U 1 1 5B9B30D6
-P 10800 2800
-F 0 "C26" H 10800 2900 50  0000 L CNN
-F 1 "100nF" H 10915 2755 50  0000 L CNN
-F 2 "Capacitors_SMD:C_0603_HandSoldering" H 10838 2650 50  0001 C CNN
-F 3 "" H 10800 2800 50  0001 C CNN
-	1    10800 2800
+P 10800 1850
+F 0 "C26" H 10800 1950 50  0000 L CNN
+F 1 "100nF" H 10915 1805 50  0000 L CNN
+F 2 "Capacitors_SMD:C_0603_HandSoldering" H 10838 1700 50  0001 C CNN
+F 3 "" H 10800 1850 50  0001 C CNN
+	1    10800 1850
 	1    0    0    -1
 $EndComp
@@
 	1    0    0    -1
 $EndComp
-Wire Wire Line
-	11300 2650 10800 2650
 Connection ~ 11300 2650
 Connection ~ 10050 2650
@@
 Wire Wire Line
 	10550 2650 10300 2650
-Connection ~ 10800 2650
-Wire Wire Line
-	10800 2650 10550 2650
 Wire Wire Line
 	9800 2950 10050 2950
@@
 Wire Wire Line
 	10300 2950 10550 2950
-Connection ~ 10550 2950
-Wire Wire Line
-	10550 2950 10800 2950
 $Comp
 L power:GND #PWR012
@@
 F 0 "D3" V 12046 3229 50  0000 L CNN
 F 1 "1N5817" V 11955 3229 50  0000 L CNN
-F 2 "Diodes_THT:D_DO-41_SOD81_Horizontal_RM10" H 12000 2975 50  0001 C CNN
+F 2 "Diodes_SMD:D_SOD-123" H 12000 2975 50  0001 C CNN
 F 3 "http://www.vishay.com/docs/88525/1n5817.pdf" H 12000 3150 50  0001 C CNN
 	1    12000 3150
@@
 	0    1    1    0
 $EndComp
+Wire Wire Line
+	10550 2650 11300 2650
+Text Label 11800 2950 1    60   ~ 0
+VCCPLL
+Text Label 12450 11800 3    60   ~ 0
+PLLGND
+$Comp
+L device:CP1 C5
+U 1 1 5BC7648D
+P 10300 1850
+F 0 "C5" H 10300 1950 50  0000 L CNN
+F 1 "10uF" H 10415 1805 50  0000 L CNN
+F 2 "Capacitors_SMD:C_0603_HandSoldering" H 10338 1700 50  0001 C CNN
+F 3 "" H 10300 1850 50  0001 C CNN
+	1    10300 1850
+	1    0    0    -1
+$EndComp
+Wire Wire Line
+	10300 1700 10300 1600
+Wire Wire Line
+	10300 1600 10800 1600
+Wire Wire Line
+	10800 1600 10800 1700
+Wire Wire Line
+	10300 2000 10300 2100
+Wire Wire Line
+	10300 2100 10800 2100
+Wire Wire Line
+	10800 2100 10800 2000
+Wire Wire Line
+	10300 1600 10050 1600
+Connection ~ 10300 1600
+Wire Wire Line
+	10800 1600 11200 1600
+Connection ~ 10800 1600
+Wire Wire Line
+	10800 2100 11200 2100
+Connection ~ 10800 2100
+Text HLabel 9600 1600 0    60   Input ~ 0
++1V2_FPGA
+$Comp
+L device:R R19
+U 1 1 5BCD929D
+P 9900 1600
+F 0 "R19" V 9800 1600 50  0000 C CNN
+F 1 "100" V 10000 1600 50  0000 C CNN
+F 2 "Resistors_SMD:R_0603_HandSoldering" V 9830 1600 50  0001 C CNN
+F 3 "" H 9900 1600 50  0001 C CNN
+	1    9900 1600
+	0    1    -1   0
+$EndComp
+Wire Wire Line
+	9750 1600 9600 1600
 Wire Bus Line
 	15900 10550 15900 10700
@@
 Wire Bus Line
 	20050 3800 20050 5500
+Text Label 10900 1600 0    60   ~ 0
+VCCPLL
+Text Label 10900 2100 0    60   ~ 0
+PLLGND
+Text Notes 8950 1450 0    60   ~ 0
+VOLTAGE SUPPLY FILTER PLL RECOMENDED BY FABRICANT\n
 $EndSCHEMATC

Commit message: soportes mecánicos y osc fpga
Parts:
- added C35, C54: 10pF, Capacitors_SMD:C_0603_HandSoldering, symbol Device:CP1
- added OSC3: 12MHz, Crystals:Crystal_SMD_Abracon_ABM8G-4pin_3.2x2.5mm, symbol device:Crystal_GND24
Connections:
- net labels added: OSC_IN, OSC_OUT
- wire segments 224 -> 232
Other:
- note added: "OSC= 12MHz"
- note added: "PLL VOLTAGE SUPPLY FILTER RECOMMENDED BY MFR.\n"
- note removed: "VOLTAGE SUPPLY FILTER PLL RECOMENDED BY FABRICANT\n"
Changed lines of the file:
@@
 Wire Wire Line
 	9750 1600 9600 1600
+Text Label 10900 1600 0    60   ~ 0
+VCCPLL
+Text Label 10900 2100 0    60   ~ 0
+PLLGND
+Text Notes 8950 1450 0    60   ~ 0
+PLL VOLTAGE SUPPLY FILTER RECOMMENDED BY MFR.\n
+Wire Wire Line
+	4900 7950 4750 7950
+Wire Wire Line
+	4750 7950 4750 7500
+Wire Wire Line
+	5200 7950 5350 7950
+Wire Wire Line
+	5350 7950 5350 7500
+$Comp
+L Device:CP1 C?
+U 1 1 5BC94ED2
+P 4750 8250
+AR Path="/5B7D9546/5BC94ED2" Ref="C?"  Part="1"
+AR Path="/5B8BCB6B/5BC94ED2" Ref="C35"  Part="1"
+F 0 "C35" H 4865 8296 50  0000 L CNN
+F 1 "10pF" H 4865 8205 50  0000 L CNN
+F 2 "Capacitors_SMD:C_0603_HandSoldering" H 4750 8250 50  0001 C CNN
+F 3 "~" H 4750 8250 50  0001 C CNN
+	1    4750 8250
+	-1   0    0    -1
+$EndComp
+$Comp
+L Device:CP1 C?
+U 1 1 5BC94ED9
+P 5350 8250
+AR Path="/5B7D9546/5BC94ED9" Ref="C?"  Part="1"
+AR Path="/5B8BCB6B/5BC94ED9" Ref="C54"  Part="1"
+F 0 "C54" H 5465 8296 50  0000 L CNN
+F 1 "10pF" H 5465 8205 50  0000 L CNN
+F 2 "Capacitors_SMD:C_0603_HandSoldering" H 5350 8250 50  0001 C CNN
+F 3 "~" H 5350 8250 50  0001 C CNN
+	1    5350 8250
+	1    0    0    -1
+$EndComp
+Wire Wire Line
+	4750 8100 4750 7950
+Connection ~ 4750 7950
+Wire Wire Line
+	5350 8100 5350 7950
+Connection ~ 5350 7950
+$Comp
+L power:GND #PWR?
+U 1 1 5BC94EE4
+P 4750 8400
+AR Path="/5B7D9546/5BC94EE4" Ref="#PWR?"  Part="1"
+AR Path="/5B8BCB6B/5BC94EE4" Ref="#PWR034"  Part="1"
+F 0 "#PWR034" H 4750 8150 50  0001 C CNN
+F 1 "GND" H 4755 8227 50  0000 C CNN
+F 2 "" H 4750 8400 50  0001 C CNN
+F 3 "" H 4750 8400 50  0001 C CNN
+	1    4750 8400
+	1    0    0    -1
+$EndComp
+$Comp
+L power:GND #PWR?
+U 1 1 5BC94EEA
+P 5350 8400
+AR Path="/5B7D9546/5BC94EEA" Ref="#PWR?"  Part="1"
+AR Path="/5B8BCB6B/5BC94EEA" Ref="#PWR053"  Part="1"
+F 0 "#PWR053" H 5350 8150 50  0001 C CNN
+F 1 "GND" H 5355 8227 50  0000 C CNN
+F 2 "" H 5350 8400 50  0001 C CNN
+F 3 "" H 5350 8400 50  0001 C CNN
+	1    5350 8400
+	1    0    0    -1
+$EndComp
+Text Notes 4400 7900 3    60   ~ 0
+OSC= 12MHz
+Text Label 4750 7850 1    60   ~ 0
+OSC_IN
+Text Label 5350 7850 1    60   ~ 0
+OSC_OUT
+$Comp
+L device:Crystal_GND24 OSC?
+U 1 1 5BC94EF3
+P 5050 7950
+AR Path="/5B7D9546/5BC94EF3" Ref="OSC?"  Part="1"
+AR Path="/5B8BCB6B/5BC94EF3" Ref="OSC3"  Part="1"
+F 0 "OSC3" H 5050 8600 50  0000 C CNN
+F 1 "12MHz" H 5050 8500 50  0000 C CNN
+F 2 "Crystals:Crystal_SMD_Abracon_ABM8G-4pin_3.2x2.5mm" H 5050 7950 50  0001 C CNN
+F 3 "https://abracon.com/Resonators/ABM8G.pdf" H 5050 7950 50  0001 C CNN
+	1    5050 7950
+	1    0    0    -1
+$EndComp
+$Comp
+L power:GND #PWR?
+U 1 1 5BC94EFA
+P 5050 8150
+AR Path="/5B7D9546/5BC94EFA" Ref="#PWR?"  Part="1"
+AR Path="/5B8BCB6B/5BC94EFA" Ref="#PWR052"  Part="1"
+F 0 "#PWR052" H 5050 7900 50  0001 C CNN
+F 1 "GND" H 5055 7977 50  0000 C CNN
+F 2 "" H 5050 8150 50  0001 C CNN
+F 3 "" H 5050 8150 50  0001 C CNN
+	1    5050 8150
+	1    0    0    -1
+$EndComp
+$Comp
+L power:GND #PWR?
+U 1 1 5BC94F00
+P 5050 7750
+AR Path="/5B7D9546/5BC94F00" Ref="#PWR?"  Part="1"
+AR Path="/5B8BCB6B/5BC94F00" Ref="#PWR051"  Part="1"
+F 0 "#PWR051" H 5050 7500 50  0001 C CNN
+F 1 "GND" H 5055 7577 50  0000 C CNN
+F 2 "" H 5050 7750 50  0001 C CNN
+F 3 "" H 5050 7750 50  0001 C CNN
+	1    5050 7750
+	-1   0    0    1
+$EndComp
+Wire Wire Line
+	9250 3800 8700 3800
+Wire Wire Line
+	9250 3900 8700 3900
 Wire Bus Line
 	15900 10550 15900 10700
@@
 Wire Bus Line
 	20050 3800 20050 5500
-Text Label 10900 1600 0    60   ~ 0
-VCCPLL
-Text Label 10900 2100 0    60   ~ 0
-PLLGND
-Text Notes 8950 1450 0    60   ~ 0
-VOLTAGE SUPPLY FILTER PLL RECOMENDED BY FABRICANT\n
+Text Label 8800 3800 0    60   ~ 0
+OSC_IN
+Text Label 8800 3900 0    60   ~ 0
+OSC_OUT
 $EndSCHEMATC

Commit message: cambio socket fpga
Parts:
- removed J5: Conn_02x11_Counter_Clockwise, Socket_Strips:Socket_Strip_Straight_2x11_Pitch2.54mm, symbol conn:Conn_02x11_Counter_Clockwise
- added J5: Conn_02x12_Counter_Clockwise, Socket_Strips:Socket_Strip_Straight_2x12_Pitch2.54mm, symbol conn:Conn_02x12_Counter_Clockwise
- added L8: L, Inductors_SMD:L_0805_HandSoldering, symbol Device:L
Connections:
- wire segments 232 -> 234
Changed lines of the file:
@@
 	12850 2950 13100 2950
 Wire Wire Line
-	4750 4650 3900 4650
-Wire Wire Line
-	4750 4750 3900 4750
-Wire Wire Line
-	4750 4850 3900 4850
-Wire Wire Line
-	4750 4950 3900 4950
-Wire Wire Line
-	4750 5050 3900 5050
-Wire Wire Line
-	4750 5150 3900 5150
-Wire Wire Line
-	4750 5250 3900 5250
-Wire Wire Line
-	4750 5350 3900 5350
-Wire Wire Line
-	4750 5450 3900 5450
-Wire Wire Line
-	6100 5450 5250 5450
-Text Label 4000 4650 0    60   ~ 0
+	4800 4950 3950 4950
+Wire Wire Line
+	4800 5050 3950 5050
+Wire Wire Line
+	4800 5150 3950 5150
+Wire Wire Line
+	4800 5250 3950 5250
+Wire Wire Line
+	4800 5350 3950 5350
+Wire Wire Line
+	4800 5450 3950 5450
+Wire Wire Line
+	4800 5550 3950 5550
+Wire Wire Line
+	4800 5650 3950 5650
+Wire Wire Line
+	4800 5750 3950 5750
+Wire Wire Line
+	4800 5850 3950 5850
+Text Label 4050 4950 0    60   ~ 0
 GPIO0
-Text Label 4000 4750 0    60   ~ 0
+Text Label 4050 5050 0    60   ~ 0
 GPIO1
-Text Label 4000 4850 0    60   ~ 0
+Text Label 4050 5150 0    60   ~ 0
 GPIO2
-Text Label 4000 4950 0    60   ~ 0
+Text Label 4050 5250 0    60   ~ 0
 GPIO3
-Text Label 4000 5050 0    60   ~ 0
+Text Label 4050 5350 0    60   ~ 0
 GPIO4
-Text Label 4000 5150 0    60   ~ 0
+Text Label 4050 5450 0    60   ~ 0
 GPIO5
-Text Label 4000 5250 0    60   ~ 0
+Text Label 4050 5550 0    60   ~ 0
 GPIO6
-Text Label 4000 5350 0    60   ~ 0
+Text Label 4050 5650 0    60   ~ 0
 GPIO7
-Text Label 4000 5450 0    60   ~ 0
+Text Label 4050 5750 0    60   ~ 0
 GPIO8
-Text Label 5350 5450 0    60   ~ 0
+Text Label 4050 5850 0    60   ~ 0
 GPIO9
 Wire Wire Line
@@
 Wire Wire Line
 	9100 11550 9250 11550
-$Comp
-L conn:Conn_02x11_Counter_Clockwise J5
-U 1 1 5BC29906
-P 4950 4950
-F 0 "J5" H 5000 5667 50  0000 C CNN
-F 1 "Conn_02x11_Counter_Clockwise" H 5000 5576 50  0000 C CNN
-F 2 "Socket_Strips:Socket_Strip_Straight_2x11_Pitch2.54mm" H 4950 4950 50  0001 C CNN
-F 3 "~" H 4950 4950 50  0001 C CNN
-	1    4950 4950
-	1    0    0    -1
-$EndComp
-Text HLabel 3550 4550 0    60   Input ~ 0
+Text HLabel 3600 4850 0    60   Input ~ 0
 +3V3_FPGA
 Wire Wire Line
-	5250 5350 6000 5350
-Wire Wire Line
-	5250 5250 6000 5250
-Wire Wire Line
-	5250 5150 6000 5150
-Wire Wire Line
-	5250 5050 6000 5050
-Text Label 5550 5350 0    60   ~ 0
+	5300 5850 6050 5850
+Wire Wire Line
+	5300 5750 6050 5750
+Wire Wire Line
+	5300 5650 6050 5650
+Wire Wire Line
+	5300 5550 6050 5550
+Text Label 5600 5850 0    60   ~ 0
 GPIO10
-Text Label 5550 5250 0    60   ~ 0
+Text Label 5600 5750 0    60   ~ 0
 GPIO11
-Text Label 5550 5150 0    60   ~ 0
+Text Label 5600 5650 0    60   ~ 0
 GPIO12
-Text Label 5550 5050 0    60   ~ 0
+Text Label 5600 5550 0    60   ~ 0
 GPIO13
-Text Label 5550 4950 0    60   ~ 0
+Text Label 5600 5450 0    60   ~ 0
 GPIO14
-Text Label 5550 4850 0    60   ~ 0
+Text Label 5600 5350 0    60   ~ 0
 GPIO15
-Text Label 5550 4750 0    60   ~ 0
+Text Label 5600 5250 0    60   ~ 0
 GPIO16
-Text Label 5550 4650 0    60   ~ 0
+Text Label 5600 5150 0    60   ~ 0
 GPIO17
-Text Label 5550 4550 0    60   ~ 0
+Text Label 5600 5050 0    60   ~ 0
 GPIO18
-Text Label 5600 4450 0    60   ~ 0
+Text Label 5650 4950 0    60   ~ 0
 GPIO19
 Wire Wire Line
-	4750 4450 4300 4450
-Wire Wire Line
-	4300 4450 4300 4200
-Wire Wire Line
-	4300 4200 4250 4200
+	4800 4750 4350 4750
+Wire Wire Line
+	4350 4750 4350 4500
+Wire Wire Line
+	4350 4500 4300 4500
 $Comp
 L power:GND #PWR0113
 U 1 1 5BCDECEA
-P 4250 4200
-F 0 "#PWR0113" H 4250 3950 50  0001 C CNN
-F 1 "GND" H 4255 4027 50  0000 C CNN
-F 2 "" H 4250 4200 50  0001 C CNN
-F 3 "" H 4250 4200 50  0001 C CNN
-	1    4250 4200
+P 4300 4500
+F 0 "#PWR0113" H 4300 4250 50  0001 C CNN
+F 1 "GND" H 4305 4327 50  0000 C CNN
+F 2 "" H 4300 4500 50  0001 C CNN
+F 3 "" H 4300 4500 50  0001 C CNN
+	1    4300 4500
 	0    1    1    0
 $EndComp
@@
 GPIO9
 Wire Wire Line
-	5250 4450 6000 4450
-Wire Wire Line
-	5250 4550 6000 4550
-Wire Wire Line
-	5250 4650 6000 4650
-Wire Wire Line
-	5250 4750 6000 4750
-Wire Wire Line
-	5250 4850 6000 4850
-Wire Wire Line
-	5250 4950 6000 4950
-Wire Wire Line
-	3850 4550 4750 4550
+	5300 4950 6050 4950
+Wire Wire Line
+	5300 5050 6050 5050
+Wire Wire Line
+	5300 5150 6050 5150
+Wire Wire Line
+	5300 5250 6050 5250
+Wire Wire Line
+	5300 5350 6050 5350
+Wire Wire Line
+	5300 5450 6050 5450
+Wire Wire Line
+	3900 4850 4800 4850
 $Comp
 L Device:L L7
 U 1 1 5BCA4948
-P 3700 4550
-F 0 "L7" V 3522 4550 50  0000 C CNN
-F 1 "L" V 3613 4550 50  0000 C CNN
-F 2 "Inductors_SMD:L_0805_HandSoldering" H 3700 4550 50  0001 C CNN
-F 3 "~" H 3700 4550 50  0001 C CNN
-	1    3700 4550
+P 3750 4850
+F 0 "L7" V 3572 4850 50  0000 C CNN
+F 1 "L" V 3663 4850 50  0000 C CNN
+F 2 "Inductors_SMD:L_0805_HandSoldering" H 3750 4850 50  0001 C CNN
+F 3 "~" H 3750 4850 50  0001 C CNN
+	1    3750 4850
 	0    1    1    0
 $EndComp
@@
 Wire Wire Line
 	9250 3900 8700 3900
+Text Label 8800 3800 0    60   ~ 0
+OSC_IN
+Text Label 8800 3900 0    60   ~ 0
+OSC_OUT
+$Comp
+L conn:Conn_02x12_Counter_Clockwise J5
+U 1 1 5BD1720C
+P 5000 5250
+F 0 "J5" H 5050 5967 50  0000 C CNN
+F 1 "Conn_02x12_Counter_Clockwise" H 5050 5876 50  0000 C CNN
+F 2 "Socket_Strips:Socket_Strip_Straight_2x12_Pitch2.54mm" H 5000 5250 50  0001 C CNN
+F 3 "~" H 5000 5250 50  0001 C CNN
+	1    5000 5250
+	1    0    0    -1
+$EndComp
+$Comp
+L power:GND #PWR0104
+U 1 1 5BD83123
+P 6100 4850
+F 0 "#PWR0104" H 6100 4600 50  0001 C CNN
+F 1 "GND" H 6105 4677 50  0000 C CNN
+F 2 "" H 6100 4850 50  0001 C CNN
+F 3 "" H 6100 4850 50  0001 C CNN
+	1    6100 4850
+	0    -1   1    0
+$EndComp
+Wire Wire Line
+	5300 4850 6100 4850
+Wire Wire Line
+	6200 4750 5300 4750
+$Comp
+L Device:L L8
+U 1 1 5BE1D34D
+P 6350 4750
+F 0 "L8" V 6172 4750 50  0000 C CNN
+F 1 "L" V 6263 4750 50  0000 C CNN
+F 2 "Inductors_SMD:L_0805_HandSoldering" H 6350 4750 50  0001 C CNN
+F 3 "~" H 6350 4750 50  0001 C CNN
+	1    6350 4750
+	0    -1   -1   0
+$EndComp
+Text HLabel 6500 4750 2    60   Input ~ 0
++3V3
 Wire Bus Line
 	15900 10550 15900 10700
@@
 Wire Bus Line
 	20050 3800 20050 5500
-Text Label 8800 3800 0    60   ~ 0
-OSC_IN
-Text Label 8800 3900 0    60   ~ 0
-OSC_OUT
 $EndSCHEMATC

Commit message: correcciones pcb
Connections:
- wire segments 234 -> 235
Changed lines of the file:
@@
 	-1   0    0    -1
 $EndComp
-Text HLabel 18550 8900 1    60   Input ~ 0
-+3V3
 Text Label 15600 7900 0    60   ~ 0
 CTRL1
@@
 Text HLabel 6500 4750 2    60   Input ~ 0
 +3V3
+$Comp
+L power:GND #PWR0117
+U 1 1 5C912591
+P 18550 8850
+F 0 "#PWR0117" H 18550 8600 50  0001 C CNN
+F 1 "GND" H 18555 8677 50  0000 C CNN
+F 2 "" H 18550 8850 50  0001 C CNN
+F 3 "" H 18550 8850 50  0001 C CNN
+	1    18550 8850
+	-1   0    0    1
+$EndComp
+Wire Wire Line
+	18550 8850 18550 8900
 Wire Bus Line
 	15900 10550 15900 10700
