File: kicad/design_emb.kicad_pcb (KiCad board)
At the start: 2 copper layers, 79.9 x 98.8 mm, 112 parts, among them J1 Conn_01x03, J2 Barrel_Jack, J3 USB_A, J4 Conn_01x03, J5 Conn_02x11_Counter_Clockwise, J6 Conn_02x10_Counter_Clockwise, J7 Screw_Terminal_01x02, J8 Screw_Terminal_01x02, K1 SANYOU_SRD_Form_C, K2 SANYOU_SRD_Form_C, Q1 MMBT3904, Q2 MMBT3904, SW1 SW_Push, SW3 SW_Push, U1 SRX.X.TCT, U10 S25FL116KOXNFIQ-11, U2 SRX.X.TCT, U3 STM32F446ZETx, U4 ICE40HX1K, U5 TLV1117LV33DCYR, U6 TLV1117LV33DCYR, U7 TLV1117LV12DCYR, U8 OMEGA2, U9 RCLAMP0502B

Commit message: design_emb.kicad_pcb
Parts:
- moved U8 70.5 mm to (88.9, 110.5), turned to 90 degrees
- moved D8 47.9 mm to (129.5, 149.7)
- moved D7 47.4 mm to (129.9, 152.4)
- moved C11 29.2 mm to (96.8, 154.7)
- moved C14 29.2 mm to (99.3, 157.2)
- moved C17 29.2 mm to (104.4, 162.3)
- moved J6 29.2 mm to (150.8, 154.5)
- moved C9 29.2 mm to (89.1, 147.1)
- moved OSC1 29.2 mm to (93.0, 150.9)
- moved U3 29.2 mm to (108.2, 143.3)
- moved U4 29.2 mm to (108.2, 143.3)
- moved OSC2 29.2 mm to (101.8, 159.8)
- moved C27 19.6 mm to (156.9, 66.0)
- moved C22 18.9 mm to (163.4, 67.2)
- moved C31 18.9 mm to (162.0, 63.9)
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Routing:
- net /sheet3/GPIO2: track 52.0 -> 0.00 mm
- net /sheet3/GPIO17: track 55.4 -> 27.4 mm
- net /sheet3/GPIO11: track 54.0 -> 26.0 mm
- net /sheet3/GPIO7: track 54.5 -> 26.6 mm
- net /sheet3/GPIO9: track 54.3 -> 26.4 mm
- net /sheet3/GPIO5: track 54.9 -> 27.0 mm
- net /sheet3/GPIO15: track 53.9 -> 26.0 mm
- net /sheet3/GPIO10: track 51.1 -> 23.1 mm
- net /sheet3/GPIO1: track 55.5 -> 27.5 mm
- net /sheet3/GPIO3: track 55.0 -> 27.1 mm
- net /sheet3/GPIO19: track 57.0 -> 29.1 mm
- net /sheet3/GPIO13: track 52.2 -> 24.2 mm
- net /sheet3/GPIO0: track 53.6 -> 25.6 mm
- net /sheet3/GPIO8: track 51.3 -> 23.3 mm
- net /sheet3/GPIO4: track 51.9 -> 23.9 mm
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Other:
- net class signals: trace_width 0.15 -> 0.25

Commit message: design_emb.kicad_pcb
Parts:
- moved J1 154.7 mm to (83.8, 90.2)
- moved J3 141.9 mm to (38.1, 59.7)
- moved U1 131.5 mm to (109.4, 92.6)
- moved U2 131.5 mm to (109.4, 89.0)
- moved U10 112.0 mm to (100.6, 115.9)
- moved K1 111.8 mm to (155.6, 114.7)
- moved K2 111.8 mm to (155.8, 96.4)
- moved R9 92.4 mm to (110.5, 114.3)
- moved R12 91.3 mm to (144.8, 160.0)
- moved LSRF1 83.6 mm to (104.9, 92.7)
- moved U9 83.6 mm to (104.9, 88.3)
- moved R8 82.5 mm to (114.3, 92.7), turned to 90 degrees
- moved J7 81.4 mm to (128.3, 115.6)
- moved R16 76.7 mm to (105.4, 119.4)
- moved R17 71.7 mm to (110.5, 119.4)
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Routing:
- net /Sheet1/USR5: track 44.3 -> 46.8 mm
- net /Sheet1/USR3: track 45.0 -> 47.3 mm
- net /Sheet1/USR4: track 47.8 -> 49.7 mm
- net /Sheet1/USR2: track 48.4 -> 49.9 mm
- net /Sheet1/USR1: track 46.6 -> 47.3 mm

Commit message: design_emb.kicad_pcb
Parts:
- moved J3 152.7 mm to (146.1, 167.6)
- moved D10 101.0 mm to (145.9, 158.8)
- moved R13 99.0 mm to (135.9, 149.9), turned to 180 degrees
- moved C1 84.8 mm to (105.4, 102.3), turned to 270 degrees
- moved C2 83.5 mm to (108.2, 102.3), turned to 270 degrees
- moved C7 83.1 mm to (114.3, 102.3), turned to 270 degrees
- moved C4 83.0 mm to (111.8, 102.3), turned to 270 degrees
- moved C10 80.4 mm to (88.9, 102.9), turned to 270 degrees
- moved C12 77.6 mm to (83.5, 102.8), turned to 270 degrees
- moved C6 76.3 mm to (91.4, 102.9), turned to 270 degrees
- moved C13 72.5 mm to (118.1, 101.6), turned to 270 degrees
- moved C8 72.2 mm to (86.4, 102.9), turned to 270 degrees
- moved C5 70.5 mm to (96.5, 102.9)
- moved C16 69.7 mm to (101.6, 102.5)
- moved C15 67.5 mm to (94.0, 102.9)
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
Commit message: ruteo
Parts:
- J4: footprint Connectors:PINHEAD1-3 -> Pin_Headers:Pin_Header_Straight_1x03_Pitch2.54mm
- U10: moved to B.Cu
- moved SW1 173.1 mm to (95.6, 174.4)
- moved R3 131.2 mm to (93.2, 168.3), turned to 180 degrees
- moved SW3 112.0 mm to (118.3, 126.2)
- moved J1 98.3 mm to (152.3, 160.7), turned to 90 degrees
- moved C46 97.6 mm to (185.6, 135.8), turned to 180 degrees
- moved U9 89.6 mm to (181.3, 135.1), turned to 180 degrees
- moved LSRF1 85.4 mm to (181.4, 130.7), turned to 180 degrees
- moved C28 75.3 mm to (169.7, 138.3), turned to 180 degrees
- moved J3 73.5 mm to (152.2, 94.4), turned to 180 degrees
- moved D6 71.5 mm to (170.7, 134.5), turned to 180 degrees
- moved R8 69.0 mm to (171.9, 130.7), turned to 270 degrees
- moved Q1 62.4 mm to (94.7, 113.0)
- moved R15 60.0 mm to (100.5, 122.3)
- moved D10 60.0 mm to (100.3, 119.7)
- moved D11 60.0 mm to (99.2, 115.9)
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Routing:
- net /Sheet2/SPI3: track 0.00 -> 75.2 mm, vias 0 -> 3
- net /Sheet2/SPI2: track 0.00 -> 75.1 mm, vias 0 -> 3
- net /Sheet2/SPI0: track 0.00 -> 67.6 mm, vias 0 -> 1
- net /Sheet2/SPI1: track 0.00 -> 65.1 mm, vias 0 -> 1
- net /Sheet1/USR18: track 49.6 -> 24.4 mm
- net /Sheet1/USR15: track 44.3 -> 19.2 mm
- net /Sheet1/USR16: track 47.9 -> 23.0 mm
- net /Sheet1/USR14: track 46.9 -> 22.2 mm
- net /Sheet1/USR17: track 45.4 -> 20.7 mm
- net /Sheet1/USR13: track 43.0 -> 19.2 mm
- net /Sheet1/USR12: track 45.4 -> 22.3 mm
- net /Sheet1/USR5: track 46.8 -> 24.9 mm
- net /Sheet1/USR3: track 47.3 -> 25.7 mm
- net /Sheet1/USR4: track 49.7 -> 28.4 mm
- net /Sheet1/USR10: track 35.9 -> 14.8 mm
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
Commit message: design_emb.kicad_pcb
Parts:
- C1, C10, C12, C13, C15, C16, C19, C2, C3, C37, C38, C4, C46, C47, C5, C51, C6, C7, C8, L3, R5, R7: moved to B.Cu
- moved R5 156.8 mm to (105.4, 163.8)
- moved R4 150.6 mm to (104.1, 162.6)
- moved D1 143.5 mm to (92.7, 163.8), turned to 90 degrees
- moved C36 141.4 mm to (104.4, 168.5)
- moved R1 139.6 mm to (96.5, 160.0), turned to 90 degrees
- moved D2 139.2 mm to (104.1, 165.1)
- moved L1 132.8 mm to (130.8, 160.0), turned to 180 degrees
- moved C20 123.6 mm to (113.0, 167.6), turned to 315 degrees
- moved R7 123.2 mm to (132.1, 141.0)
- moved R10 119.1 mm to (138.4, 137.2), turned to 180 degrees
- moved R11 116.1 mm to (138.4, 132.1)
- moved L2 114.3 mm to (92.7, 141.0)
- moved C51 112.4 mm to (134.6, 137.8)
- moved C21 107.4 mm to (129.5, 152.4), turned to 45 degrees
- moved C41 99.7 mm to (128.3, 52.1), turned to 180 degrees
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Routing:
- net /Sheet2/SPI0: track 67.6 -> 60.6 mm
- net Net-(R9-Pad1): track 2.98 -> 4.48 mm
- net /Sheet1/USR1: track 27.0 -> 25.9 mm
- net /Sheet1/USR2: track 29.2 -> 28.2 mm

Commit message: ruteo
Parts:
- added L4: L, Inductors_SMD:L_0805_HandSoldering, F.Cu at (155.3, 159.5)
- added L5: L, Inductors_SMD:L_0805_HandSoldering, F.Cu at (155.3, 161.6)
- added L6: L, Inductors_SMD:L_0805_HandSoldering, F.Cu at (105.9, 179.6)
- added L7: L, Inductors_SMD:L_0805_HandSoldering, F.Cu at (111.8, 179.8)
- C1, C2, C3: moved to F.Cu
- J1: value Conn_01x03 -> Conn_01x04; footprint Connectors_Terminal_Blocks:TerminalBlock_Altech_AK300-3_P5.00mm -> Connector_PinSocket_2.54mm:PinSocket_1x04_P2.54mm_Horizontal
- U6, U7: moved to B.Cu
- moved J2 109.8 mm to (89.4, 87.9), turned to 0 degrees
- moved Q2 109.0 mm to (82.5, 66.3)
- moved R13 104.0 mm to (89.2, 66.5)
- moved D8 92.5 mm to (107.2, 76.2), turned to 0 degrees
- moved C22 91.6 mm to (94.5, 142.0), turned to 180 degrees
- moved D7 82.6 mm to (92.2, 77.5)
- moved R12 80.7 mm to (100.8, 77.2)
- moved D11 80.4 mm to (87.4, 70.9), turned to 90 degrees
- moved Q1 79.6 mm to (83.1, 75.9)
- moved C3 62.5 mm to (95.5, 153.4), turned to 90 degrees
- moved C2 54.9 mm to (94.7, 143.8), turned to 180 degrees
- moved C1 44.4 mm to (105.4, 140.0), turned to 45 degrees
- moved R15 35.5 mm to (109.7, 66.5)
- moved D12 35.3 mm to (104.6, 66.5), turned to 0 degrees
- moved J7 25.4 mm to (85.9, 102.7), turned to 270 degrees
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Connections:
- J1 pad 3: GND -> Net-(J1-Pad3)
- J6 pad 1: VDD -> Net-(J6-Pad1)
- J6 pad 2: GND -> Net-(J6-Pad2)
- U3 pad 13: Net-(U3-Pad13) -> /Sheet5/IN_REL1
- U3 pad 14: Net-(U3-Pad14) -> /Sheet5/IN_REL2
- U3 pad 56: /Sheet5/IN_REL1 -> Net-(U3-Pad56)
- U3 pad 57: /Sheet5/IN_REL2 -> Net-(U3-Pad57)
- U8 pad 25: /Sheet2/V3.3OUT -> /3V3_O
Routing:
- net VDD: track 0.00 -> 22.2 mm, vias 0 -> 2
- net +5VA: track 0.00 -> 16.0 mm, vias 0 -> 3
- net /Sheet4/+1V2_FPGA: track 0.00 -> 8.99 mm, vias 0 -> 1
- net /Sheet1/VDDA: track 0.00 -> 6.71 mm
- net /Sheet1/OSC_IN: track 9.50 -> 5.15 mm
- net /Sheet1/USR14: track 22.2 -> 23.6 mm
- net /Sheet1/USR12: track 22.3 -> 23.6 mm
- net /Sheet1/USR13: track 19.2 -> 20.5 mm
- net /Sheet1/OSC_OUT: track 10.5 -> 11.7 mm
- net /Sheet1/USR15: track 19.2 -> 20.4 mm
- net /Sheet1/OSC32_IN: track 10.9 -> 12.0 mm
- net /sheet3/GPIO5: track 19.6 -> 20.4 mm
- net /Sheet1/USR16: track 23.0 -> 23.7 mm
- net /sheet3/GPIO13: track 18.5 -> 17.9 mm
- net /sheet3/GPIO14: track 15.3 -> 14.7 mm
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Other:
- net class power added: clearance 0.25, trace_width 1, via_dia 1.5, via_drill 0.4

Commit message: ruteo
Parts:
- C10, C13, C15, C16, C19, C4, C5, C6, C7: moved to F.Cu
- C23, C24, C25, C27, C28, C29, C30, C31, C32, C33, C34, C35, C36, C53: moved to B.Cu
- moved C31 110.9 mm to (126.6, 155.2), turned to 45 degrees
- moved C34 98.7 mm to (121.2, 160.6), turned to 225 degrees
- moved C30 97.9 mm to (112.1, 166.4), turned to 315 degrees
- moved C23 97.6 mm to (103.3, 159.3), turned to 225 degrees
- moved C27 95.9 mm to (107.6, 135.5), turned to 135 degrees
- moved C32 93.9 mm to (123.9, 140.6), turned to 45 degrees
- moved C29 92.7 mm to (104.2, 161.9), turned to 225 degrees
- moved C28 92.0 mm to (97.2, 161.5), turned to 225 degrees
- moved C53 90.4 mm to (97.9, 144.8)
- moved C35 84.6 mm to (132.8, 149.3), turned to 45 degrees
- moved C24 83.1 mm to (123.8, 158.0), turned to 45 degrees
- moved C18 77.5 mm to (97.9, 145.7), turned to 180 degrees
- moved C25 74.9 mm to (128.9, 145.7), turned to 45 degrees
- moved C33 71.0 mm to (121.0, 138.0), turned to 45 degrees
- moved C6 64.2 mm to (114.0, 166.3), turned to 315 degrees
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Connections:
- U8 pad 2: /Sheet1/JTAG2 -> /Sheet1/JTAG0
- U8 pad 4: /Sheet1/JTAG0 -> /Sheet1/JTAG2
- U8 pad 5: /Sheet2/JNRST -> /Sheet1/JTAG3
- U8 pad 7: /Sheet1/JTAG3 -> /Sheet2/JNRST
Routing:
- net /Sheet1/JTAG1: track 0.00 -> 44.8 mm, vias 0 -> 1
- net /Sheet1/JTAG0: track 0.00 -> 41.7 mm, vias 0 -> 1
- net /Sheet2/JNRST: track 0.00 -> 39.1 mm, vias 0 -> 1
- net /Sheet1/JTAG2: track 0.00 -> 37.4 mm, vias 0 -> 1
- net VDD: track 22.2 -> 57.8 mm
- net /sheet3/CRESET_B: track 0.00 -> 30.3 mm, vias 0 -> 5
- net /Sheet4/+3V3_FPGA: track 0.00 -> 30.0 mm, vias 0 -> 2
- net /Sheet1/JTAG3: track 0.00 -> 28.8 mm, vias 0 -> 1
- net /Sheet1/UART4_TX: track 0.00 -> 27.4 mm, vias 0 -> 1
- net /Sheet1/JTAG4: track 0.00 -> 26.8 mm, vias 0 -> 1
- net /Sheet1/UART4_RX: track 0.00 -> 25.2 mm, vias 0 -> 1
- net /Sheet1/BOOT1: track 0.00 -> 18.5 mm, vias 0 -> 1
- net /Sheet1/PROBE: track 0.00 -> 10.4 mm, vias 0 -> 2
- net Net-(R4-Pad1): track 0.00 -> 7.91 mm, vias 0 -> 3
- net /Sheet4/+1V2_FPGA: track 8.99 -> 16.0 mm
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
Commit message: ruteo
Parts:
- L4, L5, U1, U2: moved to B.Cu
- moved U2 33.5 mm to (145.7, 150.7), turned to 0 degrees
- moved U1 33.4 mm to (145.8, 155.1), turned to 0 degrees
- moved L5 19.1 mm to (145.4, 145.3), turned to 180 degrees
- moved L4 15.5 mm to (145.4, 147.7), turned to 180 degrees
- moved LSRF1 13.3 mm to (149.2, 112.1), turned to 270 degrees
- moved U9 9.51 mm to (161.7, 103.5)
- moved SW3 2.01 mm to (140.2, 160.1)
Routing:
- net /TX_IN: track 0.00 -> 3.81 mm
- net Net-(J1-Pad3): track 0.00 -> 3.70 mm
- net Net-(J1-Pad4): track 0.00 -> 3.66 mm
- net /RX_OUT: track 0.00 -> 2.97 mm
